File: ConvertedSchematicFiles/1-PH_BRIDGE_INVERT_RECT/1-PH_BRIDGE_INVERT_RECT.sch (KiCad schematic (older format))
At the start: 20 parts, among them U18 7408, X12 SCR3T, X13 SCR3T, X15 SCR3T, X20 SCR3T

Commit message: Excluded some components. These no longer appear after conversion. When calling shell commands, filenames are in "quotes"
Parts:
- removed U18: 7408, symbol 7408_PSPICE
- removed X12, X15: SCR3T, symbol SCR3T_PSPICE
- removed nodeMarker: nodeMarker, symbol NODEMARKER_PSPICE
- removed titleblk: titleblk, symbol TITLEBLK_PSPICE
- removed vdiffMarker (x2): vdiffMarker, symbol VDIFFMARKER_PSPICE
- U18: renamed from VG1; value VPULSE -> 7408; symbol VPULSE_PSPICE -> 7408_PSPICE
- VG1: renamed from PM6; value PARAM -> VPULSE; symbol PARAM_PSPICE -> VPULSE_PSPICE
- X13: renamed from PM7; value PARAM -> SCR3T; symbol PARAM_PSPICE -> SCR3T_PSPICE
- X20: renamed from PM8; value PARAM -> SCR3T; symbol PARAM_PSPICE -> SCR3T_PSPICE
- renumbered X20 to X12, X13 to X15
Other:
- moved on the sheet: X12, X15
Changed lines of the file:
@@
-$EndComp
-$Comp
-L PARAM_PSPICE PM6
-U 1 1 39760492
-P 1200 1200
-F 0 "PM6" H 1200 1200 30  0001 L CNN
-F 1 "PARAM" H 1200 1280 30  0001 L CNN
-	1    1200 1200
-	1    0    0    1
-$EndComp
-$Comp
-L PARAM_PSPICE PM7
-U 1 1 66516649
-P 1200 2100
-F 0 "PM7" H 1200 2100 30  0000 L CNN
-F 1 "PARAM" H 1200 2180 30  0000 L CNN
-	1    1200 2100
-	1    0    0    1
-$EndComp
-$Comp
-L PARAM_PSPICE PM8
-U 1 1 29641421
-P 1200 2900
-F 0 "PM8" H 1200 2900 30  0000 L CNN
-F 1 "PARAM" H 1200 2980 30  0000 L CNN
-	1    1200 2900
-	1    0    0    1
 $EndComp
 $Comp
 L VPULSE_PSPICE VG1
-U 1 1 45202362
+U 1 1 39760492
 P 7800 3600
 F 0 "VG1" H 7800 3600 30  0000 L CNN
@@
 $Comp
 L SCR3T_PSPICE X13
-U 1 1 10490027
+U 1 1 66516649
 P 6600 1100
 F 0 "X13" H 6600 1100 30  0000 L CNN
@@
 $Comp
 L SCR3T_PSPICE X20
-U 1 1 73368690
+U 1 1 29641421
 P 5400 2400
 F 0 "X20" H 5400 2400 30  0000 L CNN
@@
 $Comp
 L 7408_PSPICE U18
-U 1 1 32520059
+U 1 1 45202362
 P 6900 3600
 F 0 "U18" H 6900 3600 30  0000 L CNN
@@
 $Comp
 L SCR3T_PSPICE X15
-U 1 1 74897763
+U 1 1 10490027
 P 6600 2400
 F 0 "X15" H 6600 2400 30  0000 L CNN
@@
 $Comp
 L SCR3T_PSPICE X12
-U 1 1 87513926
+U 1 1 73368690
 P 5400 1100
 F 0 "X12" H 5400 1100 30  0000 L CNN
@@
 	0    -1    1    0
 $EndComp
-$Comp
-L TITLEBLK_PSPICE titleblk
-U 1 1 25180540
-P 9700 7200
-F 0 "titleblk" H 19400 14400 30  0001 L CNN
-F 1 "titleblk" H 19400 14480 30  0001 L CNN
-	1    9700 7200
-	1    0    0    1
-$EndComp
-$Comp
-L NODEMARKER_PSPICE nodeMarker
-U 1 1 20383426
-P 3900 700
-F 0 "nodeMarker" H 7800 1400 30  0001 L CNN
-F 1 "nodeMarker" H 7800 1480 30  0001 L CNN
-	1    3900 700
-	-1    0    0    1
-$EndComp
-$Comp
-L VDIFFMARKER_PSPICE vdiffMarker
-U 1 1 44089172
-P 5400 1900
-F 0 "vdiffMarker" H 10800 3800 30  0001 L CNN
-F 1 "vdiffMarker" H 10800 3880 30  0001 L CNN
-	1    5400 1900
-	1    0    0    1
-$EndComp
-$Comp
-L VDIFFMARKER_PSPICE vdiffMarker
-U 1 1 53455736
-P 6600 1900
-F 0 "vdiffMarker" H 13200 3800 30  0001 L CNN
-F 1 "vdiffMarker" H 13200 3880 30  0001 L CNN
-	1    6600 1900
-	1    0    0    1
-$EndComp
 Wire Wire Line

Commit message: Ports issue fixed. Now annotation for ports is #PWR? function added "itos"
Parts:
- removed EGND (x3): EGND, symbol EGND_PSPICE
Connections:
- net labels added: EGND
Changed lines of the file:
@@
 $EndDescr
 $Comp
-L EGND_PSPICE EGND
+L EGND_PSPICE #PWR1
 U 1 1 14289383
 P 7300 4400
-F 0 "EGND" H 14600 8800 30  0001 L CNN
+F 0 "#PWR1" H 14600 8800 30  0001 L CNN
 F 1 "EGND" H 14600 8880 30  0001 L CNN
 	1    7300 4400
@@
 $EndComp
 $Comp
-L EGND_PSPICE EGND
+L EGND_PSPICE #PWR2
 U 1 1 46930886
 P 7800 4000
-F 0 "EGND" H 15600 8000 30  0001 L CNN
+F 0 "#PWR2" H 15600 8000 30  0001 L CNN
 F 1 "EGND" H 15600 8080 30  0001 L CNN
 	1    7800 4000
@@
 $EndComp
 $Comp
-L EGND_PSPICE EGND
+L EGND_PSPICE #PWR3
 U 1 1 71692777
 P 4000 3100
-F 0 "EGND" H 8000 6200 30  0001 L CNN
+F 0 "#PWR3" H 8000 6200 30  0001 L CNN
 F 1 "EGND" H 8000 6280 30  0001 L CNN
 	1    4000 3100

Commit message: Added LICENSE.txt
Parts:
- VCYCLO, VG1: value VPULSE -> PULSE
- VIN: value VSIN -> SINE
Changed lines of the file:
@@
 $EndDescr
 $Comp
-L EGND_PSPICE #PWR1
+L GND #PWR1
 U 1 1 14289383
 P 7300 4400
@@
 $EndComp
 $Comp
-L EGND_PSPICE #PWR2
+L GND #PWR2
 U 1 1 46930886
 P 7800 4000
@@
 $EndComp
 $Comp
-L EGND_PSPICE #PWR3
+L GND #PWR3
 U 1 1 71692777
 P 4000 3100
@@
 P 5800 1900
 F 0 "VIN" H 5800 1900 30  0001 L CNN
-F 1 "VSIN" H 5800 1980 30  0001 L CNN
+F 1 "SINE" H 5800 1980 30  0001 L CNN
 	1    5800 1900
 	0    1    -1    0
@@
 P 7300 4000
 F 0 "VCYCLO" H 7300 4000 30  0000 L CNN
-F 1 "VPULSE" H 7300 4080 30  0000 L CNN
+F 1 "PULSE" H 7300 4080 30  0000 L CNN
 	1    7300 4000
 	-1    0    0    1
@@
 P 7800 3600
 F 0 "VG1" H 7800 3600 30  0000 L CNN
-F 1 "VPULSE" H 7800 3680 30  0000 L CNN
+F 1 "PULSE" H 7800 3680 30  0000 L CNN
 	1    7800 3600
 	-1    0    0    1

Commit message: Orientation fix. Library components are now inverted, with +ve y axis going up. In Schematic files, +ve y axis is downwards. This is how the KiCad libraries are. As a result of the above fixed, the converted GND is now oriented correctly.
Other:
- moved on the sheet: U18, VCYCLO, VG1, X12, X13, X15, X20
Changed lines of the file:
@@
 F 1 "EGND" H 14600 8880 30  0001 L CNN
 	1    7300 4400
-	-1    0    0    1
+	-1    0    0    -1
 $EndComp
 $Comp
@@
 F 1 "EGND" H 15600 8080 30  0001 L CNN
 	1    7800 4000
-	-1    0    0    1
+	-1    0    0    -1
 $EndComp
 $Comp
@@
 F 1 "EGND" H 8000 6280 30  0001 L CNN
 	1    4000 3100
-	-1    0    0    1
+	-1    0    0    -1
 $EndComp
 $Comp
@@
 F 1 "SINE" H 5800 1980 30  0001 L CNN
 	1    5800 1900
-	0    1    -1    0
+	0    -1    -1    0
 $EndComp
 $Comp
@@
 F 1 "50mh" H 3700 2030 30  0000 L CNN
 	1    3700 1600
-	0    1    1    0
+	0    -1    1    0
 $EndComp
 $Comp
@@
 F 1 "100" H 3700 1370 30  0000 L CNN
 	1    3700 1100
-	0    1    1    0
+	0    -1    1    0
 $EndComp
 $Comp
@@
 F 1 "PULSE" H 7300 4080 30  0000 L CNN
 	1    7300 4000
-	-1    0    0    1
+	-1    0    0    -1
 $EndComp
 $Comp
@@
 F 1 "PULSE" H 7800 3680 30  0000 L CNN
 	1    7800 3600
-	-1    0    0    1
+	-1    0    0    -1
 $EndComp
 $Comp
@@
 F 1 "SCR3T" H 6600 1180 30  0000 L CNN
 	1    6600 1100
-	0    -1    1    0
+	0    1    1    0
 $EndComp
 $Comp
@@
 F 1 "SCR3T" H 5400 2480 30  0000 L CNN
 	1    5400 2400
-	0    -1    1    0
+	0    1    1    0
 $EndComp
 $Comp
@@
 F 1 "7408" H 6900 3680 30  0000 L CNN
 	1    6900 3600
-	-1    0    0    1
+	-1    0    0    -1
 $EndComp
 $Comp
@@
 F 1 "SCR3T" H 6600 2480 30  0000 L CNN
 	1    6600 2400
-	0    -1    1    0
+	0    1    1    0
 $EndComp
 $Comp
@@
 F 1 "SCR3T" H 5400 1180 30  0000 L CNN
 	1    5400 1100
-	0    -1    1    0
+	0    1    1    0
 $EndComp
 Wire Wire Line

Commit message: Removed the use of exec, wrote basename function, made integration with eSim easier.
Parts:
- added U18: 7408, symbol 7408_PSPICE
- added X12, X15: SCR3T, symbol SCR3T_PSPICE
- added nodeMarker: nodeMarker, symbol nodeMarker_PSPICE
- added titleblk: titleblk, symbol titleblk_PSPICE
- added vdiffMarker (x2): vdiffMarker, symbol vdiffMarker_PSPICE
- PM6: renamed from VG1; value PULSE -> PARAM; symbol VPULSE_PSPICE -> PARAM_PSPICE
- PM7: renamed from X13; value SCR3T -> PARAM; symbol SCR3T_PSPICE -> PARAM_PSPICE
- PM8: renamed from X20; value SCR3T -> PARAM; symbol SCR3T_PSPICE -> PARAM_PSPICE
- VG1: renamed from U18; value 7408 -> PULSE; symbol 7408_PSPICE -> VPULSE_PSPICE
- renumbered X15 to X13, X12 to X20
Other:
- moved on the sheet: X13, X20
Changed lines of the file:
@@
-EESchema Schematic File Version 2  date Tuesday 07 March 2000 09:18:43 PM IST
+EESchema Schematic File Version 2  date
 LIBS:power
 LIBS:device
@@
 LIBS:contrib
 LIBS:valves
-LIBS:ConvertedSchematicFiles/1-PH_BRIDGE_INVERT_RECT-cache
 EELAYER 25  0
 EELAYER END
@@
 Sheet 1 1
 Title ""
-Date "07 Mar 2000"
+Date ""
 Rev ""
 Comp ""
@@
 $EndComp
 $Comp
+L PARAM_PSPICE PM6
+U 1 1 39760492
+P 1200 1200
+F 0 "PM6" H 1200 1200 30  0001 L CNN
+F 1 "PARAM" H 1200 1280 30  0001 L CNN
+	1    1200 1200
+	1    0    0    -1
+$EndComp
+$Comp
+L PARAM_PSPICE PM7
+U 1 1 66516649
+P 1200 2100
+F 0 "PM7" H 1200 2100 30  0000 L CNN
+F 1 "PARAM" H 1200 2180 30  0000 L CNN
+	1    1200 2100
+	1    0    0    -1
+$EndComp
+$Comp
+L PARAM_PSPICE PM8
+U 1 1 29641421
+P 1200 2900
+F 0 "PM8" H 1200 2900 30  0000 L CNN
+F 1 "PARAM" H 1200 2980 30  0000 L CNN
+	1    1200 2900
+	1    0    0    -1
+$EndComp
+$Comp
 L VPULSE_PSPICE VG1
-U 1 1 39760492
+U 1 1 45202362
 P 7800 3600
 F 0 "VG1" H 7800 3600 30  0000 L CNN
@@
 $Comp
 L SCR3T_PSPICE X13
-U 1 1 66516649
+U 1 1 10490027
 P 6600 1100
 F 0 "X13" H 6600 1100 30  0000 L CNN
@@
 $Comp
 L SCR3T_PSPICE X20
-U 1 1 29641421
+U 1 1 73368690
 P 5400 2400
 F 0 "X20" H 5400 2400 30  0000 L CNN
@@
 $Comp
 L 7408_PSPICE U18
-U 1 1 45202362
+U 1 1 32520059
 P 6900 3600
 F 0 "U18" H 6900 3600 30  0000 L CNN
@@
 $Comp
 L SCR3T_PSPICE X15
-U 1 1 10490027
+U 1 1 74897763
 P 6600 2400
 F 0 "X15" H 6600 2400 30  0000 L CNN
@@
 $Comp
 L SCR3T_PSPICE X12
-U 1 1 73368690
+U 1 1 87513926
 P 5400 1100
 F 0 "X12" H 5400 1100 30  0000 L CNN
@@
 	0    1    1    0
 $EndComp
+$Comp
+L titleblk_PSPICE titleblk
+U 1 1 25180540
+P 9700 7200
+F 0 "titleblk" H 19400 14400 30  0001 L CNN
+F 1 "titleblk" H 19400 14480 30  0001 L CNN
+	1    9700 7200
+	1    0    0    -1
+$EndComp
+$Comp
+L nodeMarker_PSPICE nodeMarker
+U 1 1 20383426
+P 3900 700
+F 0 "nodeMarker" H 7800 1400 30  0001 L CNN
+F 1 "nodeMarker" H 7800 1480 30  0001 L CNN
+	1    3900 700
+	-1    0    0    -1
+$EndComp
+$Comp
+L vdiffMarker_PSPICE vdiffMarker
+U 1 1 44089172
+P 5400 1900
+F 0 "vdiffMarker" H 10800 3800 30  0001 L CNN
+F 1 "vdiffMarker" H 10800 3880 30  0001 L CNN
+	1    5400 1900
+	1    0    0    -1
+$EndComp
+$Comp
+L vdiffMarker_PSPICE vdiffMarker
+U 1 1 53455736
+P 6600 1900
+F 0 "vdiffMarker" H 13200 3800 30  0001 L CNN
+F 1 "vdiffMarker" H 13200 3880 30  0001 L CNN
+	1    6600 1900
+	1    0    0    -1
+$EndComp
 Wire Wire Line
