File: ConvertedSchematicFiles/D_2_LEVEL(SE_SE)/D_2_LEVEL(SE_SE).sch (KiCad schematic (older format))
At the start: 10 parts

Commit message: Ports issue fixed. Now annotation for ports is #PWR? function added "itos"
Parts:
- removed EGND (x3): EGND, symbol EGND_PSPICE
Changed lines of the file:
@@
 $EndDescr
 $Comp
-L EGND_PSPICE EGND
+L EGND_PSPICE #PWR1
 U 1 1 14289383
 P 2800 1800
-F 0 "EGND" H 5600 3600 30  0001 L CNN
+F 0 "#PWR1" H 5600 3600 30  0001 L CNN
 F 1 "EGND" H 5600 3680 30  0001 L CNN
 	1    2800 1800
@@
 $EndComp
 $Comp
-L EGND_PSPICE EGND
+L EGND_PSPICE #PWR2
 U 1 1 46930886
 P 1900 1800
-F 0 "EGND" H 3800 3600 30  0001 L CNN
+F 0 "#PWR2" H 3800 3600 30  0001 L CNN
 F 1 "EGND" H 3800 3680 30  0001 L CNN
 	1    1900 1800
@@
 $EndComp
 $Comp
-L EGND_PSPICE EGND
+L EGND_PSPICE #PWR3
 U 1 1 71692777
 P 900 1200
-F 0 "EGND" H 1800 2400 30  0001 L CNN
+F 0 "#PWR3" H 1800 2400 30  0001 L CNN
 F 1 "EGND" H 1800 2480 30  0001 L CNN
 	1    900 1200

Commit message: Added LICENSE.txt
Changed lines of the file:
@@
 $EndDescr
 $Comp
-L EGND_PSPICE #PWR1
+L GND #PWR1
 U 1 1 14289383
 P 2800 1800
@@
 $EndComp
 $Comp
-L EGND_PSPICE #PWR2
+L GND #PWR2
 U 1 1 46930886
 P 1900 1800
@@
 $EndComp
 $Comp
-L EGND_PSPICE #PWR3
+L GND #PWR3
 U 1 1 71692777
 P 900 1200

Commit message: Orientation fix. Library components are now inverted, with +ve y axis going up. In Schematic files, +ve y axis is downwards. This is how the KiCad libraries are. As a result of the above fixed, the converted GND is now oriented correctly.
Other:
- moved on the sheet: V9
Changed lines of the file:
@@
 F 1 "EGND" H 5600 3680 30  0001 L CNN
 	1    2800 1800
-	1    0    0    1
+	1    0    0    -1
 $EndComp
 $Comp
@@
 F 1 "EGND" H 3800 3680 30  0001 L CNN
 	1    1900 1800
-	1    0    0    1
+	1    0    0    -1
 $EndComp
 $Comp
@@
 F 1 "EGND" H 1800 2480 30  0001 L CNN
 	1    900 1200
-	1    0    0    1
+	1    0    0    -1
 $EndComp
 $Comp
@@
 F 1 "D1N4002" H 2500 680 30  0001 L CNN
 	1    2500 600
-	-1    0    0    -1
+	-1    0    0    1
 $EndComp
 $Comp
@@
 F 1 "{VREF2}" H 1900 1690 30  0000 C CNN
 	1    1900 1300
-	1    0    0    1
+	1    0    0    -1
 $EndComp
 $Comp
@@
 F 1 "D1N4002" H 1400 680 30  0001 L CNN
 	1    1400 600
-	1    0    0    1
+	1    0    0    -1
 $EndComp
 $Comp
@@
 F 1 "{VREF1}" H 2800 1690 30  0000 C CNN
 	1    2800 1300
-	1    0    0    1
+	1    0    0    -1
 $EndComp
 $Comp
@@
 F 1 "100k" H 1900 970 30  0000 L CNN
 	1    1900 700
-	0    -1    1    0
+	0    1    1    0
 $EndComp
 $Comp
@@
 F 1 "200K" H 2800 970 30  0000 L CNN
 	1    2800 700
-	0    -1    1    0
+	0    1    1    0
 $EndComp
 $Comp
@@
 F 1 "VPWL" H 900 880 30  0000 L CNN
 	1    900 800
-	1    0    0    1
+	1    0    0    -1
 $EndComp
 Wire Wire Line

Commit message: Removed the use of exec, wrote basename function, made integration with eSim easier.
Parts:
- added PM1: PARAM, symbol PARAM_PSPICE
- added V9: VPWL, symbol VPWL_PSPICE
- PM2: renamed from V9; value VPWL -> PARAM; symbol VPWL_PSPICE -> PARAM_PSPICE
Changed lines of the file:
@@
-EESchema Schematic File Version 2  date Sunday 06 June 1999 09:39:02 AM IST
+EESchema Schematic File Version 2  date
 LIBS:power
 LIBS:device
@@
 LIBS:contrib
 LIBS:valves
-LIBS:ConvertedSchematicFiles/D_2_LEVEL(SE_SE)-cache
 EELAYER 25  0
 EELAYER END
@@
 Sheet 1 1
 Title ""
-Date "06 Jun 1999"
+Date ""
 Rev ""
 Comp ""
@@
 $EndComp
 $Comp
+L PARAM_PSPICE PM2
+U 1 1 29641421
+P 4100 1400
+F 0 "PM2" H 4100 1400 30  0000 L CNN
+F 1 "PARAM" H 4100 1480 30  0000 L CNN
+	1    4100 1400
+	1    0    0    -1
+$EndComp
+$Comp
 L VPWL_PSPICE V9
-U 1 1 29641421
+U 1 1 45202362
 P 900 800
 F 0 "V9" H 900 800 30  0000 L CNN
@@
 	1    0    0    -1
 $EndComp
+$Comp
+L PARAM_PSPICE PM1
+U 1 1 10490027
+P 4100 900
+F 0 "PM1" H 4100 900 30  0000 L CNN
+F 1 "PARAM" H 4100 980 30  0000 L CNN
+	1    4100 900
+	1    0    0    -1
+$EndComp
