File: ConvertedSchematicFiles/EXP10_3/EXP10_3.sch (KiCad schematic (older format))
At the start: 21 parts

Commit message: Excluded some components. These no longer appear after conversion. When calling shell commands, filenames are in "quotes"
Parts:
- removed PM2: PARAM, symbol PARAM_PSPICE
- removed R3: 100k, symbol R_PSPICE
- removed titleblk: titleblk, symbol TITLEBLK_PSPICE
- R3: renamed from PM1; value PARAM -> 100k; symbol PARAM_PSPICE -> R_PSPICE
Connections:
- net at C1.2, D1.1, V5.-: now also R3.2
- net at EGND.EGND: now also R3.1
Changed lines of the file:
@@
-$EndComp
-$Comp
-L PARAM_PSPICE PM1
-U 1 1 20383426
-P 4900 900
-F 0 "PM1" H 4900 900 30  0000 L CNN
-F 1 "PARAM" H 4900 980 30  0000 L CNN
-	1    4900 900
-	1    0    0    1
-$EndComp
-$Comp
-L PARAM_PSPICE PM2
-U 1 1 44089172
-P 4900 1500
-F 0 "PM2" H 4900 1500 30  0000 L CNN
-F 1 "PARAM" H 4900 1580 30  0000 L CNN
-	1    4900 1500
-	1    0    0    1
 $EndComp
 $Comp
 L R_PSPICE R3
-U 1 1 53455736
+U 1 1 20383426
 P 3000 1700
 F 0 "R3" H 3000 1700 30  0001 L CNN
@@
 	0    1    -1    0
 $EndComp
-$Comp
-L TITLEBLK_PSPICE titleblk
-U 1 1 45005211
-P 9700 7200
-F 0 "titleblk" H 19400 14400 30  0001 L CNN
-F 1 "titleblk" H 19400 14480 30  0001 L CNN
-	1    9700 7200
-	1    0    0    1
-$EndComp
 Wire Wire Line

Commit message: Ports issue fixed. Now annotation for ports is #PWR? function added "itos"
Parts:
- removed EGND (x8): EGND, symbol EGND_PSPICE
Changed lines of the file:
@@
 $EndDescr
 $Comp
-L EGND_PSPICE EGND
+L EGND_PSPICE #PWR1
 U 1 1 14289383
 P 1800 1300
-F 0 "EGND" H 3600 2600 30  0001 L CNN
+F 0 "#PWR1" H 3600 2600 30  0001 L CNN
 F 1 "EGND" H 3600 2680 30  0001 L CNN
 	1    1800 1300
@@
 $EndComp
 $Comp
-L EGND_PSPICE EGND
+L EGND_PSPICE #PWR2
 U 1 1 46930886
 P 1700 3100
-F 0 "EGND" H 3400 6200 30  0001 L CNN
+F 0 "#PWR2" H 3400 6200 30  0001 L CNN
 F 1 "EGND" H 3400 6280 30  0001 L CNN
 	1    1700 3100
@@
 $EndComp
 $Comp
-L EGND_PSPICE EGND
+L EGND_PSPICE #PWR3
 U 1 1 71692777
 P 1800 2600
-F 0 "EGND" H 3600 5200 30  0001 L CNN
+F 0 "#PWR3" H 3600 5200 30  0001 L CNN
 F 1 "EGND" H 3600 5280 30  0001 L CNN
 	1    1800 2600
@@
 $EndComp
 $Comp
-L EGND_PSPICE EGND
+L EGND_PSPICE #PWR4
 U 1 1 14636915
 P 1700 1800
-F 0 "EGND" H 3400 3600 30  0001 L CNN
+F 0 "#PWR4" H 3400 3600 30  0001 L CNN
 F 1 "EGND" H 3400 3680 30  0001 L CNN
 	1    1700 1800
@@
 $EndComp
 $Comp
-L EGND_PSPICE EGND
+L EGND_PSPICE #PWR5
 U 1 1 77747793
 P 1100 1500
-F 0 "EGND" H 2200 3000 30  0001 L CNN
+F 0 "#PWR5" H 2200 3000 30  0001 L CNN
 F 1 "EGND" H 2200 3080 30  0001 L CNN
 	1    1100 1500
@@
 $EndComp
 $Comp
-L EGND_PSPICE EGND
+L EGND_PSPICE #PWR6
 U 1 1 74238335
 P 1100 2900
-F 0 "EGND" H 2200 5800 30  0001 L CNN
+F 0 "#PWR6" H 2200 5800 30  0001 L CNN
 F 1 "EGND" H 2200 5880 30  0001 L CNN
 	1    1100 2900
@@
 $EndComp
 $Comp
-L EGND_PSPICE EGND
+L EGND_PSPICE #PWR7
 U 1 1 99885386
 P 3000 1900
-F 0 "EGND" H 6000 3800 30  0001 L CNN
+F 0 "#PWR7" H 6000 3800 30  0001 L CNN
 F 1 "EGND" H 6000 3880 30  0001 L CNN
 	1    3000 1900
@@
 $EndComp
 $Comp
-L EGND_PSPICE EGND
+L EGND_PSPICE #PWR8
 U 1 1 39760492
 P 3500 2200
-F 0 "EGND" H 7000 4400 30  0001 L CNN
+F 0 "#PWR8" H 7000 4400 30  0001 L CNN
 F 1 "EGND" H 7000 4480 30  0001 L CNN
 	1    3500 2200

Commit message: Added LICENSE.txt
Parts:
- V1, V2: value VPULSE -> PULSE
- V3, V4: value VSIN -> SINE
Changed lines of the file:
@@
 $EndDescr
 $Comp
-L EGND_PSPICE #PWR1
+L GND #PWR1
 U 1 1 14289383
 P 1800 1300
@@
 $EndComp
 $Comp
-L EGND_PSPICE #PWR2
+L GND #PWR2
 U 1 1 46930886
 P 1700 3100
@@
 $EndComp
 $Comp
-L EGND_PSPICE #PWR3
+L GND #PWR3
 U 1 1 71692777
 P 1800 2600
@@
 $EndComp
 $Comp
-L EGND_PSPICE #PWR4
+L GND #PWR4
 U 1 1 14636915
 P 1700 1800
@@
 $EndComp
 $Comp
-L EGND_PSPICE #PWR5
+L GND #PWR5
 U 1 1 77747793
 P 1100 1500
@@
 $EndComp
 $Comp
-L EGND_PSPICE #PWR6
+L GND #PWR6
 U 1 1 74238335
 P 1100 2900
@@
 $EndComp
 $Comp
-L EGND_PSPICE #PWR7
+L GND #PWR7
 U 1 1 99885386
 P 3000 1900
@@
 $EndComp
 $Comp
-L EGND_PSPICE #PWR8
+L GND #PWR8
 U 1 1 39760492
 P 3500 2200
@@
 P 1700 1400
 F 0 "V1" H 1700 1400 30  0001 L CNN
-F 1 "VPULSE" H 1700 1480 30  0001 L CNN
+F 1 "PULSE" H 1700 1480 30  0001 L CNN
 	1    1700 1400
 	1    0    0    1
@@
 P 1700 2700
 F 0 "V2" H 1700 2700 30  0001 L CNN
-F 1 "VPULSE" H 1700 2780 30  0001 L CNN
+F 1 "PULSE" H 1700 2780 30  0001 L CNN
 	1    1700 2700
 	1    0    0    1
@@
 P 1100 1100
 F 0 "V3" H 1100 1100 30  0001 L CNN
-F 1 "VSIN" H 1100 1180 30  0001 L CNN
+F 1 "SINE" H 1100 1180 30  0001 L CNN
 	1    1100 1100
 	1    0    0    1
@@
 P 1100 2500
 F 0 "V4" H 1100 2500 30  0001 L CNN
-F 1 "VSIN" H 1100 2580 30  0001 L CNN
+F 1 "SINE" H 1100 2580 30  0001 L CNN
 	1    1100 2500
 	1    0    0    1

Commit message: Orientation fix. Library components are now inverted, with +ve y axis going up. In Schematic files, +ve y axis is downwards. This is how the KiCad libraries are. As a result of the above fixed, the converted GND is now oriented correctly.
Other:
- moved on the sheet: V5
Changed lines of the file:
@@
 F 1 "EGND" H 3600 2680 30  0001 L CNN
 	1    1800 1300
-	0    1    -1    0
+	0    -1    -1    0
 $EndComp
 $Comp
@@
 F 1 "EGND" H 3400 6280 30  0001 L CNN
 	1    1700 3100
-	1    0    0    1
+	1    0    0    -1
 $EndComp
 $Comp
@@
 F 1 "EGND" H 3600 5280 30  0001 L CNN
 	1    1800 2600
-	0    1    -1    0
+	0    -1    -1    0
 $EndComp
 $Comp
@@
 F 1 "EGND" H 3400 3680 30  0001 L CNN
 	1    1700 1800
-	1    0    0    1
+	1    0    0    -1
 $EndComp
 $Comp
@@
 F 1 "EGND" H 2200 3080 30  0001 L CNN
 	1    1100 1500
-	1    0    0    1
+	1    0    0    -1
 $EndComp
 $Comp
@@
 F 1 "EGND" H 2200 5880 30  0001 L CNN
 	1    1100 2900
-	1    0    0    1
+	1    0    0    -1
 $EndComp
 $Comp
@@
 F 1 "EGND" H 6000 3880 30  0001 L CNN
 	1    3000 1900
-	1    0    0    1
+	1    0    0    -1
 $EndComp
 $Comp
@@
 F 1 "EGND" H 7000 4480 30  0001 L CNN
 	1    3500 2200
-	1    0    0    1
+	1    0    0    -1
 $EndComp
 $Comp
@@
 F 1 "PULSE" H 1700 1480 30  0001 L CNN
 	1    1700 1400
-	1    0    0    1
+	1    0    0    -1
 $EndComp
 $Comp
@@
 F 1 "PULSE" H 1700 2780 30  0001 L CNN
 	1    1700 2700
-	1    0    0    1
+	1    0    0    -1
 $EndComp
 $Comp
@@
 F 1 "0.01u" H 2500 1050 30  0000 L CNN
 	1    2500 900
-	1    0    0    1
+	1    0    0    -1
 $EndComp
 $Comp
@@
 F 1 "Sbreak" H 1700 2680 30  0001 L CNN
 	1    1700 2600
-	0    1    -1    0
+	0    -1    -1    0
 $EndComp
 $Comp
@@
 F 1 "Sbreak" H 1700 1380 30  0001 L CNN
 	1    1700 1300
-	0    1    -1    0
+	0    -1    -1    0
 $EndComp
 $Comp
@@
 F 1 "SINE" H 1100 1180 30  0001 L CNN
 	1    1100 1100
-	1    0    0    1
+	1    0    0    -1
 $EndComp
 $Comp
@@
 F 1 "SINE" H 1100 2580 30  0001 L CNN
 	1    1100 2500
-	1    0    0    1
+	1    0    0    -1
 $EndComp
 $Comp
@@
 F 1 "{VREF}" H 3500 2170 30  0000 C CNN
 	1    3500 1800
-	1    0    0    1
+	1    0    0    -1
 $EndComp
 $Comp
@@
 F 1 "D1N4002" H 3500 1480 30  0001 L CNN
 	1    3500 1400
-	0    -1    1    0
+	0    1    1    0
 $EndComp
 $Comp
@@
 F 1 "100k" H 3000 1710 30  0000 L CNN
 	1    3000 1700
-	0    1    -1    0
+	0    -1    -1    0
 $EndComp
 Wire Wire Line

Commit message: Removed the use of exec, wrote basename function, made integration with eSim easier.
Parts:
- added PM2: PARAM, symbol PARAM_PSPICE
- added R3: 100k, symbol R_PSPICE
- added titleblk: titleblk, symbol titleblk_PSPICE
- PM1: renamed from R3; value 100k -> PARAM; symbol R_PSPICE -> PARAM_PSPICE
Changed lines of the file:
@@
-EESchema Schematic File Version 2  date Wednesday 01 March 2000 08:19:28 PM IST
+EESchema Schematic File Version 2  date
 LIBS:power
 LIBS:device
@@
 LIBS:contrib
 LIBS:valves
-LIBS:ConvertedSchematicFiles/EXP10_3-cache
 EELAYER 25  0
 EELAYER END
@@
 Sheet 1 1
 Title ""
-Date "01 Mar 2000"
+Date ""
 Rev ""
 Comp ""
@@
 $EndComp
 $Comp
+L PARAM_PSPICE PM1
+U 1 1 20383426
+P 4900 900
+F 0 "PM1" H 4900 900 30  0000 L CNN
+F 1 "PARAM" H 4900 980 30  0000 L CNN
+	1    4900 900
+	1    0    0    -1
+$EndComp
+$Comp
+L PARAM_PSPICE PM2
+U 1 1 44089172
+P 4900 1500
+F 0 "PM2" H 4900 1500 30  0000 L CNN
+F 1 "PARAM" H 4900 1580 30  0000 L CNN
+	1    4900 1500
+	1    0    0    -1
+$EndComp
+$Comp
 L R_PSPICE R3
-U 1 1 20383426
+U 1 1 53455736
 P 3000 1700
 F 0 "R3" H 3000 1700 30  0001 L CNN
@@
 	0    -1    -1    0
 $EndComp
+$Comp
+L titleblk_PSPICE titleblk
+U 1 1 45005211
+P 9700 7200
+F 0 "titleblk" H 19400 14400 30  0001 L CNN
+F 1 "titleblk" H 19400 14480 30  0001 L CNN
+	1    9700 7200
+	1    0    0    -1
+$EndComp
 Wire Wire Line
