File: ConvertedSchematicFiles/EXP11_13/EXP11_13.sch (KiCad schematic (older format))
At the start: 15 parts, among them U1 SCR2T, U2 SCR2T, U3 SCR2T, U4 SCR2T, U5 SCR2T, U6 SCR2T

Commit message: Excluded some components. These no longer appear after conversion. When calling shell commands, filenames are in "quotes"
Parts:
- removed U4, U6: SCR2T, symbol SCR2T_PSPICE
- removed titleblk: titleblk, symbol TITLEBLK_PSPICE
- L2: renamed from R1; value 100 -> 50mH; symbol R_PSPICE -> L_PSPICE
- R1: renamed from PM3; value PARAM -> 100; symbol PARAM_PSPICE -> R_PSPICE
- U2: renamed from PM2; value PARAM -> SCR2T; symbol PARAM_PSPICE -> SCR2T_PSPICE
- U5: renamed from V3; value VSIN -> SCR2T; symbol VSIN_PSPICE -> SCR2T_PSPICE
- V1: renamed from L2; value 50mH -> VSIN; symbol L_PSPICE -> VSIN_PSPICE
- renumbered U5 to U1, U2 to U3, U3 to U4, U1 to U6, V1 to V2, V2 to V3
Connections:
- net at U4.A: now also L2.2, U2.A, U6.A; no longer V3.+
- net at U3.A: now also U4.K, V2.+; no longer V1.2
- new net: U1.A, U6.K, V1.+
- new net: R1.1, U1.K, U3.K, U5.K
- new net: U2.K, U5.A, V3.+
- new net: L2.1, R1.2
Other:
- moved on the sheet: U1, U3, U4, U6, V2, V3
Changed lines of the file:
@@
-$EndComp
-$Comp
-L PARAM_PSPICE PM3
-U 1 1 46930886
-P 8300 3200
-F 0 "PM3" H 8300 3200 30  0000 L CNN
-F 1 "PARAM" H 8300 3280 30  0000 L CNN
-	1    8300 3200
-	1    0    0    1
 $EndComp
 $Comp
 L R_PSPICE R1
-U 1 1 71692777
+U 1 1 46930886
 P 7100 2700
 F 0 "R1" H 7100 2700 30  0000 L CNN
@@
 $Comp
 L L_PSPICE L2
-U 1 1 14636915
+U 1 1 71692777
 P 7100 3100
 F 0 "L2" H 7100 3100 30  0000 L CNN
@@
 $Comp
 L VSIN_PSPICE V1
-U 1 1 77747793
+U 1 1 14636915
 P 4100 2700
 F 0 "V1" H 4100 2700 30  0000 L CNN
@@
 $Comp
 L VSIN_PSPICE V2
-U 1 1 74238335
+U 1 1 77747793
 P 4100 3200
 F 0 "V2" H 4100 3200 30  0000 L CNN
@@
 $Comp
 L VSIN_PSPICE V3
-U 1 1 99885386
+U 1 1 74238335
 P 4100 3700
 F 0 "V3" H 4100 3700 30  0000 L CNN
@@
 $EndComp
 $Comp
-L PARAM_PSPICE PM2
-U 1 1 39760492
-P 8200 2200
-F 0 "PM2" H 8200 2200 30  0001 L CNN
-F 1 "PARAM" H 8200 2280 30  0001 L CNN
-	1    8200 2200
-	1    0    0    1
-$EndComp
-$Comp
 L SCR2T_PSPICE U5
-U 1 1 66516649
+U 1 1 99885386
 P 6300 3000
 F 0 "U5" H 6300 3000 30  0000 L CNN
@@
 $Comp
 L SCR2T_PSPICE U2
-U 1 1 29641421
+U 1 1 39760492
 P 6300 4100
 F 0 "U2" H 6300 4100 30  0000 L CNN
@@
 $Comp
 L SCR2T_PSPICE U1
-U 1 1 45202362
+U 1 1 66516649
 P 5100 3000
 F 0 "U1" H 5100 3000 30  0000 L CNN
@@
 $Comp
 L SCR2T_PSPICE U3
-U 1 1 10490027
+U 1 1 29641421
 P 5700 3000
 F 0 "U3" H 5700 3000 30  0000 L CNN
@@
 $Comp
 L SCR2T_PSPICE U6
-U 1 1 73368690
+U 1 1 45202362
 P 5100 4100
 F 0 "U6" H 5100 4100 30  0000 L CNN
@@
 $Comp
 L SCR2T_PSPICE U4
-U 1 1 32520059
+U 1 1 10490027
 P 5700 4100
 F 0 "U4" H 5700 4100 30  0000 L CNN
@@
 	0    1    -1    0
 $EndComp
-$Comp
-L TITLEBLK_PSPICE titleblk
-U 1 1 74897763
-P 9700 7200
-F 0 "titleblk" H 19400 14400 30  0001 L CNN
-F 1 "titleblk" H 19400 14480 30  0001 L CNN
-	1    9700 7200
-	1    0    0    1
-$EndComp
 Wire Wire Line

Commit message: Ports issue fixed. Now annotation for ports is #PWR? function added "itos"
Parts:
- removed EGND: EGND, symbol EGND_PSPICE
Changed lines of the file:
@@
 $EndDescr
 $Comp
-L EGND_PSPICE EGND
+L EGND_PSPICE #PWR1
 U 1 1 14289383
 P 3300 3200
-F 0 "EGND" H 6600 6400 30  0001 L CNN
+F 0 "#PWR1" H 6600 6400 30  0001 L CNN
 F 1 "EGND" H 6600 6480 30  0001 L CNN
 	1    3300 3200

Commit message: Added LICENSE.txt
Changed lines of the file:
@@
 $EndDescr
 $Comp
-L EGND_PSPICE #PWR1
+L GND #PWR1
 U 1 1 14289383
 P 3300 3200

Commit message: Orientation fix. Library components are now inverted, with +ve y axis going up. In Schematic files, +ve y axis is downwards. This is how the KiCad libraries are. As a result of the above fixed, the converted GND is now oriented correctly.
Parts:
- V1, V2, V3: value VSIN -> SINE
Other:
- moved on the sheet: L2, V1, V2, V3
Changed lines of the file:
@@
 F 1 "EGND" H 6600 6480 30  0001 L CNN
 	1    3300 3200
-	1    0    0    1
+	1    0    0    -1
 $EndComp
 $Comp
@@
 F 1 "100" H 7100 3030 30  0000 L CNN
 	1    7100 2700
-	0    -1    1    0
+	0    1    1    0
 $EndComp
 $Comp
@@
 F 1 "50mH" H 7100 3430 30  0000 L CNN
 	1    7100 3100
-	0    -1    1    0
+	0    1    1    0
 $EndComp
 $Comp
@@
 P 4100 2700
 F 0 "V1" H 4100 2700 30  0000 L CNN
-F 1 "VSIN" H 4100 2780 30  0000 L CNN
+F 1 "SINE" H 4100 2780 30  0000 L CNN
 	1    4100 2700
-	0    -1    1    0
+	0    1    1    0
 $EndComp
 $Comp
@@
 P 4100 3200
 F 0 "V2" H 4100 3200 30  0000 L CNN
-F 1 "VSIN" H 4100 3280 30  0000 L CNN
+F 1 "SINE" H 4100 3280 30  0000 L CNN
 	1    4100 3200
-	0    -1    1    0
+	0    1    1    0
 $EndComp
 $Comp
@@
 P 4100 3700
 F 0 "V3" H 4100 3700 30  0000 L CNN
-F 1 "VSIN" H 4100 3780 30  0000 L CNN
+F 1 "SINE" H 4100 3780 30  0000 L CNN
 	1    4100 3700
-	0    -1    1    0
+	0    1    1    0
 $EndComp
 $Comp
@@
 F 1 "SCR2T" H 6300 3080 30  0000 L CNN
 	1    6300 3000
-	0    1    -1    0
+	0    -1    -1    0
 $EndComp
 $Comp
@@
 F 1 "SCR2T" H 6300 4180 30  0000 L CNN
 	1    6300 4100
-	0    1    -1    0
+	0    -1    -1    0
 $EndComp
 $Comp
@@
 F 1 "SCR2T" H 5100 3080 30  0000 L CNN
 	1    5100 3000
-	0    1    -1    0
+	0    -1    -1    0
 $EndComp
 $Comp
@@
 F 1 "SCR2T" H 5700 3080 30  0000 L CNN
 	1    5700 3000
-	0    1    -1    0
+	0    -1    -1    0
 $EndComp
 $Comp
@@
 F 1 "SCR2T" H 5100 4180 30  0000 L CNN
 	1    5100 4100
-	0    1    -1    0
+	0    -1    -1    0
 $EndComp
 $Comp
@@
 F 1 "SCR2T" H 5700 4180 30  0000 L CNN
 	1    5700 4100
-	0    1    -1    0
+	0    -1    -1    0
 $EndComp
 Wire Wire Line

Commit message: Removed the use of exec, wrote basename function, made integration with eSim easier.
Parts:
- added U4, U6: SCR2T, symbol SCR2T_PSPICE
- added titleblk: titleblk, symbol titleblk_PSPICE
- L2: renamed from V1; value SINE -> 50mH; symbol VSIN_PSPICE -> L_PSPICE
- PM2: renamed from U2; value SCR2T -> PARAM; symbol SCR2T_PSPICE -> PARAM_PSPICE
- PM3: renamed from R1; value 100 -> PARAM; symbol R_PSPICE -> PARAM_PSPICE
- R1: renamed from L2; value 50mH -> 100; symbol L_PSPICE -> R_PSPICE
- V3: renamed from U5; value SCR2T -> SINE; symbol SCR2T_PSPICE -> VSIN_PSPICE
- renumbered U6 to U1, U3 to U2, U4 to U3, U1 to U5, V2 to V1, V3 to V2
Other:
- moved on the sheet: U1, U2, U3, U5, V1, V2
Changed lines of the file:
@@
-EESchema Schematic File Version 2  date Tuesday 07 March 2000 10:18:46 PM IST
+EESchema Schematic File Version 2  date
 LIBS:power
 LIBS:device
@@
 LIBS:contrib
 LIBS:valves
-LIBS:ConvertedSchematicFiles/EXP11_13-cache
 EELAYER 25  0
 EELAYER END
@@
 Sheet 1 1
 Title ""
-Date "07 Mar 2000"
+Date ""
 Rev ""
 Comp ""
@@
 $EndComp
 $Comp
+L PARAM_PSPICE PM3
+U 1 1 46930886
+P 8300 3200
+F 0 "PM3" H 8300 3200 30  0000 L CNN
+F 1 "PARAM" H 8300 3280 30  0000 L CNN
+	1    8300 3200
+	1    0    0    -1
+$EndComp
+$Comp
 L R_PSPICE R1
-U 1 1 46930886
+U 1 1 71692777
 P 7100 2700
 F 0 "R1" H 7100 2700 30  0000 L CNN
@@
 $Comp
 L L_PSPICE L2
-U 1 1 71692777
+U 1 1 14636915
 P 7100 3100
 F 0 "L2" H 7100 3100 30  0000 L CNN
@@
 $Comp
 L VSIN_PSPICE V1
-U 1 1 14636915
+U 1 1 77747793
 P 4100 2700
 F 0 "V1" H 4100 2700 30  0000 L CNN
@@
 $Comp
 L VSIN_PSPICE V2
-U 1 1 77747793
+U 1 1 74238335
 P 4100 3200
 F 0 "V2" H 4100 3200 30  0000 L CNN
@@
 $Comp
 L VSIN_PSPICE V3
-U 1 1 74238335
+U 1 1 99885386
 P 4100 3700
 F 0 "V3" H 4100 3700 30  0000 L CNN
@@
 $EndComp
 $Comp
+L PARAM_PSPICE PM2
+U 1 1 39760492
+P 8200 2200
+F 0 "PM2" H 8200 2200 30  0001 L CNN
+F 1 "PARAM" H 8200 2280 30  0001 L CNN
+	1    8200 2200
+	1    0    0    -1
+$EndComp
+$Comp
 L SCR2T_PSPICE U5
-U 1 1 99885386
+U 1 1 66516649
 P 6300 3000
 F 0 "U5" H 6300 3000 30  0000 L CNN
@@
 $Comp
 L SCR2T_PSPICE U2
-U 1 1 39760492
+U 1 1 29641421
 P 6300 4100
 F 0 "U2" H 6300 4100 30  0000 L CNN
@@
 $Comp
 L SCR2T_PSPICE U1
-U 1 1 66516649
+U 1 1 45202362
 P 5100 3000
 F 0 "U1" H 5100 3000 30  0000 L CNN
@@
 $Comp
 L SCR2T_PSPICE U3
-U 1 1 29641421
+U 1 1 10490027
 P 5700 3000
 F 0 "U3" H 5700 3000 30  0000 L CNN
@@
 $Comp
 L SCR2T_PSPICE U6
-U 1 1 45202362
+U 1 1 73368690
 P 5100 4100
 F 0 "U6" H 5100 4100 30  0000 L CNN
@@
 $Comp
 L SCR2T_PSPICE U4
-U 1 1 10490027
+U 1 1 32520059
 P 5700 4100
 F 0 "U4" H 5700 4100 30  0000 L CNN
@@
 	0    -1    -1    0
 $EndComp
+$Comp
+L titleblk_PSPICE titleblk
+U 1 1 74897763
+P 9700 7200
+F 0 "titleblk" H 19400 14400 30  0001 L CNN
+F 1 "titleblk" H 19400 14480 30  0001 L CNN
+	1    9700 7200
+	1    0    0    -1
+$EndComp
 Wire Wire Line
