File: ConvertedSchematicFiles/EXP13_11/EXP13_11.sch (KiCad schematic (older format))
At the start: 10 parts, among them U1 CD4016BD

Commit message: Excluded some components. These no longer appear after conversion. When calling shell commands, filenames are in "quotes"
Parts:
- removed V1: VSIN, symbol VSIN_PSPICE
- removed titleblk: titleblk, symbol TITLEBLK_PSPICE
- V1: renamed from PM1; value PARAM -> VSIN; symbol PARAM_PSPICE -> VSIN_PSPICE
Connections:
- net at U1.IN: now also V1.+
Changed lines of the file:
@@
-$EndComp
-$Comp
-L PARAM_PSPICE PM1
-U 1 1 39760492
-P 4000 400
-F 0 "PM1" H 4000 400 30  0000 L CNN
-F 1 "PARAM" H 4000 480 30  0000 L CNN
-	1    4000 400
-	1    0    0    1
 $EndComp
 $Comp
 L VSIN_PSPICE V1
-U 1 1 66516649
+U 1 1 39760492
 P 400 800
 F 0 "V1" H 400 800 30  0000 L CNN
@@
 	1    0    0    1
 $EndComp
-$Comp
-L TITLEBLK_PSPICE titleblk
-U 1 1 29641421
-P 11880 8400
-F 0 "titleblk" H 23760 16800 30  0001 L CNN
-F 1 "titleblk" H 23760 16880 30  0001 L CNN
-	1    11880 8400
-	1    0    0    1
-$EndComp

Commit message: Ports issue fixed. Now annotation for ports is #PWR? function added "itos"
Parts:
- removed +5V: +5V, symbol +5V_PSPICE
- removed EGND (x3): EGND, symbol EGND_PSPICE
Changed lines of the file:
@@
 $EndDescr
 $Comp
-L EGND_PSPICE EGND
+L EGND_PSPICE #PWR1
 U 1 1 14289383
 P 1900 1500
-F 0 "EGND" H 3800 3000 30  0001 L CNN
+F 0 "#PWR1" H 3800 3000 30  0001 L CNN
 F 1 "EGND" H 3800 3080 30  0001 L CNN
 	1    1900 1500
@@
 $EndComp
 $Comp
-L EGND_PSPICE EGND
+L EGND_PSPICE #PWR2
 U 1 1 46930886
 P 2700 1200
-F 0 "EGND" H 5400 2400 30  0001 L CNN
+F 0 "#PWR2" H 5400 2400 30  0001 L CNN
 F 1 "EGND" H 5400 2480 30  0001 L CNN
 	1    2700 1200
@@
 $EndComp
 $Comp
-L +5V_PSPICE +5V
+L +5V_PSPICE #PWR3
 U 1 1 71692777
 P 1900 500
-F 0 "+5V" H 3800 1000 30  0001 L CNN
+F 0 "#PWR3" H 3800 1000 30  0001 L CNN
 F 1 "+5V" H 3800 1080 30  0001 L CNN
 	1    1900 500
@@
 $EndComp
 $Comp
-L EGND_PSPICE EGND
+L EGND_PSPICE #PWR4
 U 1 1 14636915
 P 400 1200
-F 0 "EGND" H 800 2400 30  0001 L CNN
+F 0 "#PWR4" H 800 2400 30  0001 L CNN
 F 1 "EGND" H 800 2480 30  0001 L CNN
 	1    400 1200

Commit message: Added LICENSE.txt
Changed lines of the file:
@@
 $EndDescr
 $Comp
-L EGND_PSPICE #PWR1
+L GND #PWR1
 U 1 1 14289383
 P 1900 1500
@@
 $EndComp
 $Comp
-L EGND_PSPICE #PWR2
+L GND #PWR2
 U 1 1 46930886
 P 2700 1200
@@
 $EndComp
 $Comp
-L +5V_PSPICE #PWR3
+L +5V #PWR3
 U 1 1 71692777
 P 1900 500
@@
 $EndComp
 $Comp
-L EGND_PSPICE #PWR4
+L GND #PWR4
 U 1 1 14636915
 P 400 1200

Commit message: Orientation fix. Library components are now inverted, with +ve y axis going up. In Schematic files, +ve y axis is downwards. This is how the KiCad libraries are. As a result of the above fixed, the converted GND is now oriented correctly.
Parts:
- V1: value VSIN -> SINE
Other:
- moved on the sheet: U1, V1
Changed lines of the file:
@@
 F 1 "EGND" H 3800 3080 30  0001 L CNN
 	1    1900 1500
-	1    0    0    1
+	1    0    0    -1
 $EndComp
 $Comp
@@
 F 1 "EGND" H 5400 2480 30  0001 L CNN
 	1    2700 1200
-	1    0    0    1
+	1    0    0    -1
 $EndComp
 $Comp
@@
 F 1 "+5V" H 3800 1080 30  0001 L CNN
 	1    1900 500
-	1    0    0    1
+	1    0    0    -1
 $EndComp
 $Comp
@@
 F 1 "EGND" H 800 2480 30  0001 L CNN
 	1    400 1200
-	1    0    0    1
+	1    0    0    -1
 $EndComp
 $Comp
@@
 F 1 "10k" H 2700 1170 30  0000 L CNN
 	1    2700 900
-	0    -1    1    0
+	0    1    1    0
 $EndComp
 $Comp
@@
 F 1 "DigStim" H 1300 1180 30  0000 L CNN
 	1    1300 1100
-	1    0    0    1
+	1    0    0    -1
 $EndComp
 $Comp
@@
 F 1 "CD4016BD" H 1600 980 30  0000 L CNN
 	1    1600 900
-	1    0    0    1
+	1    0    0    -1
 $EndComp
 $Comp
@@
 P 400 800
 F 0 "V1" H 400 800 30  0000 L CNN
-F 1 "VSIN" H 400 880 30  0000 L CNN
+F 1 "SINE" H 400 880 30  0000 L CNN
 	1    400 800
-	1    0    0    1
+	1    0    0    -1
 $EndComp
 Wire Wire Line

Commit message: Removed the use of exec, wrote basename function, made integration with eSim easier.
Parts:
- added V1: SINE, symbol VSIN_PSPICE
- added titleblk: titleblk, symbol titleblk_PSPICE
- PM1: renamed from V1; value SINE -> PARAM; symbol VSIN_PSPICE -> PARAM_PSPICE
Changed lines of the file:
@@
-EESchema Schematic File Version 2  date Friday 09 July 1999 05:51:08 PM IST
+EESchema Schematic File Version 2  date
 LIBS:power
 LIBS:device
@@
 LIBS:contrib
 LIBS:valves
-LIBS:ConvertedSchematicFiles/EXP13_11-cache
 EELAYER 25  0
 EELAYER END
@@
 Sheet 1 1
 Title ""
-Date "09 Jul 1999"
+Date ""
 Rev ""
 Comp ""
@@
 $EndComp
 $Comp
+L PARAM_PSPICE PM1
+U 1 1 39760492
+P 4000 400
+F 0 "PM1" H 4000 400 30  0000 L CNN
+F 1 "PARAM" H 4000 480 30  0000 L CNN
+	1    4000 400
+	1    0    0    -1
+$EndComp
+$Comp
 L VSIN_PSPICE V1
-U 1 1 39760492
+U 1 1 66516649
 P 400 800
 F 0 "V1" H 400 800 30  0000 L CNN
@@
 	1    0    0    -1
 $EndComp
+$Comp
+L titleblk_PSPICE titleblk
+U 1 1 29641421
+P 11880 8400
+F 0 "titleblk" H 23760 16800 30  0001 L CNN
+F 1 "titleblk" H 23760 16880 30  0001 L CNN
+	1    11880 8400
+	1    0    0    -1
+$EndComp
