File: ConvertedSchematicFiles/EXP13_8/EXP13_8.sch (KiCad schematic (older format))
At the start: 10 parts, among them Q1 Q2N2222

Commit message: Excluded some components. These no longer appear after conversion. When calling shell commands, filenames are in "quotes"
Parts:
- removed Rb: 100k, symbol R_PSPICE
- removed titleblk: titleblk, symbol TITLEBLK_PSPICE
- Rb: renamed from V1; value VSIN -> 100k; symbol VSIN_PSPICE -> R_PSPICE
- V1: renamed from PM1; value PARAM -> VSIN; symbol PARAM_PSPICE -> VSIN_PSPICE
Connections:
- net at Q1.2: now also Rb.2
- new net: Rb.1, V1.+
Changed lines of the file:
@@
-$EndComp
-$Comp
-L PARAM_PSPICE PM1
-U 1 1 99885386
-P 3700 1000
-F 0 "PM1" H 3700 1000 30  0001 L CNN
-F 1 "PARAM" H 3700 1080 30  0001 L CNN
-	1    3700 1000
-	1    0    0    1
 $EndComp
 $Comp
 L VSIN_PSPICE V1
-U 1 1 39760492
+U 1 1 99885386
 P 1200 1800
 F 0 "V1" H 1200 1800 30  0001 L CNN
@@
 $Comp
 L R_PSPICE Rb
-U 1 1 66516649
+U 1 1 39760492
 P 1600 1800
 F 0 "Rb" H 1600 1800 30  0000 L CNN
@@
 	1    0    0    1
 $EndComp
-$Comp
-L TITLEBLK_PSPICE titleblk
-U 1 1 29641421
-P 9700 7200
-F 0 "titleblk" H 19400 14400 30  0001 L CNN
-F 1 "titleblk" H 19400 14480 30  0001 L CNN
-	1    9700 7200
-	1    0    0    1
-$EndComp

Commit message: Ports issue fixed. Now annotation for ports is #PWR? function added "itos"
Parts:
- removed GND_EARTH (x3): GND_EARTH, symbol GND_EARTH_PSPICE
Changed lines of the file:
@@
 $EndDescr
 $Comp
-L GND_EARTH_PSPICE GND_EARTH
+L GND_EARTH_PSPICE #PWR1
 U 1 1 14289383
 P 2800 400
-F 0 "GND_EARTH" H 5600 800 30  0001 L CNN
+F 0 "#PWR1" H 5600 800 30  0001 L CNN
 F 1 "GND_EARTH" H 5600 880 30  0001 L CNN
 	1    2800 400
@@
 $EndComp
 $Comp
-L GND_EARTH_PSPICE GND_EARTH
+L GND_EARTH_PSPICE #PWR2
 U 1 1 46930886
 P 2400 2100
-F 0 "GND_EARTH" H 4800 4200 30  0001 L CNN
+F 0 "#PWR2" H 4800 4200 30  0001 L CNN
 F 1 "GND_EARTH" H 4800 4280 30  0001 L CNN
 	1    2400 2100
@@
 $EndComp
 $Comp
-L GND_EARTH_PSPICE GND_EARTH
+L GND_EARTH_PSPICE #PWR3
 U 1 1 71692777
 P 1200 2200
-F 0 "GND_EARTH" H 2400 4400 30  0001 L CNN
+F 0 "#PWR3" H 2400 4400 30  0001 L CNN
 F 1 "GND_EARTH" H 2400 4480 30  0001 L CNN
 	1    1200 2200

Commit message: Added LICENSE.txt
Parts:
- V1: value VSIN -> SINE
Changed lines of the file:
@@
 $EndDescr
 $Comp
-L GND_EARTH_PSPICE #PWR1
+L GND #PWR1
 U 1 1 14289383
 P 2800 400
@@
 $EndComp
 $Comp
-L GND_EARTH_PSPICE #PWR2
+L GND #PWR2
 U 1 1 46930886
 P 2400 2100
@@
 $EndComp
 $Comp
-L GND_EARTH_PSPICE #PWR3
+L GND #PWR3
 U 1 1 71692777
 P 1200 2200
@@
 P 1200 1800
 F 0 "V1" H 1200 1800 30  0001 L CNN
-F 1 "VSIN" H 1200 1880 30  0001 L CNN
+F 1 "SINE" H 1200 1880 30  0001 L CNN
 	1    1200 1800
 	1    0    0    1

Commit message: Orientation fix. Library components are now inverted, with +ve y axis going up. In Schematic files, +ve y axis is downwards. This is how the KiCad libraries are. As a result of the above fixed, the converted GND is now oriented correctly.
Changed lines of the file:
@@
 F 1 "GND_EARTH" H 5600 880 30  0001 L CNN
 	1    2800 400
-	1    0    0    1
+	1    0    0    -1
 $EndComp
 $Comp
@@
 F 1 "GND_EARTH" H 4800 4280 30  0001 L CNN
 	1    2400 2100
-	1    0    0    1
+	1    0    0    -1
 $EndComp
 $Comp
@@
 F 1 "GND_EARTH" H 2400 4480 30  0001 L CNN
 	1    1200 2200
-	1    0    0    1
+	1    0    0    -1
 $EndComp
 $Comp
@@
 F 1 "2.2k" H 2400 1150 30  0000 L CNN
 	1    2400 900
-	0    -1    1    0
+	0    1    1    0
 $EndComp
 $Comp
@@
 F 1 "Q2N2222" H 2200 1880 30  0001 L CNN
 	1    2200 1800
-	1    0    0    1
+	1    0    0    -1
 $EndComp
 $Comp
@@
 F 1 "15V" H 2400 690 30  0000 C CNN
 	1    2400 800
-	-1    0    0    -1
+	-1    0    0    1
 $EndComp
 $Comp
@@
 F 1 "SINE" H 1200 1880 30  0001 L CNN
 	1    1200 1800
-	1    0    0    1
+	1    0    0    -1
 $EndComp
 $Comp
@@
 F 1 "100k" H 1600 1950 30  0000 L CNN
 	1    1600 1800
-	1    0    0    1
+	1    0    0    -1
 $EndComp
 Wire Wire Line

Commit message: Removed the use of exec, wrote basename function, made integration with eSim easier.
Parts:
- added Rb: 100k, symbol R_PSPICE
- added titleblk: titleblk, symbol titleblk_PSPICE
- PM1: renamed from V1; value SINE -> PARAM; symbol VSIN_PSPICE -> PARAM_PSPICE
- V1: renamed from Rb; value 100k -> SINE; symbol R_PSPICE -> VSIN_PSPICE
Changed lines of the file:
@@
-EESchema Schematic File Version 2  date Sunday 06 June 1999 10:50:58 AM IST
+EESchema Schematic File Version 2  date
 LIBS:power
 LIBS:device
@@
 LIBS:contrib
 LIBS:valves
-LIBS:ConvertedSchematicFiles/EXP13_8-cache
 EELAYER 25  0
 EELAYER END
@@
 Sheet 1 1
 Title ""
-Date "06 Jun 1999"
+Date ""
 Rev ""
 Comp ""
@@
 $EndComp
 $Comp
+L PARAM_PSPICE PM1
+U 1 1 99885386
+P 3700 1000
+F 0 "PM1" H 3700 1000 30  0001 L CNN
+F 1 "PARAM" H 3700 1080 30  0001 L CNN
+	1    3700 1000
+	1    0    0    -1
+$EndComp
+$Comp
 L VSIN_PSPICE V1
-U 1 1 99885386
+U 1 1 39760492
 P 1200 1800
 F 0 "V1" H 1200 1800 30  0001 L CNN
@@
 $Comp
 L R_PSPICE Rb
-U 1 1 39760492
+U 1 1 66516649
 P 1600 1800
 F 0 "Rb" H 1600 1800 30  0000 L CNN
@@
 	1    0    0    -1
 $EndComp
+$Comp
+L titleblk_PSPICE titleblk
+U 1 1 29641421
+P 9700 7200
+F 0 "titleblk" H 19400 14400 30  0001 L CNN
+F 1 "titleblk" H 19400 14480 30  0001 L CNN
+	1    9700 7200
+	1    0    0    -1
+$EndComp
