File: ConvertedSchematicFiles/EXP14_13/EXP14_13.sch (KiCad schematic (older format))
At the start: 1 part

Commit message: Excluded some components. These no longer appear after conversion. When calling shell commands, filenames are in "quotes"
Parts:
- removed titleblk: titleblk, symbol TITLEBLK_PSPICE
Changed lines of the file:
@@
 Comment4 ""
 $EndDescr
-$Comp
-L TITLEBLK_PSPICE titleblk
-U 1 1 14289383
-P 9700 7200
-F 0 "titleblk" H 19400 14400 30  0001 L CNN
-F 1 "titleblk" H 19400 14480 30  0001 L CNN
-	1    9700 7200
-	1    0    0    1
-$EndComp
 $EndSCHEMATC

Commit message: Removed the use of exec, wrote basename function, made integration with eSim easier.
Parts:
- added titleblk: titleblk, symbol titleblk_PSPICE
Changed lines of the file:
@@
-EESchema Schematic File Version 2  date Sunday 27 June 1999 07:15:56 AM IST
+EESchema Schematic File Version 2  date
 LIBS:power
 LIBS:device
@@
 LIBS:contrib
 LIBS:valves
-LIBS:ConvertedSchematicFiles/EXP14_13-cache
 EELAYER 25  0
 EELAYER END
@@
 Sheet 1 1
 Title ""
-Date "27 Jun 1999"
+Date ""
 Rev ""
 Comp ""
@@
 Comment4 ""
 $EndDescr
+$Comp
+L titleblk_PSPICE titleblk
+U 1 1 14289383
+P 9700 7200
+F 0 "titleblk" H 19400 14400 30  0001 L CNN
+F 1 "titleblk" H 19400 14480 30  0001 L CNN
+	1    9700 7200
+	1    0    0    -1
+$EndComp
 $EndSCHEMATC
