File: ConvertedSchematicFiles/EXP16_13/EXP16_13.sch (KiCad schematic (older format))
At the start: 23 parts, among them U1 SCR2T, U2 SCR2T

Commit message: Excluded some components. These no longer appear after conversion. When calling shell commands, filenames are in "quotes"
Parts:
- removed PM3: PARAM, symbol PARAM_PSPICE
- removed R16: 1meg, symbol R_PSPICE
- removed titleblk: titleblk, symbol TITLEBLK_PSPICE
- removed vdiffMarker (x4): vdiffMarker, symbol VDIFFMARKER_PSPICE
- C1: renamed from R1; value 0.1 -> 16u; symbol R_PSPICE -> C_PSPICE
- R1: renamed from PM2; value PARAM -> 0.1; symbol PARAM_PSPICE -> R_PSPICE
- R15: renamed from TX26; value COUPLED_INDUCTOR -> 100k; symbol COUPLED_INDUCTOR_PSPICE -> R_PSPICE
- R16: renamed from R15; value 100k -> 1meg
- TX25: renamed from C1; value 16u -> COUPLED_INDUCTOR; symbol C_PSPICE -> COUPLED_INDUCTOR_PSPICE
- renumbered TX25 to TX26
Connections:
- net at C1.1: now also R14.2, TX25.1, U1.A; no longer V1.+
- net at C1.2: now also R13.1, R3.2, U2.A; no longer R15.1
- net at R16.2: now also R3.1
- net at TX26.3: no longer R16.1
- net at R15.2: now also R16.1
- new net: R1.1, V1.+
- new net: R1.2, TX26.1
- new net: R15.1, TX25.3
- now unconnected: TX25.2
Other:
- moved on the sheet: R16, TX26
Changed lines of the file:
@@
-$EndComp
-$Comp
-L PARAM_PSPICE PM2
-U 1 1 45202362
-P 6200 3300
-F 0 "PM2" H 6200 3300 30  0000 L CNN
-F 1 "PARAM" H 6200 3380 30  0000 L CNN
-	1    6200 3300
-	1    0    0    1
 $EndComp
 $Comp
 L R_PSPICE R1
-U 1 1 10490027
+U 1 1 45202362
 P 1600 1900
 F 0 "R1" H 1600 1900 30  0000 L CNN
@@
 $Comp
 L C_PSPICE C1
-U 1 1 73368690
+U 1 1 10490027
 P 3500 2400
 F 0 "C1" H 3500 2400 30  0000 L CNN
@@
 $Comp
 L COUPLED_INDUCTOR_PSPICE TX25
-U 1 1 32520059
+U 1 1 73368690
 P 3400 1900
 F 0 "TX25" H 3400 1900 30  0000 L CNN
@@
 $Comp
 L COUPLED_INDUCTOR_PSPICE TX26
-U 1 1 74897763
+U 1 1 32520059
 P 4300 1900
 F 0 "TX26" H 4300 1900 30  0000 L CNN
@@
 $Comp
 L R_PSPICE R15
-U 1 1 87513926
+U 1 1 74897763
 P 4100 1100
 F 0 "R15" H 4100 1100 30  0000 L CNN
@@
 $Comp
 L R_PSPICE R16
-U 1 1 25180540
+U 1 1 87513926
 P 5400 1500
 F 0 "R16" H 5400 1500 30  0000 L CNN
@@
 	0    -1    1    0
 $EndComp
-$Comp
-L PARAM_PSPICE PM3
-U 1 1 20383426
-P 6100 2400
-F 0 "PM3" H 6100 2400 30  0000 L CNN
-F 1 "PARAM" H 6100 2480 30  0000 L CNN
-	1    6100 2400
-	1    0    0    1
-$EndComp
-$Comp
-L TITLEBLK_PSPICE titleblk
-U 1 1 44089172
-P 11880 8400
-F 0 "titleblk" H 23760 16800 30  0001 L CNN
-F 1 "titleblk" H 23760 16880 30  0001 L CNN
-	1    11880 8400
-	1    0    0    1
-$EndComp
-$Comp
-L VDIFFMARKER_PSPICE vdiffMarker
-U 1 1 53455736
-P 4300 2400
-F 0 "vdiffMarker" H 8600 4800 30  0001 L CNN
-F 1 "vdiffMarker" H 8600 4880 30  0001 L CNN
-	1    4300 2400
-	1    0    0    1
-$EndComp
-$Comp
-L VDIFFMARKER_PSPICE vdiffMarker
-U 1 1 45005211
-P 3100 2400
-F 0 "vdiffMarker" H 6200 4800 30  0001 L CNN
-F 1 "vdiffMarker" H 6200 4880 30  0001 L CNN
-	1    3100 2400
-	1    0    0    1
-$EndComp
-$Comp
-L VDIFFMARKER_PSPICE vdiffMarker
-U 1 1 81595368
-P 3400 1500
-F 0 "vdiffMarker" H 6800 3000 30  0001 L CNN
-F 1 "vdiffMarker" H 6800 3080 30  0001 L CNN
-	1    3400 1500
-	1    0    0    1
-$EndComp
-$Comp
-L VDIFFMARKER_PSPICE vdiffMarker
-U 1 1 34702567
-P 4900 1500
-F 0 "vdiffMarker" H 9800 3000 30  0001 L CNN
-F 1 "vdiffMarker" H 9800 3080 30  0001 L CNN
-	1    4900 1500
-	1    0    0    1
-$EndComp
 Wire Wire Line

Commit message: Ports issue fixed. Now annotation for ports is #PWR? function added "itos"
Parts:
- removed EGND: EGND, symbol EGND_PSPICE
Changed lines of the file:
@@
 $EndDescr
 $Comp
-L EGND_PSPICE EGND
+L EGND_PSPICE #PWR1
 U 1 1 14289383
 P 1200 4800
-F 0 "EGND" H 2400 9600 30  0001 L CNN
+F 0 "#PWR1" H 2400 9600 30  0001 L CNN
 F 1 "EGND" H 2400 9680 30  0001 L CNN
 	1    1200 4800

Commit message: Added LICENSE.txt
Changed lines of the file:
@@
 $EndDescr
 $Comp
-L EGND_PSPICE #PWR1
+L GND #PWR1
 U 1 1 14289383
 P 1200 4800

Commit message: Orientation fix. Library components are now inverted, with +ve y axis going up. In Schematic files, +ve y axis is downwards. This is how the KiCad libraries are. As a result of the above fixed, the converted GND is now oriented correctly.
Other:
- moved on the sheet: L1, TX25, TX26, V1
Changed lines of the file:
@@
 F 1 "EGND" H 2400 9680 30  0001 L CNN
 	1    1200 4800
-	1    0    0    1
+	1    0    0    -1
 $EndComp
 $Comp
@@
 F 1 "3mh" H 3700 4350 30  0000 L CNN
 	1    3700 4000
-	0    -1    1    0
+	0    1    1    0
 $EndComp
 $Comp
@@
 F 1 "D1N914" H 2300 3580 30  0000 L CNN
 	1    2300 3500
-	0    1    -1    0
+	0    -1    -1    0
 $EndComp
 $Comp
@@
 F 1 "D1N914" H 5000 3580 30  0000 L CNN
 	1    5000 3500
-	0    1    -1    0
+	0    -1    -1    0
 $EndComp
 $Comp
@@
 F 1 "1" H 4500 2950 30  0000 L CNN
 	1    4500 2800
-	1    0    0    1
+	1    0    0    -1
 $EndComp
 $Comp
@@
 F 1 "0.1" H 4900 2310 30  0000 L CNN
 	1    4900 2000
-	0    -1    1    0
+	0    1    1    0
 $EndComp
 $Comp
@@
 F 1 "SCR2T" H 4300 2980 30  0000 L CNN
 	1    4300 2900
-	0    -1    1    0
+	0    1    1    0
 $EndComp
 $Comp
@@
 F 1 "SCR2T" H 3100 2980 30  0000 L CNN
 	1    3100 2900
-	0    -1    1    0
+	0    1    1    0
 $EndComp
 $Comp
@@
 F 1 "1" H 2500 2950 30  0000 L CNN
 	1    2500 2800
-	1    0    0    1
+	1    0    0    -1
 $EndComp
 $Comp
@@
 F 1 "25v" H 1200 2890 30  0000 C CNN
 	1    1200 3000
-	1    0    0    1
+	1    0    0    -1
 $EndComp
 $Comp
@@
 F 1 "0.1" H 1600 2050 30  0000 L CNN
 	1    1600 1900
-	1    0    0    1
+	1    0    0    -1
 $EndComp
 $Comp
@@
 F 1 "16u" H 3500 2470 30  0000 L CNN
 	1    3500 2400
-	1    0    0    1
+	1    0    0    -1
 $EndComp
 $Comp
@@
 F 1 "COUPLED_INDUCTOR" H 3400 1980 30  0000 L CNN
 	1    3400 1900
-	0    1    -1    0
+	0    -1    -1    0
 $EndComp
 $Comp
@@
 F 1 "COUPLED_INDUCTOR" H 4300 1980 30  0000 L CNN
 	1    4300 1900
-	0    1    -1    0
+	0    -1    -1    0
 $EndComp
 $Comp
@@
 F 1 "100k" H 4100 1250 30  0000 L CNN
 	1    4100 1100
-	1    0    0    1
+	1    0    0    -1
 $EndComp
 $Comp
@@
 F 1 "1meg" H 5400 1850 30  0000 L CNN
 	1    5400 1500
-	0    -1    1    0
+	0    1    1    0
 $EndComp
 Wire Wire Line

Commit message: Removed the use of exec, wrote basename function, made integration with eSim easier.
Parts:
- added PM3: PARAM, symbol PARAM_PSPICE
- added R16: 1meg, symbol R_PSPICE
- added titleblk: titleblk, symbol titleblk_PSPICE
- added vdiffMarker (x4): vdiffMarker, symbol vdiffMarker_PSPICE
- C1: renamed from TX25; value COUPLED_INDUCTOR -> 16u; symbol COUPLED_INDUCTOR_PSPICE -> C_PSPICE
- PM2: renamed from R1; value 0.1 -> PARAM; symbol R_PSPICE -> PARAM_PSPICE
- R1: renamed from C1; value 16u -> 0.1; symbol C_PSPICE -> R_PSPICE
- R15: renamed from R16; value 1meg -> 100k
- TX26: renamed from R15; value 100k -> COUPLED_INDUCTOR; symbol R_PSPICE -> COUPLED_INDUCTOR_PSPICE
- renumbered TX26 to TX25
Other:
- moved on the sheet: R15, TX25
Changed lines of the file:
@@
-EESchema Schematic File Version 2  date Wednesday 08 March 2000 12:23:53 AM IST
+EESchema Schematic File Version 2  date
 LIBS:power
 LIBS:device
@@
 LIBS:contrib
 LIBS:valves
-LIBS:ConvertedSchematicFiles/EXP16_13-cache
 EELAYER 25  0
 EELAYER END
@@
 Sheet 1 1
 Title ""
-Date "08 Mar 2000"
+Date ""
 Rev ""
 Comp ""
@@
 $EndComp
 $Comp
+L PARAM_PSPICE PM2
+U 1 1 45202362
+P 6200 3300
+F 0 "PM2" H 6200 3300 30  0000 L CNN
+F 1 "PARAM" H 6200 3380 30  0000 L CNN
+	1    6200 3300
+	1    0    0    -1
+$EndComp
+$Comp
 L R_PSPICE R1
-U 1 1 45202362
+U 1 1 10490027
 P 1600 1900
 F 0 "R1" H 1600 1900 30  0000 L CNN
@@
 $Comp
 L C_PSPICE C1
-U 1 1 10490027
+U 1 1 73368690
 P 3500 2400
 F 0 "C1" H 3500 2400 30  0000 L CNN
@@
 $Comp
 L COUPLED_INDUCTOR_PSPICE TX25
-U 1 1 73368690
+U 1 1 32520059
 P 3400 1900
 F 0 "TX25" H 3400 1900 30  0000 L CNN
@@
 $Comp
 L COUPLED_INDUCTOR_PSPICE TX26
-U 1 1 32520059
+U 1 1 74897763
 P 4300 1900
 F 0 "TX26" H 4300 1900 30  0000 L CNN
@@
 $Comp
 L R_PSPICE R15
-U 1 1 74897763
+U 1 1 87513926
 P 4100 1100
 F 0 "R15" H 4100 1100 30  0000 L CNN
@@
 $Comp
 L R_PSPICE R16
-U 1 1 87513926
+U 1 1 25180540
 P 5400 1500
 F 0 "R16" H 5400 1500 30  0000 L CNN
@@
 	0    1    1    0
 $EndComp
+$Comp
+L PARAM_PSPICE PM3
+U 1 1 20383426
+P 6100 2400
+F 0 "PM3" H 6100 2400 30  0000 L CNN
+F 1 "PARAM" H 6100 2480 30  0000 L CNN
+	1    6100 2400
+	1    0    0    -1
+$EndComp
+$Comp
+L titleblk_PSPICE titleblk
+U 1 1 44089172
+P 11880 8400
+F 0 "titleblk" H 23760 16800 30  0001 L CNN
+F 1 "titleblk" H 23760 16880 30  0001 L CNN
+	1    11880 8400
+	1    0    0    -1
+$EndComp
+$Comp
+L vdiffMarker_PSPICE vdiffMarker
+U 1 1 53455736
+P 4300 2400
+F 0 "vdiffMarker" H 8600 4800 30  0001 L CNN
+F 1 "vdiffMarker" H 8600 4880 30  0001 L CNN
+	1    4300 2400
+	1    0    0    -1
+$EndComp
+$Comp
+L vdiffMarker_PSPICE vdiffMarker
+U 1 1 45005211
+P 3100 2400
+F 0 "vdiffMarker" H 6200 4800 30  0001 L CNN
+F 1 "vdiffMarker" H 6200 4880 30  0001 L CNN
+	1    3100 2400
+	1    0    0    -1
+$EndComp
+$Comp
+L vdiffMarker_PSPICE vdiffMarker
+U 1 1 81595368
+P 3400 1500
+F 0 "vdiffMarker" H 6800 3000 30  0001 L CNN
+F 1 "vdiffMarker" H 6800 3080 30  0001 L CNN
+	1    3400 1500
+	1    0    0    -1
+$EndComp
+$Comp
+L vdiffMarker_PSPICE vdiffMarker
+U 1 1 34702567
+P 4900 1500
+F 0 "vdiffMarker" H 9800 3000 30  0001 L CNN
+F 1 "vdiffMarker" H 9800 3080 30  0001 L CNN
+	1    4900 1500
+	1    0    0    -1
+$EndComp
 Wire Wire Line
