File: ConvertedSchematicFiles/EXP16_2/EXP16_2.sch (KiCad schematic (older format))
At the start: 19 parts

Commit message: Excluded some components. These no longer appear after conversion. When calling shell commands, filenames are in "quotes"
Parts:
- removed D1: D1N4002, symbol D1N4002_PSPICE
- removed titleblk: titleblk, symbol TITLEBLK_PSPICE
- C1: renamed from RL2; value 100 -> {C_FILT}; symbol R_PSPICE -> C_PSPICE
- D7: renamed from C1; value {C_FILT} -> D1N4002; symbol C_PSPICE -> D1N4002_PSPICE
- L1: renamed from PM1; value PARAM -> 100mH; symbol PARAM_PSPICE -> L_PSPICE
- RL1: renamed from L2; value 100mH -> 100; symbol L_PSPICE -> R_PSPICE
- renumbered D2 to D1, D4 to D2, D8 to D3, D3 to D4, D6 to D5, D7 to D6, D5 to D8, L1 to L2, RL1 to RL2
Other:
- moved on the sheet: D1, D2, D3, D4, D5, D6, D8, L2, RL2
Changed lines of the file:
@@
-$EndComp
-$Comp
-L PARAM_PSPICE PM1
-U 1 1 77747793
-P 8600 1400
-F 0 "PM1" H 8600 1400 30  0000 L CNN
-F 1 "PARAM" H 8600 1480 30  0000 L CNN
-	1    8600 1400
-	1    0    0    1
 $EndComp
 $Comp
 L L_PSPICE L1
-U 1 1 74238335
+U 1 1 77747793
 P 6100 900
 F 0 "L1" H 6100 900 30  0000 L CNN
@@
 $Comp
 L L_PSPICE L2
-U 1 1 99885386
+U 1 1 74238335
 P 6900 3000
 F 0 "L2" H 6900 3000 30  0000 L CNN
@@
 $Comp
 L R_PSPICE RL1
-U 1 1 39760492
+U 1 1 99885386
 P 7700 1400
 F 0 "RL1" H 7700 1400 30  0000 L CNN
@@
 $Comp
 L R_PSPICE RL2
-U 1 1 66516649
+U 1 1 39760492
 P 8200 3600
 F 0 "RL2" H 8200 3600 30  0000 L CNN
@@
 $Comp
 L C_PSPICE C1
-U 1 1 29641421
+U 1 1 66516649
 P 7100 1500
 F 0 "C1" H 7100 1500 30  0000 L CNN
@@
 $Comp
 L D1N4002_PSPICE D7
-U 1 1 45202362
+U 1 1 29641421
 P 5100 4300
 F 0 "D7" H 5100 4300 30  0000 L CNN
@@
 $Comp
 L D1N4002_PSPICE D6
-U 1 1 10490027
+U 1 1 45202362
 P 5800 4300
 F 0 "D6" H 5800 4300 30  0000 L CNN
@@
 $Comp
 L D1N4002_PSPICE D5
-U 1 1 73368690
+U 1 1 10490027
 P 5800 3500
 F 0 "D5" H 5800 3500 30  0000 L CNN
@@
 $Comp
 L D1N4002_PSPICE D8
-U 1 1 32520059
+U 1 1 73368690
 P 5100 3500
 F 0 "D8" H 5100 3500 30  0000 L CNN
@@
 $Comp
 L D1N4002_PSPICE D3
-U 1 1 74897763
+U 1 1 32520059
 P 5100 2200
 F 0 "D3" H 5100 2200 30  0000 L CNN
@@
 $Comp
 L D1N4002_PSPICE D4
-U 1 1 87513926
+U 1 1 74897763
 P 5800 2200
 F 0 "D4" H 5800 2200 30  0000 L CNN
@@
 $Comp
 L D1N4002_PSPICE D2
-U 1 1 25180540
+U 1 1 87513926
 P 5800 1400
 F 0 "D2" H 5800 1400 30  0000 L CNN
@@
 $Comp
 L D1N4002_PSPICE D1
-U 1 1 20383426
+U 1 1 25180540
 P 5100 1400
 F 0 "D1" H 5100 1400 30  0000 L CNN
@@
 	0    1    -1    0
 $EndComp
-$Comp
-L TITLEBLK_PSPICE titleblk
-U 1 1 44089172
-P 11880 8400
-F 0 "titleblk" H 23760 16800 30  0001 L CNN
-F 1 "titleblk" H 23760 16880 30  0001 L CNN
-	1    11880 8400
-	1    0    0    1
-$EndComp
 Wire Wire Line

Commit message: Ports issue fixed. Now annotation for ports is #PWR? function added "itos"
Parts:
- removed EGND (x2): EGND, symbol EGND_PSPICE
Connections:
- net labels added: EGND
Changed lines of the file:
@@
 $EndDescr
 $Comp
-L EGND_PSPICE EGND
+L EGND_PSPICE #PWR1
 U 1 1 14289383
 P 5800 4500
-F 0 "EGND" H 11600 9000 30  0001 L CNN
+F 0 "#PWR1" H 11600 9000 30  0001 L CNN
 F 1 "EGND" H 11600 9080 30  0001 L CNN
 	1    5800 4500
@@
 $EndComp
 $Comp
-L EGND_PSPICE EGND
+L EGND_PSPICE #PWR2
 U 1 1 46930886
 P 5800 2400
-F 0 "EGND" H 11600 4800 30  0001 L CNN
+F 0 "#PWR2" H 11600 4800 30  0001 L CNN
 F 1 "EGND" H 11600 4880 30  0001 L CNN
 	1    5800 2400

Commit message: Added LICENSE.txt
Changed lines of the file:
@@
 $EndDescr
 $Comp
-L EGND_PSPICE #PWR1
+L GND #PWR1
 U 1 1 14289383
 P 5800 4500
@@
 $EndComp
 $Comp
-L EGND_PSPICE #PWR2
+L GND #PWR2
 U 1 1 46930886
 P 5800 2400

Commit message: Orientation fix. Library components are now inverted, with +ve y axis going up. In Schematic files, +ve y axis is downwards. This is how the KiCad libraries are. As a result of the above fixed, the converted GND is now oriented correctly.
Parts:
- V1, V2: value VSIN -> SINE
Other:
- moved on the sheet: L1, L2, V1, V2
Changed lines of the file:
@@
 F 1 "EGND" H 11600 9080 30  0001 L CNN
 	1    5800 4500
-	1    0    0    1
+	1    0    0    -1
 $EndComp
 $Comp
@@
 F 1 "EGND" H 11600 4880 30  0001 L CNN
 	1    5800 2400
-	1    0    0    1
+	1    0    0    -1
 $EndComp
 $Comp
@@
 P 4000 1500
 F 0 "V1" H 4000 1500 30  0000 L CNN
-F 1 "VSIN" H 4000 1580 30  0000 L CNN
+F 1 "SINE" H 4000 1580 30  0000 L CNN
 	1    4000 1500
-	1    0    0    1
+	1    0    0    -1
 $EndComp
 $Comp
@@
 P 4000 3600
 F 0 "V2" H 4000 3600 30  0000 L CNN
-F 1 "VSIN" H 4000 3680 30  0000 L CNN
+F 1 "SINE" H 4000 3680 30  0000 L CNN
 	1    4000 3600
-	1    0    0    1
+	1    0    0    -1
 $EndComp
 $Comp
@@
 F 1 "100mH" H 6100 1050 30  0000 L CNN
 	1    6100 900
-	1    0    0    1
+	1    0    0    -1
 $EndComp
 $Comp
@@
 F 1 "100mH" H 6900 3150 30  0000 L CNN
 	1    6900 3000
-	1    0    0    1
+	1    0    0    -1
 $EndComp
 $Comp
@@
 F 1 "100" H 7700 1670 30  0000 L CNN
 	1    7700 1400
-	0    -1    1    0
+	0    1    1    0
 $EndComp
 $Comp
@@
 F 1 "100" H 8200 3870 30  0000 L CNN
 	1    8200 3600
-	0    -1    1    0
+	0    1    1    0
 $EndComp
 $Comp
@@
 F 1 "{C_FILT}" H 7100 1810 30  0000 L CNN
 	1    7100 1500
-	0    -1    1    0
+	0    1    1    0
 $EndComp
 $Comp
@@
 F 1 "D1N4002" H 5100 4380 30  0000 L CNN
 	1    5100 4300
-	0    1    -1    0
+	0    -1    -1    0
 $EndComp
 $Comp
@@
 F 1 "D1N4002" H 5800 4380 30  0000 L CNN
 	1    5800 4300
-	0    1    -1    0
+	0    -1    -1    0
 $EndComp
 $Comp
@@
 F 1 "D1N4002" H 5800 3580 30  0000 L CNN
 	1    5800 3500
-	0    1    -1    0
+	0    -1    -1    0
 $EndComp
 $Comp
@@
 F 1 "D1N4002" H 5100 3580 30  0000 L CNN
 	1    5100 3500
-	0    1    -1    0
+	0    -1    -1    0
 $EndComp
 $Comp
@@
 F 1 "D1N4002" H 5100 2280 30  0000 L CNN
 	1    5100 2200
-	0    1    -1    0
+	0    -1    -1    0
 $EndComp
 $Comp
@@
 F 1 "D1N4002" H 5800 2280 30  0000 L CNN
 	1    5800 2200
-	0    1    -1    0
+	0    -1    -1    0
 $EndComp
 $Comp
@@
 F 1 "D1N4002" H 5800 1480 30  0000 L CNN
 	1    5800 1400
-	0    1    -1    0
+	0    -1    -1    0
 $EndComp
 $Comp
@@
 F 1 "D1N4002" H 5100 1480 30  0000 L CNN
 	1    5100 1400
-	0    1    -1    0
+	0    -1    -1    0
 $EndComp
 Wire Wire Line

Commit message: Removed the use of exec, wrote basename function, made integration with eSim easier.
Parts:
- added D1: D1N4002, symbol D1N4002_PSPICE
- added titleblk: titleblk, symbol titleblk_PSPICE
- C1: renamed from D7; value D1N4002 -> {C_FILT}; symbol D1N4002_PSPICE -> C_PSPICE
- L2: renamed from RL1; value 100 -> 100mH; symbol R_PSPICE -> L_PSPICE
- PM1: renamed from L1; value 100mH -> PARAM; symbol L_PSPICE -> PARAM_PSPICE
- RL2: renamed from C1; value {C_FILT} -> 100; symbol C_PSPICE -> R_PSPICE
- renumbered D1 to D2, D4 to D3, D2 to D4, D8 to D5, D5 to D6, D6 to D7, D3 to D8, L2 to L1, RL2 to RL1
Other:
- moved on the sheet: D2, D3, D4, D5, D6, D7, D8, L1, RL1
Changed lines of the file:
@@
-EESchema Schematic File Version 2  date Saturday 26 June 1999 09:01:58 AM IST
+EESchema Schematic File Version 2  date
 LIBS:power
 LIBS:device
@@
 LIBS:contrib
 LIBS:valves
-LIBS:ConvertedSchematicFiles/EXP16_2-cache
 EELAYER 25  0
 EELAYER END
@@
 Sheet 1 1
 Title ""
-Date "26 Jun 1999"
+Date ""
 Rev ""
 Comp ""
@@
 $EndComp
 $Comp
+L PARAM_PSPICE PM1
+U 1 1 77747793
+P 8600 1400
+F 0 "PM1" H 8600 1400 30  0000 L CNN
+F 1 "PARAM" H 8600 1480 30  0000 L CNN
+	1    8600 1400
+	1    0    0    -1
+$EndComp
+$Comp
 L L_PSPICE L1
-U 1 1 77747793
+U 1 1 74238335
 P 6100 900
 F 0 "L1" H 6100 900 30  0000 L CNN
@@
 $Comp
 L L_PSPICE L2
-U 1 1 74238335
+U 1 1 99885386
 P 6900 3000
 F 0 "L2" H 6900 3000 30  0000 L CNN
@@
 $Comp
 L R_PSPICE RL1
-U 1 1 99885386
+U 1 1 39760492
 P 7700 1400
 F 0 "RL1" H 7700 1400 30  0000 L CNN
@@
 $Comp
 L R_PSPICE RL2
-U 1 1 39760492
+U 1 1 66516649
 P 8200 3600
 F 0 "RL2" H 8200 3600 30  0000 L CNN
@@
 $Comp
 L C_PSPICE C1
-U 1 1 66516649
+U 1 1 29641421
 P 7100 1500
 F 0 "C1" H 7100 1500 30  0000 L CNN
@@
 $Comp
 L D1N4002_PSPICE D7
-U 1 1 29641421
+U 1 1 45202362
 P 5100 4300
 F 0 "D7" H 5100 4300 30  0000 L CNN
@@
 $Comp
 L D1N4002_PSPICE D6
-U 1 1 45202362
+U 1 1 10490027
 P 5800 4300
 F 0 "D6" H 5800 4300 30  0000 L CNN
@@
 $Comp
 L D1N4002_PSPICE D5
-U 1 1 10490027
+U 1 1 73368690
 P 5800 3500
 F 0 "D5" H 5800 3500 30  0000 L CNN
@@
 $Comp
 L D1N4002_PSPICE D8
-U 1 1 73368690
+U 1 1 32520059
 P 5100 3500
 F 0 "D8" H 5100 3500 30  0000 L CNN
@@
 $Comp
 L D1N4002_PSPICE D3
-U 1 1 32520059
+U 1 1 74897763
 P 5100 2200
 F 0 "D3" H 5100 2200 30  0000 L CNN
@@
 $Comp
 L D1N4002_PSPICE D4
-U 1 1 74897763
+U 1 1 87513926
 P 5800 2200
 F 0 "D4" H 5800 2200 30  0000 L CNN
@@
 $Comp
 L D1N4002_PSPICE D2
-U 1 1 87513926
+U 1 1 25180540
 P 5800 1400
 F 0 "D2" H 5800 1400 30  0000 L CNN
@@
 $Comp
 L D1N4002_PSPICE D1
-U 1 1 25180540
+U 1 1 20383426
 P 5100 1400
 F 0 "D1" H 5100 1400 30  0000 L CNN
@@
 	0    -1    -1    0
 $EndComp
+$Comp
+L titleblk_PSPICE titleblk
+U 1 1 44089172
+P 11880 8400
+F 0 "titleblk" H 23760 16800 30  0001 L CNN
+F 1 "titleblk" H 23760 16880 30  0001 L CNN
+	1    11880 8400
+	1    0    0    -1
+$EndComp
 Wire Wire Line
