File: ConvertedSchematicFiles/EXP18_13/EXP18_13.sch (KiCad schematic (older format))
At the start: 11 parts, among them U1 SCR2T, U2 SCR2T

Commit message: Excluded some components. These no longer appear after conversion. When calling shell commands, filenames are in "quotes"
Parts:
- removed PM1: PARAM, symbol PARAM_PSPICE
- removed U2: SCR2T, symbol SCR2T_PSPICE
- removed nodeMarker: nodeMarker, symbol NODEMARKER_PSPICE
- removed titleblk: titleblk, symbol TITLEBLK_PSPICE
- U1: renamed from V1; value 25v -> SCR2T; symbol VDC_PSPICE -> SCR2T_PSPICE
- V1: renamed from PM2; value PARAM -> 25v; symbol PARAM_PSPICE -> VDC_PSPICE
- renumbered U1 to U2
Connections:
- net at EGND.EGND, R1.2: now also U2.K
- net at TX1.1: now also U1.K; no longer U2.K
- net at U2.A: no longer U1.+
- new net: U1.A, V1.+
Other:
- moved on the sheet: U2
Changed lines of the file:
@@
-$EndComp
-$Comp
-L PARAM_PSPICE PM2
-U 1 1 77747793
-P 4900 1600
-F 0 "PM2" H 4900 1600 30  0000 L CNN
-F 1 "PARAM" H 4900 1680 30  0000 L CNN
-	1    4900 1600
-	1    0    0    1
 $EndComp
 $Comp
 L VDC_PSPICE V1
-U 1 1 74238335
+U 1 1 77747793
 P 1600 1200
 F 0 "V1" H 1600 1200 30  0000 L CNN
@@
 $Comp
 L SCR2T_PSPICE U1
-U 1 1 99885386
+U 1 1 74238335
 P 2300 500
 F 0 "U1" H 2300 500 30  0000 L CNN
@@
 $Comp
 L SCR2T_PSPICE U2
-U 1 1 39760492
+U 1 1 99885386
 P 3600 1500
 F 0 "U2" H 3600 1500 30  0000 L CNN
@@
 	0    -1    1    0
 $EndComp
-$Comp
-L PARAM_PSPICE PM1
-U 1 1 66516649
-P 4900 800
-F 0 "PM1" H 4900 800 30  0000 L CNN
-F 1 "PARAM" H 4900 880 30  0000 L CNN
-	1    4900 800
-	1    0    0    1
-$EndComp
-$Comp
-L TITLEBLK_PSPICE titleblk
-U 1 1 29641421
-P 9700 7200
-F 0 "titleblk" H 19400 14400 30  0001 L CNN
-F 1 "titleblk" H 19400 14480 30  0001 L CNN
-	1    9700 7200
-	1    0    0    1
-$EndComp
-$Comp
-L NODEMARKER_PSPICE nodeMarker
-U 1 1 45202362
-P 2400 1400
-F 0 "nodeMarker" H 4800 2800 30  0001 L CNN
-F 1 "nodeMarker" H 4800 2880 30  0001 L CNN
-	1    2400 1400
-	1    0    0    1
-$EndComp
 Wire Wire Line

Commit message: Ports issue fixed. Now annotation for ports is #PWR? function added "itos"
Parts:
- removed EGND: EGND, symbol EGND_PSPICE
Changed lines of the file:
@@
 $EndDescr
 $Comp
-L EGND_PSPICE EGND
+L EGND_PSPICE #PWR1
 U 1 1 14289383
 P 3600 2400
-F 0 "EGND" H 7200 4800 30  0001 L CNN
+F 0 "#PWR1" H 7200 4800 30  0001 L CNN
 F 1 "EGND" H 7200 4880 30  0001 L CNN
 	1    3600 2400

Commit message: Added LICENSE.txt
Changed lines of the file:
@@
 $EndDescr
 $Comp
-L EGND_PSPICE #PWR1
+L GND #PWR1
 U 1 1 14289383
 P 3600 2400

Commit message: Orientation fix. Library components are now inverted, with +ve y axis going up. In Schematic files, +ve y axis is downwards. This is how the KiCad libraries are. As a result of the above fixed, the converted GND is now oriented correctly.
Other:
- moved on the sheet: TX1, V1
Changed lines of the file:
@@
 F 1 "EGND" H 7200 4880 30  0001 L CNN
 	1    3600 2400
-	1    0    0    1
+	1    0    0    -1
 $EndComp
 $Comp
@@
 F 1 "5" H 2400 1750 30  0000 L CNN
 	1    2400 1600
-	0    -1    1    0
+	0    1    1    0
 $EndComp
 $Comp
@@
 F 1 "4u" H 2700 1250 30  0000 L CNN
 	1    2700 1100
-	1    0    0    1
+	1    0    0    -1
 $EndComp
 $Comp
@@
 F 1 "XFRM_LINEAR" H 3200 580 30  0000 L CNN
 	1    3200 500
-	1    0    0    1
+	1    0    0    -1
 $EndComp
 $Comp
@@
 F 1 "25v" H 1600 1090 30  0000 C CNN
 	1    1600 1200
-	1    0    0    1
+	1    0    0    -1
 $EndComp
 $Comp
@@
 F 1 "SCR2T" H 2300 580 30  0000 L CNN
 	1    2300 500
-	1    0    0    1
+	1    0    0    -1
 $EndComp
 $Comp
@@
 F 1 "SCR2T" H 3600 1580 30  0000 L CNN
 	1    3600 1500
-	0    -1    1    0
+	0    1    1    0
 $EndComp
 Wire Wire Line

Commit message: Removed the use of exec, wrote basename function, made integration with eSim easier.
Parts:
- added PM1: PARAM, symbol PARAM_PSPICE
- added U2: SCR2T, symbol SCR2T_PSPICE
- added nodeMarker: nodeMarker, symbol nodeMarker_PSPICE
- added titleblk: titleblk, symbol titleblk_PSPICE
- PM2: renamed from V1; value 25v -> PARAM; symbol VDC_PSPICE -> PARAM_PSPICE
- V1: renamed from U1; value SCR2T -> 25v; symbol SCR2T_PSPICE -> VDC_PSPICE
- renumbered U2 to U1
Other:
- moved on the sheet: U1
Changed lines of the file:
@@
-EESchema Schematic File Version 2  date Monday 16 August 1999 06:53:18 PM IST
+EESchema Schematic File Version 2  date
 LIBS:power
 LIBS:device
@@
 LIBS:contrib
 LIBS:valves
-LIBS:ConvertedSchematicFiles/EXP18_13-cache
 EELAYER 25  0
 EELAYER END
@@
 Sheet 1 1
 Title ""
-Date "16 Aug 1999"
+Date ""
 Rev ""
 Comp ""
@@
 $EndComp
 $Comp
+L PARAM_PSPICE PM2
+U 1 1 77747793
+P 4900 1600
+F 0 "PM2" H 4900 1600 30  0000 L CNN
+F 1 "PARAM" H 4900 1680 30  0000 L CNN
+	1    4900 1600
+	1    0    0    -1
+$EndComp
+$Comp
 L VDC_PSPICE V1
-U 1 1 77747793
+U 1 1 74238335
 P 1600 1200
 F 0 "V1" H 1600 1200 30  0000 L CNN
@@
 $Comp
 L SCR2T_PSPICE U1
-U 1 1 74238335
+U 1 1 99885386
 P 2300 500
 F 0 "U1" H 2300 500 30  0000 L CNN
@@
 $Comp
 L SCR2T_PSPICE U2
-U 1 1 99885386
+U 1 1 39760492
 P 3600 1500
 F 0 "U2" H 3600 1500 30  0000 L CNN
@@
 	0    1    1    0
 $EndComp
+$Comp
+L PARAM_PSPICE PM1
+U 1 1 66516649
+P 4900 800
+F 0 "PM1" H 4900 800 30  0000 L CNN
+F 1 "PARAM" H 4900 880 30  0000 L CNN
+	1    4900 800
+	1    0    0    -1
+$EndComp
+$Comp
+L titleblk_PSPICE titleblk
+U 1 1 29641421
+P 9700 7200
+F 0 "titleblk" H 19400 14400 30  0001 L CNN
+F 1 "titleblk" H 19400 14480 30  0001 L CNN
+	1    9700 7200
+	1    0    0    -1
+$EndComp
+$Comp
+L nodeMarker_PSPICE nodeMarker
+U 1 1 45202362
+P 2400 1400
+F 0 "nodeMarker" H 4800 2800 30  0001 L CNN
+F 1 "nodeMarker" H 4800 2880 30  0001 L CNN
+	1    2400 1400
+	1    0    0    -1
+$EndComp
 Wire Wire Line
