File: ConvertedSchematicFiles/EXP1_8/EXP1_8.sch (KiCad schematic (older format))
At the start: 6 parts

Commit message: Excluded some components. These no longer appear after conversion. When calling shell commands, filenames are in "quotes"
Parts:
- removed R1: 1.6k, symbol R_PSPICE
- removed titleblk: titleblk, symbol TITLEBLK_PSPICE
- C1: renamed from PM1; value PARAM -> {CAP}; symbol PARAM_PSPICE -> C_PSPICE
- R1: renamed from V3; value VAC -> 1.6k; symbol VAC_PSPICE -> R_PSPICE
- V3: renamed from C1; value {CAP} -> VAC; symbol C_PSPICE -> VAC_PSPICE
Connections:
- net at EGND.EGND: now also C1.2; no longer V3.2
- new net: R1.1, V3.+
- new net: C1.1, R1.2
Changed lines of the file:
@@
-$EndComp
-$Comp
-L PARAM_PSPICE PM1
-U 1 1 46930886
-P 3000 600
-F 0 "PM1" H 3000 600 30  0000 L CNN
-F 1 "PARAM" H 3000 680 30  0000 L CNN
-	1    3000 600
-	1    0    0    1
 $EndComp
 $Comp
 L C_PSPICE C1
-U 1 1 71692777
+U 1 1 46930886
 P 1800 700
 F 0 "C1" H 1800 700 30  0000 L CNN
@@
 $Comp
 L VAC_PSPICE V3
-U 1 1 14636915
+U 1 1 71692777
 P 800 700
 F 0 "V3" H 800 700 30  0000 L CNN
@@
 $Comp
 L R_PSPICE R1
-U 1 1 77747793
+U 1 1 14636915
 P 1100 600
 F 0 "R1" H 1100 600 30  0000 L CNN
@@
 	1    0    0    1
 $EndComp
-$Comp
-L TITLEBLK_PSPICE titleblk
-U 1 1 74238335
-P 9700 7200
-F 0 "titleblk" H 19400 14400 30  0001 L CNN
-F 1 "titleblk" H 19400 14480 30  0001 L CNN
-	1    9700 7200
-	1    0    0    1
-$EndComp

Commit message: Ports issue fixed. Now annotation for ports is #PWR? function added "itos"
Parts:
- removed EGND: EGND, symbol EGND_PSPICE
Changed lines of the file:
@@
 $EndDescr
 $Comp
-L EGND_PSPICE EGND
+L EGND_PSPICE #PWR1
 U 1 1 14289383
 P 800 1100
-F 0 "EGND" H 1600 2200 30  0001 L CNN
+F 0 "#PWR1" H 1600 2200 30  0001 L CNN
 F 1 "EGND" H 1600 2280 30  0001 L CNN
 	1    800 1100

Commit message: Added LICENSE.txt
Parts:
- V3: value VAC -> AC
Changed lines of the file:
@@
 $EndDescr
 $Comp
-L EGND_PSPICE #PWR1
+L GND #PWR1
 U 1 1 14289383
 P 800 1100
@@
 P 800 700
 F 0 "V3" H 800 700 30  0000 L CNN
-F 1 "VAC" H 800 780 30  0000 L CNN
+F 1 "AC" H 800 780 30  0000 L CNN
 	1    800 700
 	1    0    0    1

Commit message: Orientation fix. Library components are now inverted, with +ve y axis going up. In Schematic files, +ve y axis is downwards. This is how the KiCad libraries are. As a result of the above fixed, the converted GND is now oriented correctly.
Other:
- moved on the sheet: V3
Changed lines of the file:
@@
 F 1 "EGND" H 1600 2280 30  0001 L CNN
 	1    800 1100
-	1    0    0    1
+	1    0    0    -1
 $EndComp
 $Comp
@@
 F 1 "{CAP}" H 1800 1010 30  0000 L CNN
 	1    1800 700
-	0    -1    1    0
+	0    1    1    0
 $EndComp
 $Comp
@@
 F 1 "AC" H 800 780 30  0000 L CNN
 	1    800 700
-	1    0    0    1
+	1    0    0    -1
 $EndComp
 $Comp
@@
 F 1 "1.6k" H 1100 710 30  0000 L CNN
 	1    1100 600
-	1    0    0    1
+	1    0    0    -1
 $EndComp
 Wire Wire Line

Commit message: Removed the use of exec, wrote basename function, made integration with eSim easier.
Parts:
- added R1: 1.6k, symbol R_PSPICE
- added titleblk: titleblk, symbol titleblk_PSPICE
- C1: renamed from V3; value AC -> {CAP}; symbol VAC_PSPICE -> C_PSPICE
- PM1: renamed from C1; value {CAP} -> PARAM; symbol C_PSPICE -> PARAM_PSPICE
- V3: renamed from R1; value 1.6k -> AC; symbol R_PSPICE -> VAC_PSPICE
Changed lines of the file:
@@
-EESchema Schematic File Version 2  date Sunday 02 January 2000 09:14:23 AM IST
+EESchema Schematic File Version 2  date
 LIBS:power
 LIBS:device
@@
 LIBS:contrib
 LIBS:valves
-LIBS:ConvertedSchematicFiles/EXP1_8-cache
 EELAYER 25  0
 EELAYER END
@@
 Sheet 1 1
 Title ""
-Date "02 Jan 2000"
+Date ""
 Rev ""
 Comp ""
@@
 $EndComp
 $Comp
+L PARAM_PSPICE PM1
+U 1 1 46930886
+P 3000 600
+F 0 "PM1" H 3000 600 30  0000 L CNN
+F 1 "PARAM" H 3000 680 30  0000 L CNN
+	1    3000 600
+	1    0    0    -1
+$EndComp
+$Comp
 L C_PSPICE C1
-U 1 1 46930886
+U 1 1 71692777
 P 1800 700
 F 0 "C1" H 1800 700 30  0000 L CNN
@@
 $Comp
 L VAC_PSPICE V3
-U 1 1 71692777
+U 1 1 14636915
 P 800 700
 F 0 "V3" H 800 700 30  0000 L CNN
@@
 $Comp
 L R_PSPICE R1
-U 1 1 14636915
+U 1 1 77747793
 P 1100 600
 F 0 "R1" H 1100 600 30  0000 L CNN
@@
 	1    0    0    -1
 $EndComp
+$Comp
+L titleblk_PSPICE titleblk
+U 1 1 74238335
+P 9700 7200
+F 0 "titleblk" H 19400 14400 30  0001 L CNN
+F 1 "titleblk" H 19400 14480 30  0001 L CNN
+	1    9700 7200
+	1    0    0    -1
+$EndComp
