File: ConvertedSchematicFiles/EXP2_10/EXP2_10.sch (KiCad schematic (older format))
At the start: 24 parts, among them U1 LM7815C, U2 LM7915C

Commit message: Excluded some components. These no longer appear after conversion. When calling shell commands, filenames are in "quotes"
Parts:
- removed C1: 1000uF, symbol C_PSPICE
- removed titleblk: titleblk, symbol TITLEBLK_PSPICE
- C1: renamed from U2; value LM7915C -> 1000uF; symbol LM7915C_PSPICE -> C_PSPICE
- C2: renamed from C4; value 1000uF -> 100uF
- C3: renamed from RL1; value 50 -> 100uF; symbol R_PSPICE -> C_PSPICE
- C4: renamed from PM2; value PARAM -> 1000uF; symbol PARAM_PSPICE -> C_PSPICE
- RL1: renamed from C2; value 100uF -> 50; symbol C_PSPICE -> R_PSPICE
- RL2: renamed from C3; value 100uF -> 50; symbol C_PSPICE -> R_PSPICE
- U1: renamed from RL2; value 50 -> LM7815C; symbol R_PSPICE -> LM7815C_PSPICE
- U2: renamed from U1; value LM7815C -> LM7915C; symbol LM7815C_PSPICE -> LM7915C_PSPICE
Connections:
- net at D1.2, D2.2: now also C1.1, U1.INPUT; no longer U2.INPUT
- net at C3.1, U2.OUTPUT: now also RL2.2; no longer RL1.1
- net at RL1.2: now also EGND.EGND, RL2.1; no longer EGND.EGND
- net at D3.1, D4.1: now also C4.1, U2.INPUT; no longer C1.INPUT, C2.1
- net at EGND.EGND: now also C1.2
- net at EGND.EGND: now also C3.2; no longer RL2.2
- net at C2.2: now also EGND.EGND; no longer EGND.EGND
- new net: C2.1, RL1.1, U1.OUTPUT
- new net: C4.2, EGND.EGND
Other:
- moved on the sheet: C2, U2
Changed lines of the file:
@@
-$EndComp
-$Comp
-L PARAM_PSPICE PM2
-U 1 1 74897763
-P 5700 500
-F 0 "PM2" H 5700 500 30  0000 L CNN
-F 1 "PARAM" H 5700 580 30  0000 L CNN
-	1    5700 500
-	1    0    0    1
 $EndComp
 $Comp
 L C_PSPICE C4
-U 1 1 87513926
+U 1 1 74897763
 P 3200 2700
 F 0 "C4" H 3200 2700 30  0000 L CNN
@@
 $Comp
 L C_PSPICE C2
-U 1 1 25180540
+U 1 1 87513926
 P 4900 1200
 F 0 "C2" H 4900 1200 30  0000 L CNN
@@
 $Comp
 L R_PSPICE RL1
-U 1 1 20383426
+U 1 1 25180540
 P 5600 2000
 F 0 "RL1" H 5600 2000 30  0000 L CNN
@@
 $Comp
 L C_PSPICE C3
-U 1 1 44089172
+U 1 1 20383426
 P 5000 2600
 F 0 "C3" H 5000 2600 30  0000 L CNN
@@
 $Comp
 L R_PSPICE RL2
-U 1 1 53455736
+U 1 1 44089172
 P 5600 2500
 F 0 "RL2" H 5600 2500 30  0000 L CNN
@@
 $Comp
 L LM7815C_PSPICE U1
-U 1 1 45005211
+U 1 1 53455736
 P 3200 1100
 F 0 "U1" H 3200 1100 30  0000 L CNN
@@
 $Comp
 L LM7915C_PSPICE U2
-U 1 1 81595368
+U 1 1 45005211
 P 3300 2500
 F 0 "U2" H 3300 2500 30  0000 L CNN
@@
 $Comp
 L C_PSPICE C1
-U 1 1 34702567
+U 1 1 81595368
 P 3100 1200
 F 0 "C1" H 3100 1200 30  0000 L CNN
@@
 	0    -1    1    0
 $EndComp
-$Comp
-L TITLEBLK_PSPICE titleblk
-U 1 1 26956429
-P 9700 7200
-F 0 "titleblk" H 19400 14400 30  0001 L CNN
-F 1 "titleblk" H 19400 14480 30  0001 L CNN
-	1    9700 7200
-	1    0    0    1
-$EndComp
 Wire Wire Line

Commit message: Ports issue fixed. Now annotation for ports is #PWR? function added "itos"
Parts:
- removed EGND (x8): EGND, symbol EGND_PSPICE
Changed lines of the file:
@@
 $EndDescr
 $Comp
-L EGND_PSPICE EGND
+L EGND_PSPICE #PWR1
 U 1 1 14289383
 P 5800 2400
-F 0 "EGND" H 11600 4800 30  0001 L CNN
+F 0 "#PWR1" H 11600 4800 30  0001 L CNN
 F 1 "EGND" H 11600 4880 30  0001 L CNN
 	1    5800 2400
@@
 $EndComp
 $Comp
-L EGND_PSPICE EGND
+L EGND_PSPICE #PWR2
 U 1 1 46930886
 P 500 1700
-F 0 "EGND" H 1000 3400 30  0001 L CNN
+F 0 "#PWR2" H 1000 3400 30  0001 L CNN
 F 1 "EGND" H 1000 3480 30  0001 L CNN
 	1    500 1700
@@
 $EndComp
 $Comp
-L EGND_PSPICE EGND
+L EGND_PSPICE #PWR3
 U 1 1 71692777
 P 4000 2800
-F 0 "EGND" H 8000 5600 30  0001 L CNN
+F 0 "#PWR3" H 8000 5600 30  0001 L CNN
 F 1 "EGND" H 8000 5680 30  0001 L CNN
 	1    4000 2800
@@
 $EndComp
 $Comp
-L EGND_PSPICE EGND
+L EGND_PSPICE #PWR4
 U 1 1 14636915
 P 3900 1400
-F 0 "EGND" H 7800 2800 30  0001 L CNN
+F 0 "#PWR4" H 7800 2800 30  0001 L CNN
 F 1 "EGND" H 7800 2880 30  0001 L CNN
 	1    3900 1400
@@
 $EndComp
 $Comp
-L EGND_PSPICE EGND
+L EGND_PSPICE #PWR5
 U 1 1 77747793
 P 3100 1500
-F 0 "EGND" H 6200 3000 30  0001 L CNN
+F 0 "#PWR5" H 6200 3000 30  0001 L CNN
 F 1 "EGND" H 6200 3080 30  0001 L CNN
 	1    3100 1500
@@
 $EndComp
 $Comp
-L EGND_PSPICE EGND
+L EGND_PSPICE #PWR6
 U 1 1 74238335
 P 3200 3000
-F 0 "EGND" H 6400 6000 30  0001 L CNN
+F 0 "#PWR6" H 6400 6000 30  0001 L CNN
 F 1 "EGND" H 6400 6080 30  0001 L CNN
 	1    3200 3000
@@
 $EndComp
 $Comp
-L EGND_PSPICE EGND
+L EGND_PSPICE #PWR7
 U 1 1 99885386
 P 5000 2900
-F 0 "EGND" H 10000 5800 30  0001 L CNN
+F 0 "#PWR7" H 10000 5800 30  0001 L CNN
 F 1 "EGND" H 10000 5880 30  0001 L CNN
 	1    5000 2900
@@
 $EndComp
 $Comp
-L EGND_PSPICE EGND
+L EGND_PSPICE #PWR8
 U 1 1 39760492
 P 4900 1500
-F 0 "EGND" H 9800 3000 30  0001 L CNN
+F 0 "#PWR8" H 9800 3000 30  0001 L CNN
 F 1 "EGND" H 9800 3080 30  0001 L CNN
 	1    4900 1500

Commit message: Added LICENSE.txt
Changed lines of the file:
@@
 $EndDescr
 $Comp
-L EGND_PSPICE #PWR1
+L GND #PWR1
 U 1 1 14289383
 P 5800 2400
@@
 $EndComp
 $Comp
-L EGND_PSPICE #PWR2
+L GND #PWR2
 U 1 1 46930886
 P 500 1700
@@
 $EndComp
 $Comp
-L EGND_PSPICE #PWR3
+L GND #PWR3
 U 1 1 71692777
 P 4000 2800
@@
 $EndComp
 $Comp
-L EGND_PSPICE #PWR4
+L GND #PWR4
 U 1 1 14636915
 P 3900 1400
@@
 $EndComp
 $Comp
-L EGND_PSPICE #PWR5
+L GND #PWR5
 U 1 1 77747793
 P 3100 1500
@@
 $EndComp
 $Comp
-L EGND_PSPICE #PWR6
+L GND #PWR6
 U 1 1 74238335
 P 3200 3000
@@
 $EndComp
 $Comp
-L EGND_PSPICE #PWR7
+L GND #PWR7
 U 1 1 99885386
 P 5000 2900
@@
 $EndComp
 $Comp
-L EGND_PSPICE #PWR8
+L GND #PWR8
 U 1 1 39760492
 P 4900 1500

Commit message: Orientation fix. Library components are now inverted, with +ve y axis going up. In Schematic files, +ve y axis is downwards. This is how the KiCad libraries are. As a result of the above fixed, the converted GND is now oriented correctly.
Parts:
- V1, V2: value VSIN -> SINE
Other:
- moved on the sheet: U1, U2, V1, V2
Changed lines of the file:
@@
 F 1 "EGND" H 11600 4880 30  0001 L CNN
 	1    5800 2400
-	1    0    0    1
+	1    0    0    -1
 $EndComp
 $Comp
@@
 F 1 "EGND" H 1000 3480 30  0001 L CNN
 	1    500 1700
-	1    0    0    1
+	1    0    0    -1
 $EndComp
 $Comp
@@
 F 1 "EGND" H 8000 5680 30  0001 L CNN
 	1    4000 2800
-	1    0    0    1
+	1    0    0    -1
 $EndComp
 $Comp
@@
 F 1 "EGND" H 7800 2880 30  0001 L CNN
 	1    3900 1400
-	1    0    0    1
+	1    0    0    -1
 $EndComp
 $Comp
@@
 F 1 "EGND" H 6200 3080 30  0001 L CNN
 	1    3100 1500
-	1    0    0    1
+	1    0    0    -1
 $EndComp
 $Comp
@@
 F 1 "EGND" H 6400 6080 30  0001 L CNN
 	1    3200 3000
-	1    0    0    1
+	1    0    0    -1
 $EndComp
 $Comp
@@
 F 1 "EGND" H 10000 5880 30  0001 L CNN
 	1    5000 2900
-	1    0    0    1
+	1    0    0    -1
 $EndComp
 $Comp
@@
 F 1 "EGND" H 9800 3080 30  0001 L CNN
 	1    4900 1500
-	1    0    0    1
+	1    0    0    -1
 $EndComp
 $Comp
@@
 F 1 "D1N4002" H 2200 1380 30  0000 L CNN
 	1    2200 1300
-	0    1    -1    0
+	0    -1    -1    0
 $EndComp
 $Comp
@@
 F 1 "D1N4002" H 1700 2480 30  0000 L CNN
 	1    1700 2400
-	0    1    -1    0
+	0    -1    -1    0
 $EndComp
 $Comp
@@
 F 1 "D1N4002" H 2200 2480 30  0000 L CNN
 	1    2200 2400
-	0    1    -1    0
+	0    -1    -1    0
 $EndComp
 $Comp
@@
 F 1 "D1N4002" H 1700 1380 30  0000 L CNN
 	1    1700 1300
-	0    1    -1    0
+	0    -1    -1    0
 $EndComp
 $Comp
@@
 P 800 1300
 F 0 "V1" H 800 1300 30  0000 L CNN
-F 1 "VSIN" H 800 1380 30  0000 L CNN
+F 1 "SINE" H 800 1380 30  0000 L CNN
 	1    800 1300
-	1    0    0    1
+	1    0    0    -1
 $EndComp
 $Comp
@@
 P 800 1800
 F 0 "V2" H 800 1800 30  0000 L CNN
-F 1 "VSIN" H 800 1880 30  0000 L CNN
+F 1 "SINE" H 800 1880 30  0000 L CNN
 	1    800 1800
-	1    0    0    1
+	1    0    0    -1
 $EndComp
 $Comp
@@
 F 1 "1000uF" H 3200 3050 30  0000 L CNN
 	1    3200 2700
-	0    -1    1    0
+	0    1    1    0
 $EndComp
 $Comp
@@
 F 1 "100uF" H 4900 1510 30  0000 L CNN
 	1    4900 1200
-	0    -1    1    0
+	0    1    1    0
 $EndComp
 $Comp
@@
 F 1 "50" H 5600 2230 30  0000 L CNN
 	1    5600 2000
-	0    -1    1    0
+	0    1    1    0
 $EndComp
 $Comp
@@
 F 1 "100uF" H 5000 2910 30  0000 L CNN
 	1    5000 2600
-	0    -1    1    0
+	0    1    1    0
 $EndComp
 $Comp
@@
 F 1 "50" H 5600 2930 30  0000 L CNN
 	1    5600 2500
-	0    -1    1    0
+	0    1    1    0
 $EndComp
 $Comp
@@
 F 1 "LM7815C" H 3200 1180 30  0000 L CNN
 	1    3200 1100
-	1    0    0    1
+	1    0    0    -1
 $EndComp
 $Comp
@@
 F 1 "LM7915C" H 3300 2580 30  0000 L CNN
 	1    3300 2500
-	1    0    0    1
+	1    0    0    -1
 $EndComp
 $Comp
@@
 F 1 "1000uF" H 3100 1550 30  0000 L CNN
 	1    3100 1200
-	0    -1    1    0
+	0    1    1    0
 $EndComp
 Wire Wire Line

Commit message: Removed the use of exec, wrote basename function, made integration with eSim easier.
Parts:
- added C1: 1000uF, symbol C_PSPICE
- added titleblk: titleblk, symbol titleblk_PSPICE
- C2: renamed from RL1; value 50 -> 100uF; symbol R_PSPICE -> C_PSPICE
- C3: renamed from RL2; value 50 -> 100uF; symbol R_PSPICE -> C_PSPICE
- C4: renamed from C2; value 100uF -> 1000uF
- PM2: renamed from C4; value 1000uF -> PARAM; symbol C_PSPICE -> PARAM_PSPICE
- RL1: renamed from C3; value 100uF -> 50; symbol C_PSPICE -> R_PSPICE
- RL2: renamed from U1; value LM7815C -> 50; symbol LM7815C_PSPICE -> R_PSPICE
- U1: renamed from U2; value LM7915C -> LM7815C; symbol LM7915C_PSPICE -> LM7815C_PSPICE
- U2: renamed from C1; value 1000uF -> LM7915C; symbol C_PSPICE -> LM7915C_PSPICE
Other:
- moved on the sheet: C4, U1
Changed lines of the file:
@@
-EESchema Schematic File Version 2  date Sunday 05 March 2000 07:11:03 PM IST
+EESchema Schematic File Version 2  date
 LIBS:power
 LIBS:device
@@
 LIBS:contrib
 LIBS:valves
-LIBS:ConvertedSchematicFiles/EXP2_10-cache
 EELAYER 25  0
 EELAYER END
@@
 Sheet 1 1
 Title ""
-Date "05 Mar 2000"
+Date ""
 Rev ""
 Comp ""
@@
 $EndComp
 $Comp
+L PARAM_PSPICE PM2
+U 1 1 74897763
+P 5700 500
+F 0 "PM2" H 5700 500 30  0000 L CNN
+F 1 "PARAM" H 5700 580 30  0000 L CNN
+	1    5700 500
+	1    0    0    -1
+$EndComp
+$Comp
 L C_PSPICE C4
-U 1 1 74897763
+U 1 1 87513926
 P 3200 2700
 F 0 "C4" H 3200 2700 30  0000 L CNN
@@
 $Comp
 L C_PSPICE C2
-U 1 1 87513926
+U 1 1 25180540
 P 4900 1200
 F 0 "C2" H 4900 1200 30  0000 L CNN
@@
 $Comp
 L R_PSPICE RL1
-U 1 1 25180540
+U 1 1 20383426
 P 5600 2000
 F 0 "RL1" H 5600 2000 30  0000 L CNN
@@
 $Comp
 L C_PSPICE C3
-U 1 1 20383426
+U 1 1 44089172
 P 5000 2600
 F 0 "C3" H 5000 2600 30  0000 L CNN
@@
 $Comp
 L R_PSPICE RL2
-U 1 1 44089172
+U 1 1 53455736
 P 5600 2500
 F 0 "RL2" H 5600 2500 30  0000 L CNN
@@
 $Comp
 L LM7815C_PSPICE U1
-U 1 1 53455736
+U 1 1 45005211
 P 3200 1100
 F 0 "U1" H 3200 1100 30  0000 L CNN
@@
 $Comp
 L LM7915C_PSPICE U2
-U 1 1 45005211
+U 1 1 81595368
 P 3300 2500
 F 0 "U2" H 3300 2500 30  0000 L CNN
@@
 $Comp
 L C_PSPICE C1
-U 1 1 81595368
+U 1 1 34702567
 P 3100 1200
 F 0 "C1" H 3100 1200 30  0000 L CNN
@@
 	0    1    1    0
 $EndComp
+$Comp
+L titleblk_PSPICE titleblk
+U 1 1 26956429
+P 9700 7200
+F 0 "titleblk" H 19400 14400 30  0001 L CNN
+F 1 "titleblk" H 19400 14480 30  0001 L CNN
+	1    9700 7200
+	1    0    0    -1
+$EndComp
 Wire Wire Line
