File: ConvertedSchematicFiles/EXP2_7/EXP2_7.sch (KiCad schematic (older format))
At the start: 16 parts

Commit message: Excluded some components. These no longer appear after conversion. When calling shell commands, filenames are in "quotes"
Parts:
- removed V4: VPULSE, symbol VPULSE_PSPICE
- removed titleblk: titleblk, symbol TITLEBLK_PSPICE
- V4: renamed from V5; value VPWL -> VPULSE; symbol VPWL_PSPICE -> VPULSE_PSPICE
- V5: renamed from PM1; value PARAM -> VPWL; symbol PARAM_PSPICE -> VPWL_PSPICE
Connections:
- net at E1.IN+: now also V4.+
- net at E4.IN+: now also V5.+; no longer V4.+
Changed lines of the file:
@@
-$EndComp
-$Comp
-L PARAM_PSPICE PM1
-U 1 1 73368690
-P 4200 900
-F 0 "PM1" H 4200 900 30  0001 L CNN
-F 1 "PARAM" H 4200 980 30  0001 L CNN
-	1    4200 900
-	1    0    0    1
 $EndComp
 $Comp
 L VPWL_PSPICE V5
-U 1 1 32520059
+U 1 1 73368690
 P 1800 1700
 F 0 "V5" H 1800 1700 30  0001 L CNN
@@
 $Comp
 L VPULSE_PSPICE V4
-U 1 1 74897763
+U 1 1 32520059
 P 1200 1000
 F 0 "V4" H 1200 1000 30  0001 L CNN
@@
 	1    0    0    1
 $EndComp
-$Comp
-L TITLEBLK_PSPICE titleblk
-U 1 1 87513926
-P 9700 7200
-F 0 "titleblk" H 19400 14400 30  0001 L CNN
-F 1 "titleblk" H 19400 14480 30  0001 L CNN
-	1    9700 7200
-	1    0    0    1
-$EndComp

Commit message: Ports issue fixed. Now annotation for ports is #PWR? function added "itos"
Parts:
- removed EGND (x8): EGND, symbol EGND_PSPICE
Changed lines of the file:
@@
 $EndDescr
 $Comp
-L EGND_PSPICE EGND
+L EGND_PSPICE #PWR1
 U 1 1 14289383
 P 1800 800
-F 0 "EGND" H 3600 1600 30  0001 L CNN
+F 0 "#PWR1" H 3600 1600 30  0001 L CNN
 F 1 "EGND" H 3600 1680 30  0001 L CNN
 	1    1800 800
@@
 $EndComp
 $Comp
-L EGND_PSPICE EGND
+L EGND_PSPICE #PWR2
 U 1 1 46930886
 P 3100 700
-F 0 "EGND" H 6200 1400 30  0001 L CNN
+F 0 "#PWR2" H 6200 1400 30  0001 L CNN
 F 1 "EGND" H 6200 1480 30  0001 L CNN
 	1    3100 700
@@
 $EndComp
 $Comp
-L EGND_PSPICE EGND
+L EGND_PSPICE #PWR3
 U 1 1 71692777
 P 2500 800
-F 0 "EGND" H 5000 1600 30  0001 L CNN
+F 0 "#PWR3" H 5000 1600 30  0001 L CNN
 F 1 "EGND" H 5000 1680 30  0001 L CNN
 	1    2500 800
@@
 $EndComp
 $Comp
-L EGND_PSPICE EGND
+L EGND_PSPICE #PWR4
 U 1 1 14636915
 P 1200 1400
-F 0 "EGND" H 2400 2800 30  0001 L CNN
+F 0 "#PWR4" H 2400 2800 30  0001 L CNN
 F 1 "EGND" H 2400 2880 30  0001 L CNN
 	1    1200 1400
@@
 $EndComp
 $Comp
-L EGND_PSPICE EGND
+L EGND_PSPICE #PWR5
 U 1 1 77747793
 P 4100 1700
-F 0 "EGND" H 8200 3400 30  0001 L CNN
+F 0 "#PWR5" H 8200 3400 30  0001 L CNN
 F 1 "EGND" H 8200 3480 30  0001 L CNN
 	1    4100 1700
@@
 $EndComp
 $Comp
-L EGND_PSPICE EGND
+L EGND_PSPICE #PWR6
 U 1 1 74238335
 P 1800 2100
-F 0 "EGND" H 3600 4200 30  0001 L CNN
+F 0 "#PWR6" H 3600 4200 30  0001 L CNN
 F 1 "EGND" H 3600 4280 30  0001 L CNN
 	1    1800 2100
@@
 $EndComp
 $Comp
-L EGND_PSPICE EGND
+L EGND_PSPICE #PWR7
 U 1 1 99885386
 P 3500 1800
-F 0 "EGND" H 7000 3600 30  0001 L CNN
+F 0 "#PWR7" H 7000 3600 30  0001 L CNN
 F 1 "EGND" H 7000 3680 30  0001 L CNN
 	1    3500 1800
@@
 $EndComp
 $Comp
-L EGND_PSPICE EGND
+L EGND_PSPICE #PWR8
 U 1 1 39760492
 P 2800 1800
-F 0 "EGND" H 5600 3600 30  0001 L CNN
+F 0 "#PWR8" H 5600 3600 30  0001 L CNN
 F 1 "EGND" H 5600 3680 30  0001 L CNN
 	1    2800 1800

Commit message: Added LICENSE.txt
Parts:
- V4: value VPULSE -> PULSE
Changed lines of the file:
@@
 $EndDescr
 $Comp
-L EGND_PSPICE #PWR1
+L GND #PWR1
 U 1 1 14289383
 P 1800 800
@@
 $EndComp
 $Comp
-L EGND_PSPICE #PWR2
+L GND #PWR2
 U 1 1 46930886
 P 3100 700
@@
 $EndComp
 $Comp
-L EGND_PSPICE #PWR3
+L GND #PWR3
 U 1 1 71692777
 P 2500 800
@@
 $EndComp
 $Comp
-L EGND_PSPICE #PWR4
+L GND #PWR4
 U 1 1 14636915
 P 1200 1400
@@
 $EndComp
 $Comp
-L EGND_PSPICE #PWR5
+L GND #PWR5
 U 1 1 77747793
 P 4100 1700
@@
 $EndComp
 $Comp
-L EGND_PSPICE #PWR6
+L GND #PWR6
 U 1 1 74238335
 P 1800 2100
@@
 $EndComp
 $Comp
-L EGND_PSPICE #PWR7
+L GND #PWR7
 U 1 1 99885386
 P 3500 1800
@@
 $EndComp
 $Comp
-L EGND_PSPICE #PWR8
+L GND #PWR8
 U 1 1 39760492
 P 2800 1800
@@
 P 1200 1000
 F 0 "V4" H 1200 1000 30  0001 L CNN
-F 1 "VPULSE" H 1200 1080 30  0001 L CNN
+F 1 "PULSE" H 1200 1080 30  0001 L CNN
 	1    1200 1000
 	1    0    0    1

Commit message: Orientation fix. Library components are now inverted, with +ve y axis going up. In Schematic files, +ve y axis is downwards. This is how the KiCad libraries are. As a result of the above fixed, the converted GND is now oriented correctly.
Changed lines of the file:
@@
 F 1 "EGND" H 3600 1680 30  0001 L CNN
 	1    1800 800
-	1    0    0    1
+	1    0    0    -1
 $EndComp
 $Comp
@@
 F 1 "EGND" H 6200 1480 30  0001 L CNN
 	1    3100 700
-	1    0    0    1
+	1    0    0    -1
 $EndComp
 $Comp
@@
 F 1 "EGND" H 5000 1680 30  0001 L CNN
 	1    2500 800
-	1    0    0    1
+	1    0    0    -1
 $EndComp
 $Comp
@@
 F 1 "EGND" H 2400 2880 30  0001 L CNN
 	1    1200 1400
-	1    0    0    1
+	1    0    0    -1
 $EndComp
 $Comp
@@
 F 1 "EGND" H 8200 3480 30  0001 L CNN
 	1    4100 1700
-	1    0    0    1
+	1    0    0    -1
 $EndComp
 $Comp
@@
 F 1 "EGND" H 3600 4280 30  0001 L CNN
 	1    1800 2100
-	1    0    0    1
+	1    0    0    -1
 $EndComp
 $Comp
@@
 F 1 "EGND" H 7000 3680 30  0001 L CNN
 	1    3500 1800
-	1    0    0    1
+	1    0    0    -1
 $EndComp
 $Comp
@@
 F 1 "EGND" H 5600 3680 30  0001 L CNN
 	1    2800 1800
-	1    0    0    1
+	1    0    0    -1
 $EndComp
 $Comp
@@
 F 1 "R" H 2700 780 30  0001 L CNN
 	1    2700 700
-	1    0    0    1
+	1    0    0    -1
 $EndComp
 $Comp
@@
 F 1 "R" H 3700 1780 30  0001 L CNN
 	1    3700 1700
-	1    0    0    1
+	1    0    0    -1
 $EndComp
 $Comp
@@
 F 1 "ELAPLACE" H 2800 1780 30  0001 L CNN
 	1    2800 1700
-	1    0    0    1
+	1    0    0    -1
 $EndComp
 $Comp
@@
 F 1 "ELAPLACE" H 1800 780 30  0001 L CNN
 	1    1800 700
-	1    0    0    1
+	1    0    0    -1
 $EndComp
 $Comp
@@
 F 1 "VPWL" H 1800 1780 30  0001 L CNN
 	1    1800 1700
-	1    0    0    1
+	1    0    0    -1
 $EndComp
 $Comp
@@
 F 1 "PULSE" H 1200 1080 30  0001 L CNN
 	1    1200 1000
-	1    0    0    1
+	1    0    0    -1
 $EndComp
 Wire Wire Line

Commit message: Removed the use of exec, wrote basename function, made integration with eSim easier.
Parts:
- added V4: PULSE, symbol VPULSE_PSPICE
- added titleblk: titleblk, symbol titleblk_PSPICE
- PM1: renamed from V5; value VPWL -> PARAM; symbol VPWL_PSPICE -> PARAM_PSPICE
- V5: renamed from V4; value PULSE -> VPWL; symbol VPULSE_PSPICE -> VPWL_PSPICE
Changed lines of the file:
@@
-EESchema Schematic File Version 2  date Thursday 09 March 2000 10:07:32 AM IST
+EESchema Schematic File Version 2  date
 LIBS:power
 LIBS:device
@@
 LIBS:contrib
 LIBS:valves
-LIBS:ConvertedSchematicFiles/EXP2_7-cache
 EELAYER 25  0
 EELAYER END
@@
 Sheet 1 1
 Title ""
-Date "09 Mar 2000"
+Date ""
 Rev ""
 Comp ""
@@
 $EndComp
 $Comp
+L PARAM_PSPICE PM1
+U 1 1 73368690
+P 4200 900
+F 0 "PM1" H 4200 900 30  0001 L CNN
+F 1 "PARAM" H 4200 980 30  0001 L CNN
+	1    4200 900
+	1    0    0    -1
+$EndComp
+$Comp
 L VPWL_PSPICE V5
-U 1 1 73368690
+U 1 1 32520059
 P 1800 1700
 F 0 "V5" H 1800 1700 30  0001 L CNN
@@
 $Comp
 L VPULSE_PSPICE V4
-U 1 1 32520059
+U 1 1 74897763
 P 1200 1000
 F 0 "V4" H 1200 1000 30  0001 L CNN
@@
 	1    0    0    -1
 $EndComp
+$Comp
+L titleblk_PSPICE titleblk
+U 1 1 87513926
+P 9700 7200
+F 0 "titleblk" H 19400 14400 30  0001 L CNN
+F 1 "titleblk" H 19400 14480 30  0001 L CNN
+	1    9700 7200
+	1    0    0    -1
+$EndComp
