File: ConvertedSchematicFiles/EXP4_3/EXP4_3.sch (KiCad schematic (older format))
At the start: 17 parts

Commit message: Excluded some components. These no longer appear after conversion. When calling shell commands, filenames are in "quotes"
Parts:
- removed D7: D1N4002, symbol D1N4002_PSPICE
- removed titleblk: titleblk, symbol TITLEBLK_PSPICE
- D4: renamed from V2; value VSIN -> D1N4002; symbol VSIN_PSPICE -> D1N4002_PSPICE
- RL2: renamed from PM1; value PARAM -> 1K; symbol PARAM_PSPICE -> R_PSPICE
- V2: renamed from RL2; value 1K -> VSIN; symbol R_PSPICE -> VSIN_PSPICE
- renumbered D5 to D1, D1 to D2, D4 to D3, D8 to D5, D3 to D6, D2 to D7, D6 to D8
Other:
- moved on the sheet: D1, D2, D3, D4, D5, D6, D7, D8
Changed lines of the file:
@@
-$EndComp
-$Comp
-L PARAM_PSPICE PM1
-U 1 1 74238335
-P 3800 3200
-F 0 "PM1" H 3800 3200 30  0000 L CNN
-F 1 "PARAM" H 3800 3280 30  0000 L CNN
-	1    3800 3200
-	1    0    0    1
 $EndComp
 $Comp
 L R_PSPICE RL2
-U 1 1 99885386
+U 1 1 74238335
 P 9200 1600
 F 0 "RL2" H 9200 1600 30  0000 L CNN
@@
 $Comp
 L VSIN_PSPICE V2
-U 1 1 39760492
+U 1 1 99885386
 P 6200 1600
 F 0 "V2" H 6200 1600 30  0000 L CNN
@@
 $Comp
 L D1N4002_PSPICE D4
-U 1 1 66516649
+U 1 1 39760492
 P 3900 2500
 F 0 "D4" H 3900 2500 30  0000 L CNN
@@
 $Comp
 L D1N4002_PSPICE D3
-U 1 1 29641421
+U 1 1 66516649
 P 3200 2500
 F 0 "D3" H 3200 2500 30  0000 L CNN
@@
 $Comp
 L D1N4002_PSPICE D6
-U 1 1 45202362
+U 1 1 29641421
 P 7700 2400
 F 0 "D6" H 7700 2400 30  0000 L CNN
@@
 $Comp
 L D1N4002_PSPICE D8
-U 1 1 10490027
+U 1 1 45202362
 P 7000 1600
 F 0 "D8" H 7000 1600 30  0000 L CNN
@@
 $Comp
 L D1N4002_PSPICE D5
-U 1 1 73368690
+U 1 1 10490027
 P 7700 1600
 F 0 "D5" H 7700 1600 30  0000 L CNN
@@
 $Comp
 L D1N4002_PSPICE D1
-U 1 1 32520059
+U 1 1 73368690
 P 3200 1700
 F 0 "D1" H 3200 1700 30  0000 L CNN
@@
 $Comp
 L D1N4002_PSPICE D2
-U 1 1 74897763
+U 1 1 32520059
 P 3900 1700
 F 0 "D2" H 3900 1700 30  0000 L CNN
@@
 $Comp
 L D1N4002_PSPICE D7
-U 1 1 87513926
+U 1 1 74897763
 P 7000 2400
 F 0 "D7" H 7000 2400 30  0000 L CNN
@@
 	0    1    -1    0
 $EndComp
-$Comp
-L TITLEBLK_PSPICE titleblk
-U 1 1 25180540
-P 11880 8400
-F 0 "titleblk" H 23760 16800 30  0001 L CNN
-F 1 "titleblk" H 23760 16880 30  0001 L CNN
-	1    11880 8400
-	1    0    0    1
-$EndComp
 Wire Wire Line

Commit message: Ports issue fixed. Now annotation for ports is #PWR? function added "itos"
Parts:
- removed EGND (x2): EGND, symbol EGND_PSPICE
Connections:
- net labels added: EGND
Changed lines of the file:
@@
 $EndDescr
 $Comp
-L EGND_PSPICE EGND
+L EGND_PSPICE #PWR1
 U 1 1 14289383
 P 3900 2700
-F 0 "EGND" H 7800 5400 30  0001 L CNN
+F 0 "#PWR1" H 7800 5400 30  0001 L CNN
 F 1 "EGND" H 7800 5480 30  0001 L CNN
 	1    3900 2700
@@
 $EndComp
 $Comp
-L EGND_PSPICE EGND
+L EGND_PSPICE #PWR2
 U 1 1 46930886
 P 7700 2600
-F 0 "EGND" H 15400 5200 30  0001 L CNN
+F 0 "#PWR2" H 15400 5200 30  0001 L CNN
 F 1 "EGND" H 15400 5280 30  0001 L CNN
 	1    7700 2600

Commit message: Added LICENSE.txt
Changed lines of the file:
@@
 $EndDescr
 $Comp
-L EGND_PSPICE #PWR1
+L GND #PWR1
 U 1 1 14289383
 P 3900 2700
@@
 $EndComp
 $Comp
-L EGND_PSPICE #PWR2
+L GND #PWR2
 U 1 1 46930886
 P 7700 2600

Commit message: Orientation fix. Library components are now inverted, with +ve y axis going up. In Schematic files, +ve y axis is downwards. This is how the KiCad libraries are. As a result of the above fixed, the converted GND is now oriented correctly.
Parts:
- V1, V2: value VSIN -> SINE
Other:
- moved on the sheet: V1, V2
Changed lines of the file:
@@
 F 1 "EGND" H 7800 5480 30  0001 L CNN
 	1    3900 2700
-	1    0    0    1
+	1    0    0    -1
 $EndComp
 $Comp
@@
 F 1 "EGND" H 15400 5280 30  0001 L CNN
 	1    7700 2600
-	1    0    0    1
+	1    0    0    -1
 $EndComp
 $Comp
@@
 F 1 "{C_FILT}" H 4700 2110 30  0000 L CNN
 	1    4700 1800
-	0    -1    1    0
+	0    1    1    0
 $EndComp
 $Comp
@@
 F 1 "1K" H 5400 1970 30  0000 L CNN
 	1    5400 1700
-	0    -1    1    0
+	0    1    1    0
 $EndComp
 $Comp
@@
 P 2600 1700
 F 0 "V1" H 2600 1700 30  0000 L CNN
-F 1 "VSIN" H 2600 1780 30  0000 L CNN
+F 1 "SINE" H 2600 1780 30  0000 L CNN
 	1    2600 1700
-	1    0    0    1
+	1    0    0    -1
 $EndComp
 $Comp
@@
 F 1 "1K" H 9200 1870 30  0000 L CNN
 	1    9200 1600
-	0    -1    1    0
+	0    1    1    0
 $EndComp
 $Comp
@@
 P 6200 1600
 F 0 "V2" H 6200 1600 30  0000 L CNN
-F 1 "VSIN" H 6200 1680 30  0000 L CNN
+F 1 "SINE" H 6200 1680 30  0000 L CNN
 	1    6200 1600
-	1    0    0    1
+	1    0    0    -1
 $EndComp
 $Comp
@@
 F 1 "D1N4002" H 3900 2580 30  0000 L CNN
 	1    3900 2500
-	0    1    -1    0
+	0    -1    -1    0
 $EndComp
 $Comp
@@
 F 1 "D1N4002" H 3200 2580 30  0000 L CNN
 	1    3200 2500
-	0    1    -1    0
+	0    -1    -1    0
 $EndComp
 $Comp
@@
 F 1 "D1N4002" H 7700 2480 30  0000 L CNN
 	1    7700 2400
-	0    1    -1    0
+	0    -1    -1    0
 $EndComp
 $Comp
@@
 F 1 "D1N4002" H 7000 1680 30  0000 L CNN
 	1    7000 1600
-	0    1    -1    0
+	0    -1    -1    0
 $EndComp
 $Comp
@@
 F 1 "D1N4002" H 7700 1680 30  0000 L CNN
 	1    7700 1600
-	0    1    -1    0
+	0    -1    -1    0
 $EndComp
 $Comp
@@
 F 1 "D1N4002" H 3200 1780 30  0000 L CNN
 	1    3200 1700
-	0    1    -1    0
+	0    -1    -1    0
 $EndComp
 $Comp
@@
 F 1 "D1N4002" H 3900 1780 30  0000 L CNN
 	1    3900 1700
-	0    1    -1    0
+	0    -1    -1    0
 $EndComp
 $Comp
@@
 F 1 "D1N4002" H 7000 2480 30  0000 L CNN
 	1    7000 2400
-	0    1    -1    0
+	0    -1    -1    0
 $EndComp
 Wire Wire Line

Commit message: Removed the use of exec, wrote basename function, made integration with eSim easier.
Parts:
- added D7: D1N4002, symbol D1N4002_PSPICE
- added titleblk: titleblk, symbol titleblk_PSPICE
- PM1: renamed from RL2; value 1K -> PARAM; symbol R_PSPICE -> PARAM_PSPICE
- RL2: renamed from V2; value SINE -> 1K; symbol VSIN_PSPICE -> R_PSPICE
- V2: renamed from D4; value D1N4002 -> SINE; symbol D1N4002_PSPICE -> VSIN_PSPICE
- renumbered D2 to D1, D7 to D2, D6 to D3, D3 to D4, D1 to D5, D8 to D6, D5 to D8
Other:
- moved on the sheet: D1, D2, D3, D4, D5, D6, D8, V2
Changed lines of the file:
@@
-EESchema Schematic File Version 2  date Wednesday 01 March 2000 08:02:18 PM IST
+EESchema Schematic File Version 2  date
 LIBS:power
 LIBS:device
@@
 LIBS:contrib
 LIBS:valves
-LIBS:ConvertedSchematicFiles/EXP4_3-cache
 EELAYER 25  0
 EELAYER END
@@
 Sheet 1 1
 Title ""
-Date "01 Mar 2000"
+Date ""
 Rev ""
 Comp ""
@@
 $EndComp
 $Comp
+L PARAM_PSPICE PM1
+U 1 1 74238335
+P 3800 3200
+F 0 "PM1" H 3800 3200 30  0000 L CNN
+F 1 "PARAM" H 3800 3280 30  0000 L CNN
+	1    3800 3200
+	1    0    0    -1
+$EndComp
+$Comp
 L R_PSPICE RL2
-U 1 1 74238335
+U 1 1 99885386
 P 9200 1600
 F 0 "RL2" H 9200 1600 30  0000 L CNN
@@
 $Comp
 L VSIN_PSPICE V2
-U 1 1 99885386
+U 1 1 39760492
 P 6200 1600
 F 0 "V2" H 6200 1600 30  0000 L CNN
@@
 $Comp
 L D1N4002_PSPICE D4
-U 1 1 39760492
+U 1 1 66516649
 P 3900 2500
 F 0 "D4" H 3900 2500 30  0000 L CNN
@@
 $Comp
 L D1N4002_PSPICE D3
-U 1 1 66516649
+U 1 1 29641421
 P 3200 2500
 F 0 "D3" H 3200 2500 30  0000 L CNN
@@
 $Comp
 L D1N4002_PSPICE D6
-U 1 1 29641421
+U 1 1 45202362
 P 7700 2400
 F 0 "D6" H 7700 2400 30  0000 L CNN
@@
 $Comp
 L D1N4002_PSPICE D8
-U 1 1 45202362
+U 1 1 10490027
 P 7000 1600
 F 0 "D8" H 7000 1600 30  0000 L CNN
@@
 $Comp
 L D1N4002_PSPICE D5
-U 1 1 10490027
+U 1 1 73368690
 P 7700 1600
 F 0 "D5" H 7700 1600 30  0000 L CNN
@@
 $Comp
 L D1N4002_PSPICE D1
-U 1 1 73368690
+U 1 1 32520059
 P 3200 1700
 F 0 "D1" H 3200 1700 30  0000 L CNN
@@
 $Comp
 L D1N4002_PSPICE D2
-U 1 1 32520059
+U 1 1 74897763
 P 3900 1700
 F 0 "D2" H 3900 1700 30  0000 L CNN
@@
 $Comp
 L D1N4002_PSPICE D7
-U 1 1 74897763
+U 1 1 87513926
 P 7000 2400
 F 0 "D7" H 7000 2400 30  0000 L CNN
@@
 	0    -1    -1    0
 $EndComp
+$Comp
+L titleblk_PSPICE titleblk
+U 1 1 25180540
+P 11880 8400
+F 0 "titleblk" H 23760 16800 30  0001 L CNN
+F 1 "titleblk" H 23760 16880 30  0001 L CNN
+	1    11880 8400
+	1    0    0    -1
+$EndComp
 Wire Wire Line
