File: ConvertedSchematicFiles/EXP6_12/EXP6_12.sch (KiCad schematic (older format))
At the start: 25 parts

Commit message: Excluded some components. These no longer appear after conversion. When calling shell commands, filenames are in "quotes"
Parts:
- removed C6: 0.047NF, symbol C_PSPICE
- removed C8: 0.22U, symbol C_PSPICE
- removed nodeMarker (x2): nodeMarker, symbol NODEMARKER_PSPICE
- removed titleblk: titleblk, symbol TITLEBLK_PSPICE
- C6: renamed from R3; value 1K -> 0.047NF; symbol R_PSPICE -> C_PSPICE
- C8: renamed from PM1; value PARAM -> 0.22U; symbol PARAM_PSPICE -> C_PSPICE
- R3: renamed from V1; value VSFFM -> 1K; symbol VSFFM_PSPICE -> R_PSPICE
- V2: renamed from PM2; value PARAM -> VSFFM; symbol PARAM_PSPICE -> VSFFM_PSPICE
- renumbered V2 to V1
Connections:
- net at C1.2, C2.2, D2.2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: now also C8.2
- net at C1.1, C2.1, D1.1: now also C8.1, V1.+; no longer R3.+
- net at L1.1: now also V2.+; no longer V1.+
- net at C6.2: now also C5.2, EGND.EGND, R5.2
- net at L1.2: now also R3.1; no longer C6.1
- new net: C6.1, R3.2
Other:
- moved on the sheet: V1
Changed lines of the file:
@@
-$EndComp
-$Comp
-L PARAM_PSPICE PM2
-U 1 1 87513926
-P 7300 3300
-F 0 "PM2" H 7300 3300 30  0000 L CNN
-F 1 "PARAM" H 7300 3380 30  0000 L CNN
-	1    7300 3300
-	1    0    0    1
 $EndComp
 $Comp
 L VSFFM_PSPICE V2
-U 1 1 25180540
+U 1 1 87513926
 P 3000 3500
 F 0 "V2" H 3000 3500 30  0000 L CNN
@@
 $Comp
 L VSFFM_PSPICE V1
-U 1 1 20383426
+U 1 1 25180540
 P 3000 2800
 F 0 "V1" H 3000 2800 30  0000 L CNN
@@
 $EndComp
 $Comp
-L PARAM_PSPICE PM1
-U 1 1 44089172
-P 7300 2700
-F 0 "PM1" H 7300 2700 30  0000 L CNN
-F 1 "PARAM" H 7300 2780 30  0000 L CNN
-	1    7300 2700
-	1    0    0    1
-$EndComp
-$Comp
 L R_PSPICE R3
-U 1 1 53455736
+U 1 1 20383426
 P 5300 4400
 F 0 "R3" H 5300 4400 30  0000 L CNN
@@
 $Comp
 L C_PSPICE C8
-U 1 1 45005211
+U 1 1 44089172
 P 2200 3400
 F 0 "C8" H 2200 3400 30  0000 L CNN
@@
 $Comp
 L C_PSPICE C6
-U 1 1 81595368
+U 1 1 53455736
 P 6100 4500
 F 0 "C6" H 6100 4500 30  0000 L CNN
@@
 	0    -1    1    0
 $EndComp
-$Comp
-L TITLEBLK_PSPICE titleblk
-U 1 1 34702567
-P 11880 8400
-F 0 "titleblk" H 23760 16800 30  0001 L CNN
-F 1 "titleblk" H 23760 16880 30  0001 L CNN
-	1    11880 8400
-	1    0    0    1
-$EndComp
-$Comp
-L NODEMARKER_PSPICE nodeMarker
-U 1 1 26956429
-P 6100 4400
-F 0 "nodeMarker" H 12200 8800 30  0001 L CNN
-F 1 "nodeMarker" H 12200 8880 30  0001 L CNN
-	1    6100 4400
-	1    0    0    1
-$EndComp
-$Comp
-L NODEMARKER_PSPICE nodeMarker
-U 1 1 76465782
-P 2100 2700
-F 0 "nodeMarker" H 4200 5400 30  0001 L CNN
-F 1 "nodeMarker" H 4200 5480 30  0001 L CNN
-	1    2100 2700
-	1    0    0    1
-$EndComp
 Wire Wire Line

Commit message: Ports issue fixed. Now annotation for ports is #PWR? function added "itos"
Parts:
- removed EGND (x2): EGND, symbol EGND_PSPICE
Changed lines of the file:
@@
 $EndDescr
 $Comp
-L EGND_PSPICE EGND
+L EGND_PSPICE #PWR1
 U 1 1 14289383
 P 3400 4800
-F 0 "EGND" H 6800 9600 30  0001 L CNN
+F 0 "#PWR1" H 6800 9600 30  0001 L CNN
 F 1 "EGND" H 6800 9680 30  0001 L CNN
 	1    3400 4800
@@
 $EndComp
 $Comp
-L EGND_PSPICE EGND
+L EGND_PSPICE #PWR2
 U 1 1 46930886
 P 4800 4900
-F 0 "EGND" H 9600 9800 30  0001 L CNN
+F 0 "#PWR2" H 9600 9800 30  0001 L CNN
 F 1 "EGND" H 9600 9880 30  0001 L CNN
 	1    4800 4900

Commit message: Added LICENSE.txt
Changed lines of the file:
@@
 $EndDescr
 $Comp
-L EGND_PSPICE #PWR1
+L GND #PWR1
 U 1 1 14289383
 P 3400 4800
@@
 $EndComp
 $Comp
-L EGND_PSPICE #PWR2
+L GND #PWR2
 U 1 1 46930886
 P 4800 4900

Commit message: Orientation fix. Library components are now inverted, with +ve y axis going up. In Schematic files, +ve y axis is downwards. This is how the KiCad libraries are. As a result of the above fixed, the converted GND is now oriented correctly.
Other:
- moved on the sheet: L1, V1, V2
Changed lines of the file:
@@
 F 1 "EGND" H 6800 9680 30  0001 L CNN
 	1    3400 4800
-	1    0    0    1
+	1    0    0    -1
 $EndComp
 $Comp
@@
 F 1 "EGND" H 9600 9880 30  0001 L CNN
 	1    4800 4900
-	1    0    0    1
+	1    0    0    -1
 $EndComp
 $Comp
@@
 F 1 "D1N4148" H 4300 2780 30  0000 L CNN
 	1    4300 2700
-	1    0    0    1
+	1    0    0    -1
 $EndComp
 $Comp
@@
 F 1 "D1N4148" H 4600 4080 30  0000 L CNN
 	1    4600 4000
-	-1    0    0    -1
+	-1    0    0    1
 $EndComp
 $Comp
@@
 F 1 "33mH" H 3700 4550 30  0000 L CNN
 	1    3700 4400
-	1    0    0    1
+	1    0    0    -1
 $EndComp
 $Comp
@@
 F 1 "0.022uF" H 3600 3270 30  0000 L CNN
 	1    3600 3200
-	0    -1    1    0
+	0    1    1    0
 $EndComp
 $Comp
@@
 F 1 "0.01uF" H 4100 3610 30  0000 L CNN
 	1    4100 3300
-	0    -1    1    0
+	0    1    1    0
 $EndComp
 $Comp
@@
 F 1 "10k" H 5700 3550 30  0000 L CNN
 	1    5700 3400
-	0    -1    1    0
+	0    1    1    0
 $EndComp
 $Comp
@@
 F 1 "10k" H 5700 2850 30  0000 L CNN
 	1    5700 2700
-	0    -1    1    0
+	0    1    1    0
 $EndComp
 $Comp
@@
 F 1 "0.1uF" H 6200 3510 30  0000 L CNN
 	1    6200 3200
-	0    -1    1    0
+	0    1    1    0
 $EndComp
 $Comp
@@
 F 1 "10n" H 5100 3730 30  0000 L CNN
 	1    5100 3400
-	0    -1    1    0
+	0    1    1    0
 $EndComp
 $Comp
@@
 F 1 "10n" H 5100 3010 30  0000 L CNN
 	1    5100 2700
-	0    -1    1    0
+	0    1    1    0
 $EndComp
 $Comp
@@
 F 1 "47uF" H 4800 4790 30  0000 L CNN
 	1    4800 4600
-	0    -1    1    0
+	0    1    1    0
 $EndComp
 $Comp
@@
 F 1 "100meg" H 4200 5250 30  0000 L CNN
 	1    4200 5200
-	1    0    0    1
+	1    0    0    -1
 $EndComp
 $Comp
@@
 F 1 "100meg" H 3000 4690 30  0000 L CNN
 	1    3000 4800
-	1    0    0    1
+	1    0    0    -1
 $EndComp
 $Comp
@@
 F 1 "VSFFM" H 3000 3580 30  0000 L CNN
 	1    3000 3500
-	-1    0    0    1
+	-1    0    0    -1
 $EndComp
 $Comp
@@
 F 1 "VSFFM" H 3000 2880 30  0000 L CNN
 	1    3000 2800
-	-1    0    0    1
+	-1    0    0    -1
 $EndComp
 $Comp
@@
 F 1 "1K" H 5300 4530 30  0000 L CNN
 	1    5300 4400
-	1    0    0    1
+	1    0    0    -1
 $EndComp
 $Comp
@@
 F 1 "0.22U" H 2200 3350 30  0000 L CNN
 	1    2200 3400
-	1    0    0    1
+	1    0    0    -1
 $EndComp
 $Comp
@@
 F 1 "0.047NF" H 6100 4730 30  0000 L CNN
 	1    6100 4500
-	0    -1    1    0
+	0    1    1    0
 $EndComp
 Wire Wire Line

Commit message: Removed the use of exec, wrote basename function, made integration with eSim easier.
Parts:
- added C6: 0.047NF, symbol C_PSPICE
- added C8: 0.22U, symbol C_PSPICE
- added nodeMarker (x2): nodeMarker, symbol nodeMarker_PSPICE
- added titleblk: titleblk, symbol titleblk_PSPICE
- PM1: renamed from C8; value 0.22U -> PARAM; symbol C_PSPICE -> PARAM_PSPICE
- PM2: renamed from V2; value VSFFM -> PARAM; symbol VSFFM_PSPICE -> PARAM_PSPICE
- R3: renamed from C6; value 0.047NF -> 1K; symbol C_PSPICE -> R_PSPICE
- V1: renamed from R3; value 1K -> VSFFM; symbol R_PSPICE -> VSFFM_PSPICE
- renumbered V1 to V2
Other:
- moved on the sheet: V2
Changed lines of the file:
@@
-EESchema Schematic File Version 2  date Wednesday 08 March 2000 03:32:15 AM IST
+EESchema Schematic File Version 2  date
 LIBS:power
 LIBS:device
@@
 LIBS:contrib
 LIBS:valves
-LIBS:ConvertedSchematicFiles/EXP6_12-cache
 EELAYER 25  0
 EELAYER END
@@
 Sheet 1 1
 Title ""
-Date "08 Mar 2000"
+Date ""
 Rev ""
 Comp ""
@@
 $EndComp
 $Comp
+L PARAM_PSPICE PM2
+U 1 1 87513926
+P 7300 3300
+F 0 "PM2" H 7300 3300 30  0000 L CNN
+F 1 "PARAM" H 7300 3380 30  0000 L CNN
+	1    7300 3300
+	1    0    0    -1
+$EndComp
+$Comp
 L VSFFM_PSPICE V2
-U 1 1 87513926
+U 1 1 25180540
 P 3000 3500
 F 0 "V2" H 3000 3500 30  0000 L CNN
@@
 $Comp
 L VSFFM_PSPICE V1
-U 1 1 25180540
+U 1 1 20383426
 P 3000 2800
 F 0 "V1" H 3000 2800 30  0000 L CNN
@@
 $EndComp
 $Comp
+L PARAM_PSPICE PM1
+U 1 1 44089172
+P 7300 2700
+F 0 "PM1" H 7300 2700 30  0000 L CNN
+F 1 "PARAM" H 7300 2780 30  0000 L CNN
+	1    7300 2700
+	1    0    0    -1
+$EndComp
+$Comp
 L R_PSPICE R3
-U 1 1 20383426
+U 1 1 53455736
 P 5300 4400
 F 0 "R3" H 5300 4400 30  0000 L CNN
@@
 $Comp
 L C_PSPICE C8
-U 1 1 44089172
+U 1 1 45005211
 P 2200 3400
 F 0 "C8" H 2200 3400 30  0000 L CNN
@@
 $Comp
 L C_PSPICE C6
-U 1 1 53455736
+U 1 1 81595368
 P 6100 4500
 F 0 "C6" H 6100 4500 30  0000 L CNN
@@
 	0    1    1    0
 $EndComp
+$Comp
+L titleblk_PSPICE titleblk
+U 1 1 34702567
+P 11880 8400
+F 0 "titleblk" H 23760 16800 30  0001 L CNN
+F 1 "titleblk" H 23760 16880 30  0001 L CNN
+	1    11880 8400
+	1    0    0    -1
+$EndComp
+$Comp
+L nodeMarker_PSPICE nodeMarker
+U 1 1 26956429
+P 6100 4400
+F 0 "nodeMarker" H 12200 8800 30  0001 L CNN
+F 1 "nodeMarker" H 12200 8880 30  0001 L CNN
+	1    6100 4400
+	1    0    0    -1
+$EndComp
+$Comp
+L nodeMarker_PSPICE nodeMarker
+U 1 1 76465782
+P 2100 2700
+F 0 "nodeMarker" H 4200 5400 30  0001 L CNN
+F 1 "nodeMarker" H 4200 5480 30  0001 L CNN
+	1    2100 2700
+	1    0    0    -1
+$EndComp
 Wire Wire Line
