File: ConvertedSchematicFiles/EXP6_9/EXP6_9.sch (KiCad schematic (older format))
At the start: 35 parts, among them U1 uA741, U2 uA741, U3 OP_AMP

Commit message: Excluded some components. These no longer appear after conversion. When calling shell commands, filenames are in "quotes"
Parts:
- removed PM2: PARAM, symbol PARAM_PSPICE
- removed R13: 10k, symbol R_PSPICE
- removed titleblk: titleblk, symbol TITLEBLK_PSPICE
- R13: renamed from PM1; value PARAM -> 10k; symbol PARAM_PSPICE -> R_PSPICE
Connections:
- net at GND_ANALOG.AGND: now also R13.1
- net at R9.2: now also R13.2
Changed lines of the file:
@@
-$EndComp
-$Comp
-L PARAM_PSPICE PM1
-U 1 1 11979802
-P 1500 2000
-F 0 "PM1" H 1500 2000 30  0000 L CNN
-F 1 "PARAM" H 1500 2080 30  0000 L CNN
-	1    1500 2000
-	1    0    0    1
-$EndComp
-$Comp
-L PARAM_PSPICE PM2
-U 1 1 65634022
-P 1400 5300
-F 0 "PM2" H 1400 5300 30  0000 L CNN
-F 1 "PARAM" H 1400 5380 30  0000 L CNN
-	1    1400 5300
-	1    0    0    1
 $EndComp
 $Comp
 L R_PSPICE R13
-U 1 1 15723058
+U 1 1 11979802
 P 8200 4000
 F 0 "R13" H 8200 4000 30  0001 L CNN
@@
 	0    1    -1    0
 $EndComp
-$Comp
-L TITLEBLK_PSPICE titleblk
-U 1 1 29133069
-P 11880 8400
-F 0 "titleblk" H 23760 16800 30  0001 L CNN
-F 1 "titleblk" H 23760 16880 30  0001 L CNN
-	1    11880 8400
-	1    0    0    1
-$EndComp
 Wire Wire Line

Commit message: Ports issue fixed. Now annotation for ports is #PWR? function added "itos"
Parts:
- removed EGND: EGND, symbol EGND_PSPICE
- removed GND_ANALOG (x10): GND_ANALOG, symbol GND_ANALOG_PSPICE
Changed lines of the file:
@@
 $EndDescr
 $Comp
-L GND_ANALOG_PSPICE GND_ANALOG
+L GND_ANALOG_PSPICE #PWR1
 U 1 1 14289383
 P 5000 2300
-F 0 "GND_ANALOG" H 10000 4600 30  0001 L CNN
+F 0 "#PWR1" H 10000 4600 30  0001 L CNN
 F 1 "GND_ANALOG" H 10000 4680 30  0001 L CNN
 	1    5000 2300
@@
 $EndComp
 $Comp
-L GND_ANALOG_PSPICE GND_ANALOG
+L GND_ANALOG_PSPICE #PWR2
 U 1 1 46930886
 P 4200 3500
-F 0 "GND_ANALOG" H 8400 7000 30  0001 L CNN
+F 0 "#PWR2" H 8400 7000 30  0001 L CNN
 F 1 "GND_ANALOG" H 8400 7080 30  0001 L CNN
 	1    4200 3500
@@
 $EndComp
 $Comp
-L GND_ANALOG_PSPICE GND_ANALOG
+L GND_ANALOG_PSPICE #PWR3
 U 1 1 71692777
 P 2600 1600
-F 0 "GND_ANALOG" H 5200 3200 30  0001 L CNN
+F 0 "#PWR3" H 5200 3200 30  0001 L CNN
 F 1 "GND_ANALOG" H 5200 3280 30  0001 L CNN
 	1    2600 1600
@@
 $EndComp
 $Comp
-L GND_ANALOG_PSPICE GND_ANALOG
+L GND_ANALOG_PSPICE #PWR4
 U 1 1 14636915
 P 3200 3600
-F 0 "GND_ANALOG" H 6400 7200 30  0001 L CNN
+F 0 "#PWR4" H 6400 7200 30  0001 L CNN
 F 1 "GND_ANALOG" H 6400 7280 30  0001 L CNN
 	1    3200 3600
@@
 $EndComp
 $Comp
-L GND_ANALOG_PSPICE GND_ANALOG
+L GND_ANALOG_PSPICE #PWR5
 U 1 1 77747793
 P 5200 4700
-F 0 "GND_ANALOG" H 10400 9400 30  0001 L CNN
+F 0 "#PWR5" H 10400 9400 30  0001 L CNN
 F 1 "GND_ANALOG" H 10400 9480 30  0001 L CNN
 	1    5200 4700
@@
 $EndComp
 $Comp
-L GND_ANALOG_PSPICE GND_ANALOG
+L GND_ANALOG_PSPICE #PWR6
 U 1 1 74238335
 P 4400 5900
-F 0 "GND_ANALOG" H 8800 11800 30  0001 L CNN
+F 0 "#PWR6" H 8800 11800 30  0001 L CNN
 F 1 "GND_ANALOG" H 8800 11880 30  0001 L CNN
 	1    4400 5900
@@
 $EndComp
 $Comp
-L GND_ANALOG_PSPICE GND_ANALOG
+L GND_ANALOG_PSPICE #PWR7
 U 1 1 99885386
 P 3500 6000
-F 0 "GND_ANALOG" H 7000 12000 30  0001 L CNN
+F 0 "#PWR7" H 7000 12000 30  0001 L CNN
 F 1 "GND_ANALOG" H 7000 12080 30  0001 L CNN
 	1    3500 6000
@@
 $EndComp
 $Comp
-L GND_ANALOG_PSPICE GND_ANALOG
+L GND_ANALOG_PSPICE #PWR8
 U 1 1 39760492
 P 6300 4100
-F 0 "GND_ANALOG" H 12600 8200 30  0001 L CNN
+F 0 "#PWR8" H 12600 8200 30  0001 L CNN
 F 1 "GND_ANALOG" H 12600 8280 30  0001 L CNN
 	1    6300 4100
@@
 $EndComp
 $Comp
-L GND_ANALOG_PSPICE GND_ANALOG
+L GND_ANALOG_PSPICE #PWR9
 U 1 1 66516649
 P 8200 4000
-F 0 "GND_ANALOG" H 16400 8000 30  0001 L CNN
+F 0 "#PWR9" H 16400 8000 30  0001 L CNN
 F 1 "GND_ANALOG" H 16400 8080 30  0001 L CNN
 	1    8200 4000
@@
 $EndComp
 $Comp
-L EGND_PSPICE EGND
+L EGND_PSPICE #PWR10
 U 1 1 29641421
 P 2000 3800
-F 0 "EGND" H 4000 7600 30  0001 L CNN
+F 0 "#PWR10" H 4000 7600 30  0001 L CNN
 F 1 "EGND" H 4000 7680 30  0001 L CNN
 	1    2000 3800
@@
 $EndComp
 $Comp
-L GND_ANALOG_PSPICE GND_ANALOG
+L GND_ANALOG_PSPICE #PWR11
 U 1 1 45202362
 P 3000 4200
-F 0 "GND_ANALOG" H 6000 8400 30  0001 L CNN
+F 0 "#PWR11" H 6000 8400 30  0001 L CNN
 F 1 "GND_ANALOG" H 6000 8480 30  0001 L CNN
 	1    3000 4200

Commit message: Added LICENSE.txt
Parts:
- V2: value VAC -> AC
Changed lines of the file:
@@
 $EndDescr
 $Comp
-L GND_ANALOG_PSPICE #PWR1
+L AGND #PWR1
 U 1 1 14289383
 P 5000 2300
@@
 $EndComp
 $Comp
-L GND_ANALOG_PSPICE #PWR2
+L AGND #PWR2
 U 1 1 46930886
 P 4200 3500
@@
 $EndComp
 $Comp
-L GND_ANALOG_PSPICE #PWR3
+L AGND #PWR3
 U 1 1 71692777
 P 2600 1600
@@
 $EndComp
 $Comp
-L GND_ANALOG_PSPICE #PWR4
+L AGND #PWR4
 U 1 1 14636915
 P 3200 3600
@@
 $EndComp
 $Comp
-L GND_ANALOG_PSPICE #PWR5
+L AGND #PWR5
 U 1 1 77747793
 P 5200 4700
@@
 $EndComp
 $Comp
-L GND_ANALOG_PSPICE #PWR6
+L AGND #PWR6
 U 1 1 74238335
 P 4400 5900
@@
 $EndComp
 $Comp
-L GND_ANALOG_PSPICE #PWR7
+L AGND #PWR7
 U 1 1 99885386
 P 3500 6000
@@
 $EndComp
 $Comp
-L GND_ANALOG_PSPICE #PWR8
+L AGND #PWR8
 U 1 1 39760492
 P 6300 4100
@@
 $EndComp
 $Comp
-L GND_ANALOG_PSPICE #PWR9
+L AGND #PWR9
 U 1 1 66516649
 P 8200 4000
@@
 $EndComp
 $Comp
-L EGND_PSPICE #PWR10
+L GND #PWR10
 U 1 1 29641421
 P 2000 3800
@@
 $EndComp
 $Comp
-L GND_ANALOG_PSPICE #PWR11
+L AGND #PWR11
 U 1 1 45202362
 P 3000 4200
@@
 P 2000 3200
 F 0 "V2" H 2000 3200 30  0000 L CNN
-F 1 "VAC" H 2000 3280 30  0000 L CNN
+F 1 "AC" H 2000 3280 30  0000 L CNN
 	1    2000 3200
 	1    0    0    1

Commit message: Orientation fix. Library components are now inverted, with +ve y axis going up. In Schematic files, +ve y axis is downwards. This is how the KiCad libraries are. As a result of the above fixed, the converted GND is now oriented correctly.
Other:
- moved on the sheet: U3, V2
Changed lines of the file:
@@
 F 1 "GND_ANALOG" H 10000 4680 30  0001 L CNN
 	1    5000 2300
-	1    0    0    1
+	1    0    0    -1
 $EndComp
 $Comp
@@
 F 1 "GND_ANALOG" H 8400 7080 30  0001 L CNN
 	1    4200 3500
-	1    0    0    1
+	1    0    0    -1
 $EndComp
 $Comp
@@
 F 1 "GND_ANALOG" H 5200 3280 30  0001 L CNN
 	1    2600 1600
-	1    0    0    1
+	1    0    0    -1
 $EndComp
 $Comp
@@
 F 1 "GND_ANALOG" H 6400 7280 30  0001 L CNN
 	1    3200 3600
-	1    0    0    1
+	1    0    0    -1
 $EndComp
 $Comp
@@
 F 1 "GND_ANALOG" H 10400 9480 30  0001 L CNN
 	1    5200 4700
-	1    0    0    1
+	1    0    0    -1
 $EndComp
 $Comp
@@
 F 1 "GND_ANALOG" H 8800 11880 30  0001 L CNN
 	1    4400 5900
-	1    0    0    1
+	1    0    0    -1
 $EndComp
 $Comp
@@
 F 1 "GND_ANALOG" H 7000 12080 30  0001 L CNN
 	1    3500 6000
-	1    0    0    1
+	1    0    0    -1
 $EndComp
 $Comp
@@
 F 1 "GND_ANALOG" H 12600 8280 30  0001 L CNN
 	1    6300 4100
-	1    0    0    1
+	1    0    0    -1
 $EndComp
 $Comp
@@
 F 1 "GND_ANALOG" H 16400 8080 30  0001 L CNN
 	1    8200 4000
-	1    0    0    1
+	1    0    0    -1
 $EndComp
 $Comp
@@
 F 1 "EGND" H 4000 7680 30  0001 L CNN
 	1    2000 3800
-	1    0    0    1
+	1    0    0    -1
 $EndComp
 $Comp
@@
 F 1 "GND_ANALOG" H 6000 8480 30  0001 L CNN
 	1    3000 4200
-	1    0    0    1
+	1    0    0    -1
 $EndComp
 $Comp
@@
 F 1 "-15V" H 4300 2190 30  0000 C CNN
 	1    4300 2200
-	0    1    -1    0
+	0    -1    -1    0
 $EndComp
 $Comp
@@
 F 1 "10k" H 4300 1750 30  0000 L CNN
 	1    4300 1600
-	1    0    0    1
+	1    0    0    -1
 $EndComp
 $Comp
@@
 F 1 "10k" H 2900 1750 30  0000 L CNN
 	1    2900 1600
-	1    0    0    1
+	1    0    0    -1
 $EndComp
 $Comp
@@
 F 1 "uA741" H 3800 2880 30  0001 L CNN
 	1    3800 2800
-	1    0    0    -1
+	1    0    0    1
 $EndComp
 $Comp
@@
 F 1 "+15v" H 4200 3430 30  0000 C CNN
 	1    4200 3100
-	1    0    0    1
+	1    0    0    -1
 $EndComp
 $Comp
@@
 F 1 "{RFH}" H 3200 3410 30  0000 L CNN
 	1    3200 3000
-	0    -1    1    0
+	0    1    1    0
 $EndComp
 $Comp
@@
 F 1 "10k" H 7100 2750 30  0000 L CNN
 	1    7100 2600
-	1    0    0    1
+	1    0    0    -1
 $EndComp
 $Comp
@@
 F 1 "10k" H 6200 2750 30  0000 L CNN
 	1    6200 2600
-	1    0    0    1
+	1    0    0    -1
 $EndComp
 $Comp
@@
 F 1 "uA741" H 4000 5280 30  0001 L CNN
 	1    4000 5200
-	1    0    0    -1
+	1    0    0    1
 $EndComp
 $Comp
@@
 F 1 "{CFL}" H 3500 5830 30  0000 L CNN
 	1    3500 5500
-	0    -1    1    0
+	0    1    1    0
 $EndComp
 $Comp
@@
 F 1 "+15v" H 4400 5870 30  0000 C CNN
 	1    4400 5500
-	1    0    0    1
+	1    0    0    -1
 $EndComp
 $Comp
@@
 F 1 "10k" H 4500 4350 30  0000 L CNN
 	1    4500 4200
-	1    0    0    1
+	1    0    0    -1
 $EndComp
 $Comp
@@
 F 1 "-15V" H 4500 4590 30  0000 C CNN
 	1    4500 4600
-	0    1    -1    0
+	0    -1    -1    0
 $EndComp
 $Comp
@@
 F 1 "10k" H 6100 3250 30  0000 L CNN
 	1    6100 3100
-	1    0    0    1
+	1    0    0    -1
 $EndComp
 $Comp
@@
 F 1 "OP_AMP" H 6700 3780 30  0000 L CNN
 	1    6700 3700
-	1    0    0    -1
+	1    0    0    1
 $EndComp
 $Comp
@@
 F 1 "2.2k" H 6300 3970 30  0000 L CNN
 	1    6300 3700
-	0    -1    1    0
+	0    1    1    0
 $EndComp
 $Comp
@@
 F 1 "AC" H 2000 3280 30  0000 L CNN
 	1    2000 3200
-	1    0    0    1
+	1    0    0    -1
 $EndComp
 $Comp
@@
 F 1 "{CFH}" H 2700 2870 30  0000 L CNN
 	1    2700 2800
-	1    0    0    1
+	1    0    0    -1
 $EndComp
 $Comp
@@
 F 1 "10k" H 3300 4350 30  0000 L CNN
 	1    3300 4200
-	1    0    0    1
+	1    0    0    -1
 $EndComp
 $Comp
@@
 F 1 "{RFL}" H 2900 5350 30  0000 L CNN
 	1    2900 5200
-	1    0    0    1
+	1    0    0    -1
 $EndComp
 $Comp
@@
 F 1 "10k" H 8200 4130 30  0000 L CNN
 	1    8200 4000
-	0    1    -1    0
+	0    -1    -1    0
 $EndComp
 Wire Wire Line

Commit message: Removed the use of exec, wrote basename function, made integration with eSim easier.
Parts:
- added PM2: PARAM, symbol PARAM_PSPICE
- added R13: 10k, symbol R_PSPICE
- added titleblk: titleblk, symbol titleblk_PSPICE
- PM1: renamed from R13; value 10k -> PARAM; symbol R_PSPICE -> PARAM_PSPICE
Changed lines of the file:
@@
-EESchema Schematic File Version 2  date Wednesday 23 June 1999 09:24:08 PM IST
+EESchema Schematic File Version 2  date
 LIBS:power
 LIBS:device
@@
 LIBS:contrib
 LIBS:valves
-LIBS:ConvertedSchematicFiles/EXP6_9-cache
 EELAYER 25  0
 EELAYER END
@@
 Sheet 1 1
 Title ""
-Date "23 Jun 1999"
+Date ""
 Rev ""
 Comp ""
@@
 $EndComp
 $Comp
+L PARAM_PSPICE PM1
+U 1 1 11979802
+P 1500 2000
+F 0 "PM1" H 1500 2000 30  0000 L CNN
+F 1 "PARAM" H 1500 2080 30  0000 L CNN
+	1    1500 2000
+	1    0    0    -1
+$EndComp
+$Comp
+L PARAM_PSPICE PM2
+U 1 1 65634022
+P 1400 5300
+F 0 "PM2" H 1400 5300 30  0000 L CNN
+F 1 "PARAM" H 1400 5380 30  0000 L CNN
+	1    1400 5300
+	1    0    0    -1
+$EndComp
+$Comp
 L R_PSPICE R13
-U 1 1 11979802
+U 1 1 15723058
 P 8200 4000
 F 0 "R13" H 8200 4000 30  0001 L CNN
@@
 	0    -1    -1    0
 $EndComp
+$Comp
+L titleblk_PSPICE titleblk
+U 1 1 29133069
+P 11880 8400
+F 0 "titleblk" H 23760 16800 30  0001 L CNN
+F 1 "titleblk" H 23760 16880 30  0001 L CNN
+	1    11880 8400
+	1    0    0    -1
+$EndComp
 Wire Wire Line
