File: ConvertedSchematicFiles/EXP7_13/EXP7_13.sch (KiCad schematic (older format))
At the start: 11 parts, among them U1 SCR2T, U2 SCR2T

Commit message: Excluded some components. These no longer appear after conversion. When calling shell commands, filenames are in "quotes"
Parts:
- removed U1, U2: SCR2T, symbol SCR2T_PSPICE
- removed titleblk: titleblk, symbol TITLEBLK_PSPICE
- U1: renamed from PM2; value PARAM -> SCR2T; symbol PARAM_PSPICE -> SCR2T_PSPICE
- U2: renamed from PM3; value PARAM -> SCR2T; symbol PARAM_PSPICE -> SCR2T_PSPICE
Connections:
- net at D1.2, VIN.+, VIN.-: now also U1.A
- net at D2.2: now also U2.A
- net at R1.1: now also U1.K, U2.K
Changed lines of the file:
@@
-$EndComp
-$Comp
-L PARAM_PSPICE PM2
-U 1 1 99885386
-P 5300 2700
-F 0 "PM2" H 5300 2700 30  0000 L CNN
-F 1 "PARAM" H 5300 2780 30  0000 L CNN
-	1    5300 2700
-	1    0    0    1
-$EndComp
-$Comp
-L PARAM_PSPICE PM3
-U 1 1 39760492
-P 5300 1800
-F 0 "PM3" H 5300 1800 30  0001 L CNN
-F 1 "PARAM" H 5300 1880 30  0001 L CNN
-	1    5300 1800
-	1    0    0    1
 $EndComp
 $Comp
 L SCR2T_PSPICE U1
-U 1 1 66516649
+U 1 1 99885386
 P 1800 2000
 F 0 "U1" H 1800 2000 30  0000 L CNN
@@
 $Comp
 L SCR2T_PSPICE U2
-U 1 1 29641421
+U 1 1 39760492
 P 3000 2000
 F 0 "U2" H 3000 2000 30  0000 L CNN
@@
 	0    1    -1    0
 $EndComp
-$Comp
-L TITLEBLK_PSPICE titleblk
-U 1 1 45202362
-P 9700 7200
-F 0 "titleblk" H 19400 14400 30  0001 L CNN
-F 1 "titleblk" H 19400 14480 30  0001 L CNN
-	1    9700 7200
-	1    0    0    1
-$EndComp
 Wire Wire Line

Commit message: Ports issue fixed. Now annotation for ports is #PWR? function added "itos"
Parts:
- removed EGND: EGND, symbol EGND_PSPICE
Changed lines of the file:
@@
 $EndDescr
 $Comp
-L EGND_PSPICE EGND
+L EGND_PSPICE #PWR1
 U 1 1 14289383
 P 3900 3100
-F 0 "EGND" H 7800 6200 30  0001 L CNN
+F 0 "#PWR1" H 7800 6200 30  0001 L CNN
 F 1 "EGND" H 7800 6280 30  0001 L CNN
 	1    3900 3100

Commit message: Added LICENSE.txt
Changed lines of the file:
@@
 $EndDescr
 $Comp
-L EGND_PSPICE #PWR1
+L GND #PWR1
 U 1 1 14289383
 P 3900 3100

Commit message: Orientation fix. Library components are now inverted, with +ve y axis going up. In Schematic files, +ve y axis is downwards. This is how the KiCad libraries are. As a result of the above fixed, the converted GND is now oriented correctly.
Parts:
- VIN: value VSIN -> SINE
Changed lines of the file:
@@
 F 1 "EGND" H 7800 6280 30  0001 L CNN
 	1    3900 3100
-	1    0    0    1
+	1    0    0    -1
 $EndComp
 $Comp
@@
 F 1 "100" H 3900 1770 30  0000 L CNN
 	1    3900 1500
-	0    -1    1    0
+	0    1    1    0
 $EndComp
 $Comp
@@
 F 1 "50mh" H 3900 2430 30  0000 L CNN
 	1    3900 2000
-	0    -1    1    0
+	0    1    1    0
 $EndComp
 $Comp
@@
 F 1 "D1N914" H 1800 2980 30  0000 L CNN
 	1    1800 2900
-	0    1    -1    0
+	0    -1    -1    0
 $EndComp
 $Comp
@@
 F 1 "D1N914" H 3000 2980 30  0000 L CNN
 	1    3000 2900
-	0    1    -1    0
+	0    -1    -1    0
 $EndComp
 $Comp
@@
 P 2200 2300
 F 0 "VIN" H 2200 2300 30  0001 L CNN
-F 1 "VSIN" H 2200 2380 30  0001 L CNN
+F 1 "SINE" H 2200 2380 30  0001 L CNN
 	1    2200 2300
-	0    1    -1    0
+	0    -1    -1    0
 $EndComp
 $Comp
@@
 F 1 "SCR2T" H 1800 2080 30  0000 L CNN
 	1    1800 2000
-	0    1    -1    0
+	0    -1    -1    0
 $EndComp
 $Comp
@@
 F 1 "SCR2T" H 3000 2080 30  0000 L CNN
 	1    3000 2000
-	0    1    -1    0
+	0    -1    -1    0
 $EndComp
 Wire Wire Line

Commit message: Removed the use of exec, wrote basename function, made integration with eSim easier.
Parts:
- added U1, U2: SCR2T, symbol SCR2T_PSPICE
- added titleblk: titleblk, symbol titleblk_PSPICE
- PM2: renamed from U1; value SCR2T -> PARAM; symbol SCR2T_PSPICE -> PARAM_PSPICE
- PM3: renamed from U2; value SCR2T -> PARAM; symbol SCR2T_PSPICE -> PARAM_PSPICE
Changed lines of the file:
@@
-EESchema Schematic File Version 2  date Tuesday 07 March 2000 09:29:35 PM IST
+EESchema Schematic File Version 2  date
 LIBS:power
 LIBS:device
@@
 LIBS:contrib
 LIBS:valves
-LIBS:ConvertedSchematicFiles/EXP7_13-cache
 EELAYER 25  0
 EELAYER END
@@
 Sheet 1 1
 Title ""
-Date "07 Mar 2000"
+Date ""
 Rev ""
 Comp ""
@@
 $EndComp
 $Comp
+L PARAM_PSPICE PM2
+U 1 1 99885386
+P 5300 2700
+F 0 "PM2" H 5300 2700 30  0000 L CNN
+F 1 "PARAM" H 5300 2780 30  0000 L CNN
+	1    5300 2700
+	1    0    0    -1
+$EndComp
+$Comp
+L PARAM_PSPICE PM3
+U 1 1 39760492
+P 5300 1800
+F 0 "PM3" H 5300 1800 30  0001 L CNN
+F 1 "PARAM" H 5300 1880 30  0001 L CNN
+	1    5300 1800
+	1    0    0    -1
+$EndComp
+$Comp
 L SCR2T_PSPICE U1
-U 1 1 99885386
+U 1 1 66516649
 P 1800 2000
 F 0 "U1" H 1800 2000 30  0000 L CNN
@@
 $Comp
 L SCR2T_PSPICE U2
-U 1 1 39760492
+U 1 1 29641421
 P 3000 2000
 F 0 "U2" H 3000 2000 30  0000 L CNN
@@
 	0    -1    -1    0
 $EndComp
+$Comp
+L titleblk_PSPICE titleblk
+U 1 1 45202362
+P 9700 7200
+F 0 "titleblk" H 19400 14400 30  0001 L CNN
+F 1 "titleblk" H 19400 14480 30  0001 L CNN
+	1    9700 7200
+	1    0    0    -1
+$EndComp
 Wire Wire Line
