File: ConvertedSchematicFiles/EXP7_4/EXP7_4.sch (KiCad schematic (older format))
At the start: 20 parts, among them Q19 Q2N3904

Commit message: Excluded some components. These no longer appear after conversion. When calling shell commands, filenames are in "quotes"
Parts:
- removed C11: {Cf}, symbol C_PSPICE
- removed titleblk: titleblk, symbol TITLEBLK_PSPICE
- C7: renamed from Q19; value Q2N3904 -> {Cf}; symbol Q2N3904_PSPICE -> C_PSPICE
- Q19: renamed from R10; value 6.8k -> Q2N3904; symbol R_PSPICE -> Q2N3904_PSPICE
- R10: renamed from PM1; value PARAM -> 6.8k; symbol PARAM_PSPICE -> R_PSPICE
- renumbered C7 to C10, C10 to C11
Connections:
- net at C10.2, C11.1: now also R7.2; no longer R6.2
- net at C11.2: now also R8.2; no longer R7.2
- net at C7.1, Rc1.1, V1.-: now also Q19.1; no longer C10.1
- net at R1.1, R8.1, R9.1: now also Q19.2; no longer C7.2
- net at C12.2, EGND.EGND: now also R10.2; no longer Q19.2
- new net: C10.1, C7.2, R6.2
- new net: C12.1, Q19.3, R10.1
Changed lines of the file:
@@
-$EndComp
-$Comp
-L PARAM_PSPICE PM1
-U 1 1 32520059
-P 5500 400
-F 0 "PM1" H 5500 400 30  0001 L CNN
-F 1 "PARAM" H 5500 480 30  0001 L CNN
-	1    5500 400
-	1    0    0    1
 $EndComp
 $Comp
 L R_PSPICE R10
-U 1 1 74897763
+U 1 1 32520059
 P 3600 1700
 F 0 "R10" H 3600 1700 30  0000 L CNN
@@
 $Comp
 L Q2N3904_PSPICE Q19
-U 1 1 87513926
+U 1 1 74897763
 P 3400 1500
 F 0 "Q19" H 3400 1500 30  0000 L CNN
@@
 $Comp
 L C_PSPICE C7
-U 1 1 25180540
+U 1 1 87513926
 P 4100 1200
 F 0 "C7" H 4100 1200 30  0001 L CNN
@@
 $Comp
 L C_PSPICE C10
-U 1 1 20383426
+U 1 1 25180540
 P 4800 1200
 F 0 "C10" H 4800 1200 30  0001 L CNN
@@
 $Comp
 L C_PSPICE C11
-U 1 1 44089172
+U 1 1 20383426
 P 5400 1200
 F 0 "C11" H 5400 1200 30  0001 L CNN
@@
 	1    0    0    1
 $EndComp
-$Comp
-L TITLEBLK_PSPICE titleblk
-U 1 1 53455736
-P 9700 7200
-F 0 "titleblk" H 19400 14400 30  0001 L CNN
-F 1 "titleblk" H 19400 14480 30  0001 L CNN
-	1    9700 7200
-	1    0    0    1
-$EndComp

Commit message: Ports issue fixed. Now annotation for ports is #PWR? function added "itos"
Parts:
- removed EGND (x3): EGND, symbol EGND_PSPICE
- removed GND_EARTH (x2): GND_EARTH, symbol GND_EARTH_PSPICE
Changed lines of the file:
@@
 $EndDescr
 $Comp
-L EGND_PSPICE EGND
+L EGND_PSPICE #PWR1
 U 1 1 14289383
 P 4000 200
-F 0 "EGND" H 8000 400 30  0001 L CNN
+F 0 "#PWR1" H 8000 400 30  0001 L CNN
 F 1 "EGND" H 8000 480 30  0001 L CNN
 	1    4000 200
@@
 $EndComp
 $Comp
-L GND_EARTH_PSPICE GND_EARTH
+L GND_EARTH_PSPICE #PWR2
 U 1 1 46930886
 P 4700 1600
-F 0 "GND_EARTH" H 9400 3200 30  0001 L CNN
+F 0 "#PWR2" H 9400 3200 30  0001 L CNN
 F 1 "GND_EARTH" H 9400 3280 30  0001 L CNN
 	1    4700 1600
@@
 $EndComp
 $Comp
-L GND_EARTH_PSPICE GND_EARTH
+L GND_EARTH_PSPICE #PWR3
 U 1 1 71692777
 P 5300 1600
-F 0 "GND_EARTH" H 10600 3200 30  0001 L CNN
+F 0 "#PWR3" H 10600 3200 30  0001 L CNN
 F 1 "GND_EARTH" H 10600 3280 30  0001 L CNN
 	1    5300 1600
@@
 $EndComp
 $Comp
-L EGND_PSPICE EGND
+L EGND_PSPICE #PWR4
 U 1 1 14636915
 P 2900 1900
-F 0 "EGND" H 5800 3800 30  0001 L CNN
+F 0 "#PWR4" H 5800 3800 30  0001 L CNN
 F 1 "EGND" H 5800 3880 30  0001 L CNN
 	1    2900 1900
@@
 $EndComp
 $Comp
-L EGND_PSPICE EGND
+L EGND_PSPICE #PWR5
 U 1 1 77747793
 P 3600 2100
-F 0 "EGND" H 7200 4200 30  0001 L CNN
+F 0 "#PWR5" H 7200 4200 30  0001 L CNN
 F 1 "EGND" H 7200 4280 30  0001 L CNN
 	1    3600 2100

Commit message: Added LICENSE.txt
Changed lines of the file:
@@
 $EndDescr
 $Comp
-L EGND_PSPICE #PWR1
+L GND #PWR1
 U 1 1 14289383
 P 4000 200
@@
 $EndComp
 $Comp
-L GND_EARTH_PSPICE #PWR2
+L GND #PWR2
 U 1 1 46930886
 P 4700 1600
@@
 $EndComp
 $Comp
-L GND_EARTH_PSPICE #PWR3
+L GND #PWR3
 U 1 1 71692777
 P 5300 1600
@@
 $EndComp
 $Comp
-L EGND_PSPICE #PWR4
+L GND #PWR4
 U 1 1 14636915
 P 2900 1900
@@
 $EndComp
 $Comp
-L EGND_PSPICE #PWR5
+L GND #PWR5
 U 1 1 77747793
 P 3600 2100

Commit message: Orientation fix. Library components are now inverted, with +ve y axis going up. In Schematic files, +ve y axis is downwards. This is how the KiCad libraries are. As a result of the above fixed, the converted GND is now oriented correctly.
Changed lines of the file:
@@
 F 1 "EGND" H 8000 480 30  0001 L CNN
 	1    4000 200
-	1    0    0    1
+	1    0    0    -1
 $EndComp
 $Comp
@@
 F 1 "GND_EARTH" H 9400 3280 30  0001 L CNN
 	1    4700 1600
-	1    0    0    1
+	1    0    0    -1
 $EndComp
 $Comp
@@
 F 1 "GND_EARTH" H 10600 3280 30  0001 L CNN
 	1    5300 1600
-	1    0    0    1
+	1    0    0    -1
 $EndComp
 $Comp
@@
 F 1 "EGND" H 5800 3880 30  0001 L CNN
 	1    2900 1900
-	1    0    0    1
+	1    0    0    -1
 $EndComp
 $Comp
@@
 F 1 "EGND" H 7200 4280 30  0001 L CNN
 	1    3600 2100
-	1    0    0    1
+	1    0    0    -1
 $EndComp
 $Comp
@@
 F 1 "{Rf}" H 5300 1630 30  0000 L CNN
 	1    5300 1600
-	0    1    -1    0
+	0    -1    -1    0
 $EndComp
 $Comp
@@
 F 1 "{Rph}" H 5800 1610 30  0000 L CNN
 	1    5800 1600
-	0    1    -1    0
+	0    -1    -1    0
 $EndComp
 $Comp
@@
 F 1 "150K" H 2900 1030 30  0000 L CNN
 	1    2900 1000
-	0    1    -1    0
+	0    -1    -1    0
 $EndComp
 $Comp
@@
 F 1 "47k" H 2900 1810 30  0000 L CNN
 	1    2900 1500
-	0    -1    1    0
+	0    1    1    0
 $EndComp
 $Comp
@@
 F 1 "15K" H 3700 1030 30  0000 L CNN
 	1    3700 1000
-	0    1    -1    0
+	0    -1    -1    0
 $EndComp
 $Comp
@@
 F 1 "2.2u" H 3900 1990 30  0000 L CNN
 	1    3900 1700
-	0    -1    1    0
+	0    1    1    0
 $EndComp
 $Comp
@@
 F 1 "{Rf}" H 4700 1630 30  0000 L CNN
 	1    4700 1600
-	0    1    -1    0
+	0    -1    -1    0
 $EndComp
 $Comp
@@
 F 1 "20v" H 3700 490 30  0000 C CNN
 	1    3700 600
-	-1    0    0    -1
+	-1    0    0    1
 $EndComp
 $Comp
@@
 F 1 "6.8k" H 3600 2050 30  0000 L CNN
 	1    3600 1700
-	0    -1    1    0
+	0    1    1    0
 $EndComp
 $Comp
@@
 F 1 "Q2N3904" H 3400 1580 30  0000 L CNN
 	1    3400 1500
-	1    0    0    1
+	1    0    0    -1
 $EndComp
 $Comp
@@
 F 1 "{Cf}" H 4100 1010 30  0000 L CNN
 	1    4100 1200
-	1    0    0    1
+	1    0    0    -1
 $EndComp
 $Comp
@@
 F 1 "{Cf}" H 4800 1210 30  0000 L CNN
 	1    4800 1200
-	1    0    0    1
+	1    0    0    -1
 $EndComp
 $Comp
@@
 F 1 "{Cf}" H 5400 1250 30  0000 L CNN
 	1    5400 1200
-	1    0    0    1
+	1    0    0    -1
 $EndComp
 Wire Wire Line

Commit message: Removed the use of exec, wrote basename function, made integration with eSim easier.
Parts:
- added C11: {Cf}, symbol C_PSPICE
- added titleblk: titleblk, symbol titleblk_PSPICE
- PM1: renamed from R10; value 6.8k -> PARAM; symbol R_PSPICE -> PARAM_PSPICE
- Q19: renamed from C7; value {Cf} -> Q2N3904; symbol C_PSPICE -> Q2N3904_PSPICE
- R10: renamed from Q19; value Q2N3904 -> 6.8k; symbol Q2N3904_PSPICE -> R_PSPICE
- renumbered C11 to C10, C10 to C7
Changed lines of the file:
@@
-EESchema Schematic File Version 2  date Wednesday 01 March 2000 10:03:05 PM IST
+EESchema Schematic File Version 2  date
 LIBS:power
 LIBS:device
@@
 LIBS:contrib
 LIBS:valves
-LIBS:ConvertedSchematicFiles/EXP7_4-cache
 EELAYER 25  0
 EELAYER END
@@
 Sheet 1 1
 Title ""
-Date "01 Mar 2000"
+Date ""
 Rev ""
 Comp ""
@@
 $EndComp
 $Comp
+L PARAM_PSPICE PM1
+U 1 1 32520059
+P 5500 400
+F 0 "PM1" H 5500 400 30  0001 L CNN
+F 1 "PARAM" H 5500 480 30  0001 L CNN
+	1    5500 400
+	1    0    0    -1
+$EndComp
+$Comp
 L R_PSPICE R10
-U 1 1 32520059
+U 1 1 74897763
 P 3600 1700
 F 0 "R10" H 3600 1700 30  0000 L CNN
@@
 $Comp
 L Q2N3904_PSPICE Q19
-U 1 1 74897763
+U 1 1 87513926
 P 3400 1500
 F 0 "Q19" H 3400 1500 30  0000 L CNN
@@
 $Comp
 L C_PSPICE C7
-U 1 1 87513926
+U 1 1 25180540
 P 4100 1200
 F 0 "C7" H 4100 1200 30  0001 L CNN
@@
 $Comp
 L C_PSPICE C10
-U 1 1 25180540
+U 1 1 20383426
 P 4800 1200
 F 0 "C10" H 4800 1200 30  0001 L CNN
@@
 $Comp
 L C_PSPICE C11
-U 1 1 20383426
+U 1 1 44089172
 P 5400 1200
 F 0 "C11" H 5400 1200 30  0001 L CNN
@@
 	1    0    0    -1
 $EndComp
+$Comp
+L titleblk_PSPICE titleblk
+U 1 1 53455736
+P 9700 7200
+F 0 "titleblk" H 19400 14400 30  0001 L CNN
+F 1 "titleblk" H 19400 14480 30  0001 L CNN
+	1    9700 7200
+	1    0    0    -1
+$EndComp
