File: ConvertedSchematicFiles/EXP7_6/EXP7_6.sch (KiCad schematic (older format))
At the start: 6 parts, among them U1 7474

Commit message: Excluded some components. These no longer appear after conversion. When calling shell commands, filenames are in "quotes"
Parts:
- removed titleblk: titleblk, symbol TITLEBLK_PSPICE
Changed lines of the file:
@@
-	1    0    0    1
-$EndComp
-$Comp
-L TITLEBLK_PSPICE titleblk
-U 1 1 74238335
-P 11880 8400
-F 0 "titleblk" H 23760 16800 30  0001 L CNN
-F 1 "titleblk" H 23760 16880 30  0001 L CNN
-	1    11880 8400
 	1    0    0    1
 $EndComp

Commit message: Orientation fix. Library components are now inverted, with +ve y axis going up. In Schematic files, +ve y axis is downwards. This is how the KiCad libraries are. As a result of the above fixed, the converted GND is now oriented correctly.
Connections:
- net at DSTM15.GND: now also DSTM16.PWR
- net at DSTM15.PWR: no longer DSTM16.GND
- net at DSTM11.1: now also U1.C, U1.D
Changed lines of the file:
@@
 F 1 "DigStim" H 1100 4180 30  0000 L CNN
 	1    1100 4100
-	1    0    0    1
+	1    0    0    -1
 $EndComp
 $Comp
@@
 F 1 "DigStim" H 1100 4480 30  0000 L CNN
 	1    1100 4400
-	1    0    0    1
+	1    0    0    -1
 $EndComp
 $Comp
@@
 F 1 "DigClock" H 1100 4780 30  0000 L CNN
 	1    1100 4700
-	1    0    0    1
+	1    0    0    -1
 $EndComp
 $Comp
@@
 F 1 "DigStim" H 2400 5180 30  0000 L CNN
 	1    2400 5100
-	1    0    0    1
+	1    0    0    -1
 $EndComp
 $Comp
@@
 F 1 "7474" H 2200 4480 30  0000 L CNN
 	1    2200 4400
-	1    0    0    1
+	1    0    0    -1
 $EndComp
 Wire Wire Line

Commit message: Removed the use of exec, wrote basename function, made integration with eSim easier.
Parts:
- added titleblk: titleblk, symbol titleblk_PSPICE
Changed lines of the file:
@@
-EESchema Schematic File Version 2  date Sunday 11 July 1999 10:57:59 AM IST
+EESchema Schematic File Version 2  date
 LIBS:power
 LIBS:device
@@
 LIBS:contrib
 LIBS:valves
-LIBS:ConvertedSchematicFiles/EXP7_6-cache
 EELAYER 25  0
 EELAYER END
@@
 Sheet 1 1
 Title ""
-Date "11 Jul 1999"
+Date ""
 Rev ""
 Comp ""
@@
 	1    0    0    -1
 $EndComp
+$Comp
+L titleblk_PSPICE titleblk
+U 1 1 74238335
+P 11880 8400
+F 0 "titleblk" H 23760 16800 30  0001 L CNN
+F 1 "titleblk" H 23760 16880 30  0001 L CNN
+	1    11880 8400
+	1    0    0    -1
+$EndComp
