File: ConvertedSchematicFiles/EXP8_7/EXP8_7.sch (KiCad schematic (older format))
At the start: 1 part

Commit message: Excluded some components. These no longer appear after conversion. When calling shell commands, filenames are in "quotes"
Parts:
- removed titleblk: titleblk, symbol TITLEBLK_PSPICE
Changed lines of the file:
@@
 Comment4 ""
 $EndDescr
-$Comp
-L TITLEBLK_PSPICE titleblk
-U 1 1 14289383
-P 11880 8400
-F 0 "titleblk" H 23760 16800 30  0001 L CNN
-F 1 "titleblk" H 23760 16880 30  0001 L CNN
-	1    11880 8400
-	1    0    0    1
-$EndComp
 $EndSCHEMATC

Commit message: Removed the use of exec, wrote basename function, made integration with eSim easier.
Parts:
- added titleblk: titleblk, symbol titleblk_PSPICE
Changed lines of the file:
@@
-EESchema Schematic File Version 2  date Thursday 02 March 2000 09:49:16 PM IST
+EESchema Schematic File Version 2  date
 LIBS:power
 LIBS:device
@@
 LIBS:contrib
 LIBS:valves
-LIBS:ConvertedSchematicFiles/EXP8_7-cache
 EELAYER 25  0
 EELAYER END
@@
 Sheet 1 1
 Title ""
-Date "02 Mar 2000"
+Date ""
 Rev ""
 Comp ""
@@
 Comment4 ""
 $EndDescr
+$Comp
+L titleblk_PSPICE titleblk
+U 1 1 14289383
+P 11880 8400
+F 0 "titleblk" H 23760 16800 30  0001 L CNN
+F 1 "titleblk" H 23760 16880 30  0001 L CNN
+	1    11880 8400
+	1    0    0    -1
+$EndComp
 $EndSCHEMATC
