File: ConvertedSchematicFiles/EXP8_8/EXP8_8.sch (KiCad schematic (older format))
At the start: 7 parts

Commit message: Excluded some components. These no longer appear after conversion. When calling shell commands, filenames are in "quotes"
Parts:
- removed D1: D1N4002, symbol D1N4002_PSPICE
- removed titleblk: titleblk, symbol TITLEBLK_PSPICE
- D1: renamed from R1; value R -> D1N4002; symbol R_PSPICE -> D1N4002_PSPICE
- R1: renamed from V2; value {VREF} -> R; symbol VDC_PSPICE -> R_PSPICE
- V2: renamed from PM1; value PARAM -> {VREF}; symbol PARAM_PSPICE -> VDC_PSPICE
Connections:
- net at D1.2: now also R1.1; no longer R1.+
- net at V1.+: now also D1.1
- new net: R1.2, V2.+
Changed lines of the file:
@@
-$EndComp
-$Comp
-L PARAM_PSPICE PM1
-U 1 1 71692777
-P 2500 500
-F 0 "PM1" H 2500 500 30  0000 L CNN
-F 1 "PARAM" H 2500 580 30  0000 L CNN
-	1    2500 500
-	1    0    0    1
 $EndComp
 $Comp
 L VDC_PSPICE V2
-U 1 1 14636915
+U 1 1 71692777
 P 1400 1000
 F 0 "V2" H 1400 1000 30  0000 L CNN
@@
 $Comp
 L R_PSPICE R1
-U 1 1 77747793
+U 1 1 14636915
 P 1400 500
 F 0 "R1" H 1400 500 30  0000 L CNN
@@
 $Comp
 L D1N4002_PSPICE D1
-U 1 1 74238335
+U 1 1 77747793
 P 700 500
 F 0 "D1" H 700 500 30  0000 L CNN
@@
 	1    0    0    1
 $EndComp
-$Comp
-L TITLEBLK_PSPICE titleblk
-U 1 1 99885386
-P 11880 8400
-F 0 "titleblk" H 23760 16800 30  0001 L CNN
-F 1 "titleblk" H 23760 16880 30  0001 L CNN
-	1    11880 8400
-	1    0    0    1
-$EndComp

Commit message: Ports issue fixed. Now annotation for ports is #PWR? function added "itos"
Parts:
- removed GND_EARTH: GND_EARTH, symbol GND_EARTH_PSPICE
Changed lines of the file:
@@
 $EndDescr
 $Comp
-L GND_EARTH_PSPICE GND_EARTH
+L GND_EARTH_PSPICE #PWR1
 U 1 1 14289383
 P 500 1400
-F 0 "GND_EARTH" H 1000 2800 30  0001 L CNN
+F 0 "#PWR1" H 1000 2800 30  0001 L CNN
 F 1 "GND_EARTH" H 1000 2880 30  0001 L CNN
 	1    500 1400

Commit message: Added LICENSE.txt
Changed lines of the file:
@@
 $EndDescr
 $Comp
-L GND_EARTH_PSPICE #PWR1
+L GND #PWR1
 U 1 1 14289383
 P 500 1400

Commit message: Orientation fix. Library components are now inverted, with +ve y axis going up. In Schematic files, +ve y axis is downwards. This is how the KiCad libraries are. As a result of the above fixed, the converted GND is now oriented correctly.
Parts:
- V1: value VSIN -> SINE
Other:
- moved on the sheet: V1, V2
Changed lines of the file:
@@
 F 1 "GND_EARTH" H 1000 2880 30  0001 L CNN
 	1    500 1400
-	1    0    0    1
+	1    0    0    -1
 $EndComp
 $Comp
@@
 P 500 700
 F 0 "V1" H 500 700 30  0000 L CNN
-F 1 "VSIN" H 500 780 30  0000 L CNN
+F 1 "SINE" H 500 780 30  0000 L CNN
 	1    500 700
-	1    0    0    1
+	1    0    0    -1
 $EndComp
 $Comp
@@
 F 1 "{VREF}" H 1400 1370 30  0000 C CNN
 	1    1400 1000
-	1    0    0    1
+	1    0    0    -1
 $EndComp
 $Comp
@@
 F 1 "R" H 1400 580 30  0000 L CNN
 	1    1400 500
-	0    -1    1    0
+	0    1    1    0
 $EndComp
 $Comp
@@
 F 1 "D1N4002" H 700 580 30  0000 L CNN
 	1    700 500
-	1    0    0    1
+	1    0    0    -1
 $EndComp
 Wire Wire Line

Commit message: Removed the use of exec, wrote basename function, made integration with eSim easier.
Parts:
- added D1: D1N4002, symbol D1N4002_PSPICE
- added titleblk: titleblk, symbol titleblk_PSPICE
- PM1: renamed from V2; value {VREF} -> PARAM; symbol VDC_PSPICE -> PARAM_PSPICE
- R1: renamed from D1; value D1N4002 -> R; symbol D1N4002_PSPICE -> R_PSPICE
- V2: renamed from R1; value R -> {VREF}; symbol R_PSPICE -> VDC_PSPICE
Changed lines of the file:
@@
-EESchema Schematic File Version 2  date Saturday 05 June 1999 11:13:06 PM IST
+EESchema Schematic File Version 2  date
 LIBS:power
 LIBS:device
@@
 LIBS:contrib
 LIBS:valves
-LIBS:ConvertedSchematicFiles/EXP8_8-cache
 EELAYER 25  0
 EELAYER END
@@
 Sheet 1 1
 Title ""
-Date "05 Jun 1999"
+Date ""
 Rev ""
 Comp ""
@@
 $EndComp
 $Comp
+L PARAM_PSPICE PM1
+U 1 1 71692777
+P 2500 500
+F 0 "PM1" H 2500 500 30  0000 L CNN
+F 1 "PARAM" H 2500 580 30  0000 L CNN
+	1    2500 500
+	1    0    0    -1
+$EndComp
+$Comp
 L VDC_PSPICE V2
-U 1 1 71692777
+U 1 1 14636915
 P 1400 1000
 F 0 "V2" H 1400 1000 30  0000 L CNN
@@
 $Comp
 L R_PSPICE R1
-U 1 1 14636915
+U 1 1 77747793
 P 1400 500
 F 0 "R1" H 1400 500 30  0000 L CNN
@@
 $Comp
 L D1N4002_PSPICE D1
-U 1 1 77747793
+U 1 1 74238335
 P 700 500
 F 0 "D1" H 700 500 30  0000 L CNN
@@
 	1    0    0    -1
 $EndComp
+$Comp
+L titleblk_PSPICE titleblk
+U 1 1 99885386
+P 11880 8400
+F 0 "titleblk" H 23760 16800 30  0001 L CNN
+F 1 "titleblk" H 23760 16880 30  0001 L CNN
+	1    11880 8400
+	1    0    0    -1
+$EndComp
