File: ConvertedSchematicFiles/EXP9_10/EXP9_10.sch (KiCad schematic (older format))
At the start: 17 parts, among them Q1 Q2N3904, Q2 Q2N3904

Commit message: Excluded some components. These no longer appear after conversion. When calling shell commands, filenames are in "quotes"
Parts:
- removed Q2: Q2N3904, symbol Q2N3904_PSPICE
- removed titleblk: titleblk, symbol TITLEBLK_PSPICE
- Q1: renamed from PM1; value PARAM -> Q2N3904; symbol PARAM_PSPICE -> Q2N3904_PSPICE
- renumbered Q1 to Q2
Connections:
- net at R4.2: now also Q1.2; no longer Q2.2
- net at R2.2: now also Q2.1
- net at R5.1: now also Q2.2
- net at Q2.3, R3.1, V2.-: now also Q1.3
- net at R1.2: now also Q1.1; no longer Q2.1
Other:
- moved on the sheet: Q2
Changed lines of the file:
@@
-$EndComp
-$Comp
-L PARAM_PSPICE PM1
-U 1 1 32520059
-P 4600 400
-F 0 "PM1" H 4600 400 30  0000 L CNN
-F 1 "PARAM" H 4600 480 30  0000 L CNN
-	1    4600 400
-	1    0    0    1
 $EndComp
 $Comp
 L Q2N3904_PSPICE Q1
-U 1 1 74897763
+U 1 1 32520059
 P 2000 1800
 F 0 "Q1" H 2000 1800 30  0000 L CNN
@@
 $Comp
 L Q2N3904_PSPICE Q2
-U 1 1 87513926
+U 1 1 74897763
 P 3300 1800
 F 0 "Q2" H 3300 1800 30  0000 L CNN
@@
 	-1    0    0    1
 $EndComp
-$Comp
-L TITLEBLK_PSPICE titleblk
-U 1 1 25180540
-P 9700 7200
-F 0 "titleblk" H 19400 14400 30  0001 L CNN
-F 1 "titleblk" H 19400 14480 30  0001 L CNN
-	1    9700 7200
-	1    0    0    1
-$EndComp
 Wire Wire Line

Commit message: Ports issue fixed. Now annotation for ports is #PWR? function added "itos"
Parts:
- removed EGND (x4): EGND, symbol EGND_PSPICE
Changed lines of the file:
@@
 $EndDescr
 $Comp
-L EGND_PSPICE EGND
+L EGND_PSPICE #PWR1
 U 1 1 14289383
 P 3500 900
-F 0 "EGND" H 7000 1800 30  0001 L CNN
+F 0 "#PWR1" H 7000 1800 30  0001 L CNN
 F 1 "EGND" H 7000 1880 30  0001 L CNN
 	1    3500 900
@@
 $EndComp
 $Comp
-L EGND_PSPICE EGND
+L EGND_PSPICE #PWR2
 U 1 1 46930886
 P 2700 3000
-F 0 "EGND" H 5400 6000 30  0001 L CNN
+F 0 "#PWR2" H 5400 6000 30  0001 L CNN
 F 1 "EGND" H 5400 6080 30  0001 L CNN
 	1    2700 3000
@@
 $EndComp
 $Comp
-L EGND_PSPICE EGND
+L EGND_PSPICE #PWR3
 U 1 1 71692777
 P 800 2500
-F 0 "EGND" H 1600 5000 30  0001 L CNN
+F 0 "#PWR3" H 1600 5000 30  0001 L CNN
 F 1 "EGND" H 1600 5080 30  0001 L CNN
 	1    800 2500
@@
 $EndComp
 $Comp
-L EGND_PSPICE EGND
+L EGND_PSPICE #PWR4
 U 1 1 14636915
 P 4400 2700
-F 0 "EGND" H 8800 5400 30  0001 L CNN
+F 0 "#PWR4" H 8800 5400 30  0001 L CNN
 F 1 "EGND" H 8800 5480 30  0001 L CNN
 	1    4400 2700

Commit message: Added LICENSE.txt
Changed lines of the file:
@@
 $EndDescr
 $Comp
-L EGND_PSPICE #PWR1
+L GND #PWR1
 U 1 1 14289383
 P 3500 900
@@
 $EndComp
 $Comp
-L EGND_PSPICE #PWR2
+L GND #PWR2
 U 1 1 46930886
 P 2700 3000
@@
 $EndComp
 $Comp
-L EGND_PSPICE #PWR3
+L GND #PWR3
 U 1 1 71692777
 P 800 2500
@@
 $EndComp
 $Comp
-L EGND_PSPICE #PWR4
+L GND #PWR4
 U 1 1 14636915
 P 4400 2700

Commit message: Orientation fix. Library components are now inverted, with +ve y axis going up. In Schematic files, +ve y axis is downwards. This is how the KiCad libraries are. As a result of the above fixed, the converted GND is now oriented correctly.
Parts:
- V3, V4: value VSIN -> SINE
Other:
- moved on the sheet: V1, V2, V3, V4
Changed lines of the file:
@@
 F 1 "EGND" H 7000 1880 30  0001 L CNN
 	1    3500 900
-	1    0    0    1
+	1    0    0    -1
 $EndComp
 $Comp
@@
 F 1 "EGND" H 5400 6080 30  0001 L CNN
 	1    2700 3000
-	1    0    0    1
+	1    0    0    -1
 $EndComp
 $Comp
@@
 F 1 "EGND" H 1600 5080 30  0001 L CNN
 	1    800 2500
-	1    0    0    1
+	1    0    0    -1
 $EndComp
 $Comp
@@
 F 1 "EGND" H 8800 5480 30  0001 L CNN
 	1    4400 2700
-	1    0    0    1
+	1    0    0    -1
 $EndComp
 $Comp
@@
 F 1 "-10V" H 2700 2490 30  0000 C CNN
 	1    2700 2600
-	1    0    0    1
+	1    0    0    -1
 $EndComp
 $Comp
@@
 F 1 "10V" H 3500 390 30  0000 C CNN
 	1    3500 500
-	1    0    0    1
+	1    0    0    -1
 $EndComp
 $Comp
@@
 F 1 "2.2k" H 2200 1150 30  0000 L CNN
 	1    2200 1000
-	0    -1    1    0
+	0    1    1    0
 $EndComp
 $Comp
@@
 F 1 "2.2k" H 3100 1150 30  0000 L CNN
 	1    3100 1000
-	0    -1    1    0
+	0    1    1    0
 $EndComp
 $Comp
@@
 F 1 "4.7k" H 2700 2350 30  0000 L CNN
 	1    2700 2200
-	0    -1    1    0
+	0    1    1    0
 $EndComp
 $Comp
@@
 F 1 "50" H 1200 1950 30  0000 L CNN
 	1    1200 1800
-	1    0    0    1
+	1    0    0    -1
 $EndComp
 $Comp
@@
 F 1 "50" H 3700 1950 30  0000 L CNN
 	1    3700 1800
-	1    0    0    1
+	1    0    0    -1
 $EndComp
 $Comp
@@
 P 800 2100
 F 0 "V3" H 800 2100 30  0000 L CNN
-F 1 "VSIN" H 800 2180 30  0000 L CNN
+F 1 "SINE" H 800 2180 30  0000 L CNN
 	1    800 2100
-	1    0    0    1
+	1    0    0    -1
 $EndComp
 $Comp
@@
 P 4400 2100
 F 0 "V4" H 4400 2100 30  0000 L CNN
-F 1 "VSIN" H 4400 2180 30  0000 L CNN
+F 1 "SINE" H 4400 2180 30  0000 L CNN
 	1    4400 2100
-	1    0    0    1
+	1    0    0    -1
 $EndComp
 $Comp
@@
 F 1 "Q2N3904" H 2000 1880 30  0000 L CNN
 	1    2000 1800
-	1    0    0    1
+	1    0    0    -1
 $EndComp
 $Comp
@@
 F 1 "Q2N3904" H 3300 1880 30  0000 L CNN
 	1    3300 1800
-	-1    0    0    1
+	-1    0    0    -1
 $EndComp
 Wire Wire Line

Commit message: Removed the use of exec, wrote basename function, made integration with eSim easier.
Parts:
- added Q2: Q2N3904, symbol Q2N3904_PSPICE
- added titleblk: titleblk, symbol titleblk_PSPICE
- PM1: renamed from Q1; value Q2N3904 -> PARAM; symbol Q2N3904_PSPICE -> PARAM_PSPICE
- renumbered Q2 to Q1
Other:
- moved on the sheet: Q1
Changed lines of the file:
@@
-EESchema Schematic File Version 2  date Sunday 20 June 1999 07:23:08 PM IST
+EESchema Schematic File Version 2  date
 LIBS:power
 LIBS:device
@@
 LIBS:contrib
 LIBS:valves
-LIBS:ConvertedSchematicFiles/EXP9_10-cache
 EELAYER 25  0
 EELAYER END
@@
 Sheet 1 1
 Title ""
-Date "20 Jun 1999"
+Date ""
 Rev ""
 Comp ""
@@
 $EndComp
 $Comp
+L PARAM_PSPICE PM1
+U 1 1 32520059
+P 4600 400
+F 0 "PM1" H 4600 400 30  0000 L CNN
+F 1 "PARAM" H 4600 480 30  0000 L CNN
+	1    4600 400
+	1    0    0    -1
+$EndComp
+$Comp
 L Q2N3904_PSPICE Q1
-U 1 1 32520059
+U 1 1 74897763
 P 2000 1800
 F 0 "Q1" H 2000 1800 30  0000 L CNN
@@
 $Comp
 L Q2N3904_PSPICE Q2
-U 1 1 74897763
+U 1 1 87513926
 P 3300 1800
 F 0 "Q2" H 3300 1800 30  0000 L CNN
@@
 	-1    0    0    -1
 $EndComp
+$Comp
+L titleblk_PSPICE titleblk
+U 1 1 25180540
+P 9700 7200
+F 0 "titleblk" H 19400 14400 30  0001 L CNN
+F 1 "titleblk" H 19400 14480 30  0001 L CNN
+	1    9700 7200
+	1    0    0    -1
+$EndComp
 Wire Wire Line
