File: ConvertedSchematicFiles/EXP9_11/EXP9_11.sch (KiCad schematic (older format))
At the start: 12 parts, among them U1 uA741

Commit message: Excluded some components. These no longer appear after conversion. When calling shell commands, filenames are in "quotes"
Parts:
- removed RL: {RL}, symbol R_PSPICE
- removed titleblk: titleblk, symbol TITLEBLK_PSPICE
- R2: renamed from PM1; value PARAM -> 10k; symbol PARAM_PSPICE -> R_PSPICE
- RL: renamed from U1; value uA741 -> {RL}; symbol uA741_PSPICE -> R_PSPICE
- U1: renamed from V2; value 13V -> uA741; symbol VDC_PSPICE -> uA741_PSPICE
- V1: renamed from VIN; value VSIN -> 13V; symbol VSIN_PSPICE -> VDC_PSPICE
- VIN: renamed from R2; value 10k -> VSIN; symbol R_PSPICE -> VSIN_PSPICE
- renumbered V1 to V2
Connections:
- net at GND_EARTH.EGND: now also U1.V-; no longer RL.V-
- net at GND_EARTH.EGND: now also R2.1; no longer VIN.1
- net at V1.+: no longer RL.+
- net at V2.+: now also GND_EARTH.EGND
- net at U1.+: now also VIN.+; no longer GND_EARTH.EGND
- new net: R2.2, RL.1
Changed lines of the file:
@@
-$EndComp
-$Comp
-L PARAM_PSPICE PM1
-U 1 1 77747793
-P 5600 2200
-F 0 "PM1" H 5600 2200 30  0000 L CNN
-F 1 "PARAM" H 5600 2280 30  0000 L CNN
-	1    5600 2200
-	1    0    0    1
 $EndComp
 $Comp
 L R_PSPICE R2
-U 1 1 74238335
+U 1 1 77747793
 P 2200 3200
 F 0 "R2" H 2200 3200 30  0001 L CNN
@@
 $Comp
 L VSIN_PSPICE VIN
-U 1 1 99885386
+U 1 1 74238335
 P 1800 2800
 F 0 "VIN" H 1800 2800 30  0001 L CNN
@@
 $Comp
 L VDC_PSPICE V1
-U 1 1 39760492
+U 1 1 99885386
 P 3300 2700
 F 0 "V1" H 3300 2700 30  0001 L CNN
@@
 $Comp
 L VDC_PSPICE V2
-U 1 1 66516649
+U 1 1 39760492
 P 3300 3700
 F 0 "V2" H 3300 3700 30  0001 L CNN
@@
 $Comp
 L uA741_PSPICE U1
-U 1 1 29641421
+U 1 1 66516649
 P 2900 2800
 F 0 "U1" H 2900 2800 30  0001 L CNN
@@
 $Comp
 L R_PSPICE RL
-U 1 1 45202362
+U 1 1 29641421
 P 3100 4200
 F 0 "RL" H 3100 4200 30  0001 L CNN
@@
 	1    0    0    1
 $EndComp
-$Comp
-L TITLEBLK_PSPICE titleblk
-U 1 1 10490027
-P 9700 7200
-F 0 "titleblk" H 19400 14400 30  0001 L CNN
-F 1 "titleblk" H 19400 14480 30  0001 L CNN
-	1    9700 7200
-	1    0    0    1
-$EndComp

Commit message: Ports issue fixed. Now annotation for ports is #PWR? function added "itos"
Parts:
- removed GND_EARTH (x4): GND_EARTH, symbol GND_EARTH_PSPICE
Changed lines of the file:
@@
 $EndDescr
 $Comp
-L GND_EARTH_PSPICE GND_EARTH
+L GND_EARTH_PSPICE #PWR1
 U 1 1 14289383
 P 3600 2500
-F 0 "GND_EARTH" H 7200 5000 30  0001 L CNN
+F 0 "#PWR1" H 7200 5000 30  0001 L CNN
 F 1 "GND_EARTH" H 7200 5080 30  0001 L CNN
 	1    3600 2500
@@
 $EndComp
 $Comp
-L GND_EARTH_PSPICE GND_EARTH
+L GND_EARTH_PSPICE #PWR2
 U 1 1 46930886
 P 3300 3700
-F 0 "GND_EARTH" H 6600 7400 30  0001 L CNN
+F 0 "#PWR2" H 6600 7400 30  0001 L CNN
 F 1 "GND_EARTH" H 6600 7480 30  0001 L CNN
 	1    3300 3700
@@
 $EndComp
 $Comp
-L GND_EARTH_PSPICE GND_EARTH
+L GND_EARTH_PSPICE #PWR3
 U 1 1 71692777
 P 1800 3200
-F 0 "GND_EARTH" H 3600 6400 30  0001 L CNN
+F 0 "#PWR3" H 3600 6400 30  0001 L CNN
 F 1 "GND_EARTH" H 3600 6480 30  0001 L CNN
 	1    1800 3200
@@
 $EndComp
 $Comp
-L GND_EARTH_PSPICE GND_EARTH
+L GND_EARTH_PSPICE #PWR4
 U 1 1 14636915
 P 2100 3200
-F 0 "GND_EARTH" H 4200 6400 30  0001 L CNN
+F 0 "#PWR4" H 4200 6400 30  0001 L CNN
 F 1 "GND_EARTH" H 4200 6480 30  0001 L CNN
 	1    2100 3200

Commit message: Added LICENSE.txt
Changed lines of the file:
@@
 $EndDescr
 $Comp
-L GND_EARTH_PSPICE #PWR1
+L GND #PWR1
 U 1 1 14289383
 P 3600 2500
@@
 $EndComp
 $Comp
-L GND_EARTH_PSPICE #PWR2
+L GND #PWR2
 U 1 1 46930886
 P 3300 3700
@@
 $EndComp
 $Comp
-L GND_EARTH_PSPICE #PWR3
+L GND #PWR3
 U 1 1 71692777
 P 1800 3200
@@
 $EndComp
 $Comp
-L GND_EARTH_PSPICE #PWR4
+L GND #PWR4
 U 1 1 14636915
 P 2100 3200

Commit message: Orientation fix. Library components are now inverted, with +ve y axis going up. In Schematic files, +ve y axis is downwards. This is how the KiCad libraries are. As a result of the above fixed, the converted GND is now oriented correctly.
Parts:
- VIN: value VSIN -> SINE
Changed lines of the file:
@@
 F 1 "GND_EARTH" H 7200 5080 30  0001 L CNN
 	1    3600 2500
-	1    0    0    1
+	1    0    0    -1
 $EndComp
 $Comp
@@
 F 1 "GND_EARTH" H 6600 7480 30  0001 L CNN
 	1    3300 3700
-	1    0    0    1
+	1    0    0    -1
 $EndComp
 $Comp
@@
 F 1 "GND_EARTH" H 3600 6480 30  0001 L CNN
 	1    1800 3200
-	1    0    0    1
+	1    0    0    -1
 $EndComp
 $Comp
@@
 F 1 "GND_EARTH" H 4200 6480 30  0001 L CNN
 	1    2100 3200
-	1    0    0    1
+	1    0    0    -1
 $EndComp
 $Comp
@@
 F 1 "10k" H 2200 3350 30  0000 L CNN
 	1    2200 3200
-	1    0    0    1
+	1    0    0    -1
 $EndComp
 $Comp
@@
 P 1800 2800
 F 0 "VIN" H 1800 2800 30  0001 L CNN
-F 1 "VSIN" H 1800 2880 30  0001 L CNN
+F 1 "SINE" H 1800 2880 30  0001 L CNN
 	1    1800 2800
-	1    0    0    1
+	1    0    0    -1
 $EndComp
 $Comp
@@
 F 1 "13V" H 3300 2970 30  0000 C CNN
 	1    3300 2700
-	-1    0    0    -1
+	-1    0    0    1
 $EndComp
 $Comp
@@
 F 1 "13V" H 3300 3590 30  0000 C CNN
 	1    3300 3700
-	-1    0    0    -1
+	-1    0    0    1
 $EndComp
 $Comp
@@
 F 1 "uA741" H 2900 2880 30  0001 L CNN
 	1    2900 2800
-	1    0    0    1
+	1    0    0    -1
 $EndComp
 $Comp
@@
 F 1 "{RL}" H 3100 4310 30  0000 L CNN
 	1    3100 4200
-	1    0    0    1
+	1    0    0    -1
 $EndComp
 Wire Wire Line

Commit message: Removed the use of exec, wrote basename function, made integration with eSim easier.
Parts:
- added RL: {RL}, symbol R_PSPICE
- added titleblk: titleblk, symbol titleblk_PSPICE
- PM1: renamed from R2; value 10k -> PARAM; symbol R_PSPICE -> PARAM_PSPICE
- R2: renamed from VIN; value SINE -> 10k; symbol VSIN_PSPICE -> R_PSPICE
- U1: renamed from RL; value {RL} -> uA741; symbol R_PSPICE -> uA741_PSPICE
- V2: renamed from U1; value uA741 -> 13V; symbol uA741_PSPICE -> VDC_PSPICE
- VIN: renamed from V1; value 13V -> SINE; symbol VDC_PSPICE -> VSIN_PSPICE
- renumbered V2 to V1
Changed lines of the file:
@@
-EESchema Schematic File Version 2  date Tuesday 22 June 1999 10:24:53 AM IST
+EESchema Schematic File Version 2  date
 LIBS:power
 LIBS:device
@@
 LIBS:contrib
 LIBS:valves
-LIBS:ConvertedSchematicFiles/EXP9_11-cache
 EELAYER 25  0
 EELAYER END
@@
 Sheet 1 1
 Title ""
-Date "22 Jun 1999"
+Date ""
 Rev ""
 Comp ""
@@
 $EndComp
 $Comp
+L PARAM_PSPICE PM1
+U 1 1 77747793
+P 5600 2200
+F 0 "PM1" H 5600 2200 30  0000 L CNN
+F 1 "PARAM" H 5600 2280 30  0000 L CNN
+	1    5600 2200
+	1    0    0    -1
+$EndComp
+$Comp
 L R_PSPICE R2
-U 1 1 77747793
+U 1 1 74238335
 P 2200 3200
 F 0 "R2" H 2200 3200 30  0001 L CNN
@@
 $Comp
 L VSIN_PSPICE VIN
-U 1 1 74238335
+U 1 1 99885386
 P 1800 2800
 F 0 "VIN" H 1800 2800 30  0001 L CNN
@@
 $Comp
 L VDC_PSPICE V1
-U 1 1 99885386
+U 1 1 39760492
 P 3300 2700
 F 0 "V1" H 3300 2700 30  0001 L CNN
@@
 $Comp
 L VDC_PSPICE V2
-U 1 1 39760492
+U 1 1 66516649
 P 3300 3700
 F 0 "V2" H 3300 3700 30  0001 L CNN
@@
 $Comp
 L uA741_PSPICE U1
-U 1 1 66516649
+U 1 1 29641421
 P 2900 2800
 F 0 "U1" H 2900 2800 30  0001 L CNN
@@
 $Comp
 L R_PSPICE RL
-U 1 1 29641421
+U 1 1 45202362
 P 3100 4200
 F 0 "RL" H 3100 4200 30  0001 L CNN
@@
 	1    0    0    -1
 $EndComp
+$Comp
+L titleblk_PSPICE titleblk
+U 1 1 10490027
+P 9700 7200
+F 0 "titleblk" H 19400 14400 30  0001 L CNN
+F 1 "titleblk" H 19400 14480 30  0001 L CNN
+	1    9700 7200
+	1    0    0    -1
+$EndComp
