File: ConvertedSchematicFiles/NON_INV_AMP_IC741_OPEN/NON_INV_AMP_IC741_OPEN.sch (KiCad schematic (older format))
At the start: 13 parts, among them U1 uA741

Commit message: Excluded some components. These no longer appear after conversion. When calling shell commands, filenames are in "quotes"
Parts:
- removed R6: 1000k, symbol R_PSPICE
- removed titleblk: titleblk, symbol TITLEBLK_PSPICE
- R5: renamed from PM1; value PARAM -> 50; symbol PARAM_PSPICE -> R_PSPICE
- R6: renamed from U1; value uA741 -> 1000k; symbol uA741_PSPICE -> R_PSPICE
- U1: renamed from VIN1; value VSIN -> uA741; symbol VSIN_PSPICE -> uA741_PSPICE
- VIN1: renamed from R5; value 50 -> VSIN; symbol R_PSPICE -> VSIN_PSPICE
Connections:
- net at EGND.EGND: now also R6.2
- net at U1.+: now also R5.1; no longer VIN1.2
- net at V2.-: now also U1.V+; no longer R6.V+
- new net: R5.2, VIN1.+
Changed lines of the file:
@@
-$EndComp
-$Comp
-L PARAM_PSPICE PM1
-U 1 1 39760492
-P 4600 400
-F 0 "PM1" H 4600 400 30  0000 L CNN
-F 1 "PARAM" H 4600 480 30  0000 L CNN
-	1    4600 400
-	1    0    0    1
 $EndComp
 $Comp
 L R_PSPICE R5
-U 1 1 66516649
+U 1 1 39760492
 P 1900 1400
 F 0 "R5" H 1900 1400 30  0000 L CNN
@@
 $Comp
 L VSIN_PSPICE VIN1
-U 1 1 29641421
+U 1 1 66516649
 P 1200 1400
 F 0 "VIN1" H 1200 1400 30  0000 L CNN
@@
 $Comp
 L uA741_PSPICE U1
-U 1 1 45202362
+U 1 1 29641421
 P 2100 1400
 F 0 "U1" H 2100 1400 30  0000 L CNN
@@
 $Comp
 L R_PSPICE R6
-U 1 1 10490027
+U 1 1 45202362
 P 3600 1600
 F 0 "R6" H 3600 1600 30  0000 L CNN
@@
 	0    -1    1    0
 $EndComp
-$Comp
-L TITLEBLK_PSPICE titleblk
-U 1 1 73368690
-P 9700 7200
-F 0 "titleblk" H 19400 14400 30  0001 L CNN
-F 1 "titleblk" H 19400 14480 30  0001 L CNN
-	1    9700 7200
-	1    0    0    1
-$EndComp
 Wire Wire Line

Commit message: Ports issue fixed. Now annotation for ports is #PWR? function added "itos"
Parts:
- removed EGND (x5): EGND, symbol EGND_PSPICE
Changed lines of the file:
@@
 $EndDescr
 $Comp
-L EGND_PSPICE EGND
+L EGND_PSPICE #PWR1
 U 1 1 14289383
 P 3100 1100
-F 0 "EGND" H 6200 2200 30  0001 L CNN
+F 0 "#PWR1" H 6200 2200 30  0001 L CNN
 F 1 "EGND" H 6200 2280 30  0001 L CNN
 	1    3100 1100
@@
 $EndComp
 $Comp
-L EGND_PSPICE EGND
+L EGND_PSPICE #PWR2
 U 1 1 46930886
 P 2500 2300
-F 0 "EGND" H 5000 4600 30  0001 L CNN
+F 0 "#PWR2" H 5000 4600 30  0001 L CNN
 F 1 "EGND" H 5000 4680 30  0001 L CNN
 	1    2500 2300
@@
 $EndComp
 $Comp
-L EGND_PSPICE EGND
+L EGND_PSPICE #PWR3
 U 1 1 71692777
 P 3600 2000
-F 0 "EGND" H 7200 4000 30  0001 L CNN
+F 0 "#PWR3" H 7200 4000 30  0001 L CNN
 F 1 "EGND" H 7200 4080 30  0001 L CNN
 	1    3600 2000
@@
 $EndComp
 $Comp
-L EGND_PSPICE EGND
+L EGND_PSPICE #PWR4
 U 1 1 14636915
 P 1200 2100
-F 0 "EGND" H 2400 4200 30  0001 L CNN
+F 0 "#PWR4" H 2400 4200 30  0001 L CNN
 F 1 "EGND" H 2400 4280 30  0001 L CNN
 	1    1200 2100
@@
 $EndComp
 $Comp
-L EGND_PSPICE EGND
+L EGND_PSPICE #PWR5
 U 1 1 77747793
 P 1800 1800
-F 0 "EGND" H 3600 3600 30  0001 L CNN
+F 0 "#PWR5" H 3600 3600 30  0001 L CNN
 F 1 "EGND" H 3600 3680 30  0001 L CNN
 	1    1800 1800

Commit message: Added LICENSE.txt
Changed lines of the file:
@@
 $EndDescr
 $Comp
-L EGND_PSPICE #PWR1
+L GND #PWR1
 U 1 1 14289383
 P 3100 1100
@@
 $EndComp
 $Comp
-L EGND_PSPICE #PWR2
+L GND #PWR2
 U 1 1 46930886
 P 2500 2300
@@
 $EndComp
 $Comp
-L EGND_PSPICE #PWR3
+L GND #PWR3
 U 1 1 71692777
 P 3600 2000
@@
 $EndComp
 $Comp
-L EGND_PSPICE #PWR4
+L GND #PWR4
 U 1 1 14636915
 P 1200 2100
@@
 $EndComp
 $Comp
-L EGND_PSPICE #PWR5
+L GND #PWR5
 U 1 1 77747793
 P 1800 1800

Commit message: Orientation fix. Library components are now inverted, with +ve y axis going up. In Schematic files, +ve y axis is downwards. This is how the KiCad libraries are. As a result of the above fixed, the converted GND is now oriented correctly.
Parts:
- VIN1: value VSIN -> SINE
Other:
- moved on the sheet: U1, V1, V2, VIN1
Changed lines of the file:
@@
 F 1 "EGND" H 6200 2280 30  0001 L CNN
 	1    3100 1100
-	1    0    0    1
+	1    0    0    -1
 $EndComp
 $Comp
@@
 F 1 "EGND" H 5000 4680 30  0001 L CNN
 	1    2500 2300
-	1    0    0    1
+	1    0    0    -1
 $EndComp
 $Comp
@@
 F 1 "EGND" H 7200 4080 30  0001 L CNN
 	1    3600 2000
-	1    0    0    1
+	1    0    0    -1
 $EndComp
 $Comp
@@
 F 1 "EGND" H 2400 4280 30  0001 L CNN
 	1    1200 2100
-	-1    0    0    1
+	-1    0    0    -1
 $EndComp
 $Comp
@@
 F 1 "EGND" H 3600 3680 30  0001 L CNN
 	1    1800 1800
-	1    0    0    1
+	1    0    0    -1
 $EndComp
 $Comp
@@
 F 1 "15V" H 3100 590 30  0000 C CNN
 	1    3100 700
-	1    0    0    1
+	1    0    0    -1
 $EndComp
 $Comp
@@
 F 1 "-15V" H 2500 2190 30  0000 C CNN
 	1    2500 1900
-	1    0    0    1
+	1    0    0    -1
 $EndComp
 $Comp
@@
 F 1 "50" H 1900 1550 30  0000 L CNN
 	1    1900 1400
-	-1    0    0    1
+	-1    0    0    -1
 $EndComp
 $Comp
@@
 P 1200 1400
 F 0 "VIN1" H 1200 1400 30  0000 L CNN
-F 1 "VSIN" H 1200 1480 30  0000 L CNN
+F 1 "SINE" H 1200 1480 30  0000 L CNN
 	1    1200 1400
-	-1    0    0    1
+	-1    0    0    -1
 $EndComp
 $Comp
@@
 F 1 "uA741" H 2100 1480 30  0000 L CNN
 	1    2100 1400
-	1    0    0    1
+	1    0    0    -1
 $EndComp
 $Comp
@@
 F 1 "1000k" H 3600 1890 30  0000 L CNN
 	1    3600 1600
-	0    -1    1    0
+	0    1    1    0
 $EndComp
 Wire Wire Line

Commit message: Removed the use of exec, wrote basename function, made integration with eSim easier.
Parts:
- added R6: 1000k, symbol R_PSPICE
- added titleblk: titleblk, symbol titleblk_PSPICE
- PM1: renamed from R5; value 50 -> PARAM; symbol R_PSPICE -> PARAM_PSPICE
- R5: renamed from VIN1; value SINE -> 50; symbol VSIN_PSPICE -> R_PSPICE
- U1: renamed from R6; value 1000k -> uA741; symbol R_PSPICE -> uA741_PSPICE
- VIN1: renamed from U1; value uA741 -> SINE; symbol uA741_PSPICE -> VSIN_PSPICE
Changed lines of the file:
@@
-EESchema Schematic File Version 2  date Monday 21 June 1999 12:18:02 AM IST
+EESchema Schematic File Version 2  date
 LIBS:power
 LIBS:device
@@
 LIBS:contrib
 LIBS:valves
-LIBS:ConvertedSchematicFiles/NON_INV_AMP_IC741_OPEN-cache
 EELAYER 25  0
 EELAYER END
@@
 Sheet 1 1
 Title ""
-Date "21 Jun 1999"
+Date ""
 Rev ""
 Comp ""
@@
 $EndComp
 $Comp
+L PARAM_PSPICE PM1
+U 1 1 39760492
+P 4600 400
+F 0 "PM1" H 4600 400 30  0000 L CNN
+F 1 "PARAM" H 4600 480 30  0000 L CNN
+	1    4600 400
+	1    0    0    -1
+$EndComp
+$Comp
 L R_PSPICE R5
-U 1 1 39760492
+U 1 1 66516649
 P 1900 1400
 F 0 "R5" H 1900 1400 30  0000 L CNN
@@
 $Comp
 L VSIN_PSPICE VIN1
-U 1 1 66516649
+U 1 1 29641421
 P 1200 1400
 F 0 "VIN1" H 1200 1400 30  0000 L CNN
@@
 $Comp
 L uA741_PSPICE U1
-U 1 1 29641421
+U 1 1 45202362
 P 2100 1400
 F 0 "U1" H 2100 1400 30  0000 L CNN
@@
 $Comp
 L R_PSPICE R6
-U 1 1 45202362
+U 1 1 10490027
 P 3600 1600
 F 0 "R6" H 3600 1600 30  0000 L CNN
@@
 	0    1    1    0
 $EndComp
+$Comp
+L titleblk_PSPICE titleblk
+U 1 1 73368690
+P 9700 7200
+F 0 "titleblk" H 19400 14400 30  0001 L CNN
+F 1 "titleblk" H 19400 14480 30  0001 L CNN
+	1    9700 7200
+	1    0    0    -1
+$EndComp
 Wire Wire Line
