File: ConvertedSchematicFiles/VCO/VCO.sch (KiCad schematic (older format))
At the start: 27 parts, among them M2 IRF150, U1 LF411, U2 LM111

Commit message: Excluded some components. These no longer appear after conversion. When calling shell commands, filenames are in "quotes"
Parts:
- removed C1: 12.5P, symbol C_PSPICE
- removed nodeMarker (x5): nodeMarker, symbol NODEMARKER_PSPICE
- removed titleblk: titleblk, symbol TITLEBLK_PSPICE
- C1: renamed from V1; value VPWL -> 12.5P; symbol VPWL_PSPICE -> C_PSPICE
- U1: renamed from PM1; value PARAM -> LF411; symbol PARAM_PSPICE -> LF411_PSPICE
- V1: renamed from U1; value LF411 -> VPWL; symbol LF411_PSPICE -> VPWL_PSPICE
Changed lines of the file:
@@
-$EndComp
-$Comp
-L PARAM_PSPICE PM1
-U 1 1 20383426
-P 3800 200
-F 0 "PM1" H 3800 200 30  0000 L CNN
-F 1 "PARAM" H 3800 280 30  0000 L CNN
-	1    3800 200
-	1    0    0    1
 $EndComp
 $Comp
 L LF411_PSPICE U1
-U 1 1 44089172
+U 1 1 20383426
 P 1800 1400
 F 0 "U1" H 1800 1400 30  0000 L CNN
@@
 $Comp
 L VPWL_PSPICE V1
-U 1 1 53455736
+U 1 1 44089172
 P 300 600
 F 0 "V1" H 300 600 30  0000 L CNN
@@
 $Comp
 L C_PSPICE C1
-U 1 1 45005211
+U 1 1 53455736
 P 2000 400
 F 0 "C1" H 2000 400 30  0000 L CNN
@@
 	1    0    0    1
 $EndComp
-$Comp
-L TITLEBLK_PSPICE titleblk
-U 1 1 81595368
-P 11880 8400
-F 0 "titleblk" H 23760 16800 30  0001 L CNN
-F 1 "titleblk" H 23760 16880 30  0001 L CNN
-	1    11880 8400
-	1    0    0    1
-$EndComp
-$Comp
-L NODEMARKER_PSPICE nodeMarker
-U 1 1 34702567
-P 4700 1300
-F 0 "nodeMarker" H 9400 2600 30  0001 L CNN
-F 1 "nodeMarker" H 9400 2680 30  0001 L CNN
-	1    4700 1300
-	1    0    0    1
-$EndComp
-$Comp
-L NODEMARKER_PSPICE nodeMarker
-U 1 1 26956429
-P 3100 1200
-F 0 "nodeMarker" H 6200 2400 30  0001 L CNN
-F 1 "nodeMarker" H 6200 2480 30  0001 L CNN
-	1    3100 1200
-	1    0    0    1
-$EndComp
-$Comp
-L NODEMARKER_PSPICE nodeMarker
-U 1 1 76465782
-P 300 400
-F 0 "nodeMarker" H 600 800 30  0001 L CNN
-F 1 "nodeMarker" H 600 880 30  0001 L CNN
-	1    300 400
-	1    0    0    1
-$EndComp
-$Comp
-L NODEMARKER_PSPICE nodeMarker
-U 1 1 61021530
-P 1800 1400
-F 0 "nodeMarker" H 3600 2800 30  0001 L CNN
-F 1 "nodeMarker" H 3600 2880 30  0001 L CNN
-	1    1800 1400
-	1    0    0    1
-$EndComp
-$Comp
-L NODEMARKER_PSPICE nodeMarker
-U 1 1 18722862
-P 1800 1000
-F 0 "nodeMarker" H 3600 2000 30  0001 L CNN
-F 1 "nodeMarker" H 3600 2080 30  0001 L CNN
-	1    1800 1000
-	1    0    0    1
-$EndComp

Commit message: Ports issue fixed. Now annotation for ports is #PWR? function added "itos"
Parts:
- removed EGND (x7): EGND, symbol EGND_PSPICE
Connections:
- net labels added: EGND
Changed lines of the file:
@@
 $EndDescr
 $Comp
-L EGND_PSPICE EGND
+L EGND_PSPICE #PWR1
 U 1 1 14289383
 P 300 1000
-F 0 "EGND" H 600 2000 30  0001 L CNN
+F 0 "#PWR1" H 600 2000 30  0001 L CNN
 F 1 "EGND" H 600 2080 30  0001 L CNN
 	1    300 1000
@@
 $EndComp
 $Comp
-L EGND_PSPICE EGND
+L EGND_PSPICE #PWR2
 U 1 1 46930886
 P 2800 1000
-F 0 "EGND" H 5600 2000 30  0001 L CNN
+F 0 "#PWR2" H 5600 2000 30  0001 L CNN
 F 1 "EGND" H 5600 2080 30  0001 L CNN
 	1    2800 1000
@@
 $EndComp
 $Comp
-L EGND_PSPICE EGND
+L EGND_PSPICE #PWR3
 U 1 1 71692777
 P 2800 2200
-F 0 "EGND" H 5600 4400 30  0001 L CNN
+F 0 "#PWR3" H 5600 4400 30  0001 L CNN
 F 1 "EGND" H 5600 4480 30  0001 L CNN
 	1    2800 2200
@@
 $EndComp
 $Comp
-L EGND_PSPICE EGND
+L EGND_PSPICE #PWR4
 U 1 1 14636915
 P 900 1900
-F 0 "EGND" H 1800 3800 30  0001 L CNN
+F 0 "#PWR4" H 1800 3800 30  0001 L CNN
 F 1 "EGND" H 1800 3880 30  0001 L CNN
 	1    900 1900
@@
 $EndComp
 $Comp
-L EGND_PSPICE EGND
+L EGND_PSPICE #PWR5
 U 1 1 77747793
 P 4700 2300
-F 0 "EGND" H 9400 4600 30  0001 L CNN
+F 0 "#PWR5" H 9400 4600 30  0001 L CNN
 F 1 "EGND" H 9400 4680 30  0001 L CNN
 	1    4700 2300
@@
 $EndComp
 $Comp
-L EGND_PSPICE EGND
+L EGND_PSPICE #PWR6
 U 1 1 74238335
 P 4400 1100
-F 0 "EGND" H 8800 2200 30  0001 L CNN
+F 0 "#PWR6" H 8800 2200 30  0001 L CNN
 F 1 "EGND" H 8800 2280 30  0001 L CNN
 	1    4400 1100
@@
 $EndComp
 $Comp
-L EGND_PSPICE EGND
+L EGND_PSPICE #PWR7
 U 1 1 99885386
 P 1400 2400
-F 0 "EGND" H 2800 4800 30  0001 L CNN
+F 0 "#PWR7" H 2800 4800 30  0001 L CNN
 F 1 "EGND" H 2800 4880 30  0001 L CNN
 	1    1400 2400

Commit message: Added LICENSE.txt
Parts:
- renumbered M2 to Q?
Changed lines of the file:
@@
 $EndDescr
 $Comp
-L EGND_PSPICE #PWR1
+L GND #PWR1
 U 1 1 14289383
 P 300 1000
@@
 $EndComp
 $Comp
-L EGND_PSPICE #PWR2
+L GND #PWR2
 U 1 1 46930886
 P 2800 1000
@@
 $EndComp
 $Comp
-L EGND_PSPICE #PWR3
+L GND #PWR3
 U 1 1 71692777
 P 2800 2200
@@
 $EndComp
 $Comp
-L EGND_PSPICE #PWR4
+L GND #PWR4
 U 1 1 14636915
 P 900 1900
@@
 $EndComp
 $Comp
-L EGND_PSPICE #PWR5
+L GND #PWR5
 U 1 1 77747793
 P 4700 2300
@@
 $EndComp
 $Comp
-L EGND_PSPICE #PWR6
+L GND #PWR6
 U 1 1 74238335
 P 4400 1100
@@
 $EndComp
 $Comp
-L EGND_PSPICE #PWR7
+L GND #PWR7
 U 1 1 99885386
 P 1400 2400
@@
 $EndComp
 $Comp
-L IRF150_PSPICE M2
+L IRF150_PSPICE Q?
 U 1 1 25180540
 P 1700 2200
-F 0 "M2" H 1700 2200 30  0000 L CNN
+F 0 "Q?" H 1700 2200 30  0000 L CNN
 F 1 "IRF150" H 1700 2280 30  0000 L CNN
 	1    1700 2200

Commit message: Orientation fix. Library components are now inverted, with +ve y axis going up. In Schematic files, +ve y axis is downwards. This is how the KiCad libraries are. As a result of the above fixed, the converted GND is now oriented correctly.
Other:
- moved on the sheet: U1, U2, V1, V2, V3
Changed lines of the file:
@@
 F 1 "EGND" H 600 2080 30  0001 L CNN
 	1    300 1000
-	1    0    0    1
+	1    0    0    -1
 $EndComp
 $Comp
@@
 F 1 "EGND" H 5600 2080 30  0001 L CNN
 	1    2800 1000
-	1    0    0    1
+	1    0    0    -1
 $EndComp
 $Comp
@@
 F 1 "EGND" H 5600 4480 30  0001 L CNN
 	1    2800 2200
-	1    0    0    1
+	1    0    0    -1
 $EndComp
 $Comp
@@
 F 1 "EGND" H 1800 3880 30  0001 L CNN
 	1    900 1900
-	1    0    0    1
+	1    0    0    -1
 $EndComp
 $Comp
@@
 F 1 "EGND" H 9400 4680 30  0001 L CNN
 	1    4700 2300
-	1    0    0    1
+	1    0    0    -1
 $EndComp
 $Comp
@@
 F 1 "EGND" H 8800 2280 30  0001 L CNN
 	1    4400 1100
-	1    0    0    1
+	1    0    0    -1
 $EndComp
 $Comp
@@
 F 1 "EGND" H 2800 4880 30  0001 L CNN
 	1    1400 2400
-	1    0    0    1
+	1    0    0    -1
 $EndComp
 $Comp
@@
 F 1 "-15V" H 2800 490 30  0000 C CNN
 	1    2800 600
-	1    0    0    1
+	1    0    0    -1
 $EndComp
 $Comp
@@
 F 1 "10k" H 900 1650 30  0000 L CNN
 	1    900 1500
-	0    -1    1    0
+	0    1    1    0
 $EndComp
 $Comp
@@
 F 1 "10k" H 900 850 30  0000 L CNN
 	1    900 700
-	0    -1    1    0
+	0    1    1    0
 $EndComp
 $Comp
@@
 F 1 "1.8k" H 4700 750 30  0000 L CNN
 	1    4700 600
-	0    -1    1    0
+	0    1    1    0
 $EndComp
 $Comp
@@
 F 1 "15V" H 2800 1690 30  0000 C CNN
 	1    2800 1800
-	1    0    0    1
+	1    0    0    -1
 $EndComp
 $Comp
@@
 F 1 "3.6k" H 4700 2050 30  0000 L CNN
 	1    4700 1900
-	0    -1    1    0
+	0    1    1    0
 $EndComp
 $Comp
@@
 F 1 "{2*R}" H 1200 450 30  0000 L CNN
 	1    1200 400
-	1    0    0    1
+	1    0    0    -1
 $EndComp
 $Comp
@@
 F 1 "LM111" H 3600 1580 30  0000 L CNN
 	1    3600 1500
-	1    0    0    -1
+	1    0    0    1
 $EndComp
 $Comp
@@
 F 1 "{R}" H 1400 1970 30  0000 L CNN
 	1    1400 1600
-	0    -1    1    0
+	0    1    1    0
 $EndComp
 $Comp
@@
 F 1 "IRF150" H 1700 2280 30  0000 L CNN
 	1    1700 2200
-	-1    0    0    1
+	-1    0    0    -1
 $EndComp
 $Comp
@@
 F 1 "LF411" H 1800 1480 30  0000 L CNN
 	1    1800 1400
-	1    0    0    -1
+	1    0    0    1
 $EndComp
 $Comp
@@
 F 1 "VPWL" H 300 680 30  0000 L CNN
 	1    300 600
-	1    0    0    1
+	1    0    0    -1
 $EndComp
 $Comp
@@
 F 1 "12.5P" H 2000 550 30  0000 L CNN
 	1    2000 400
-	1    0    0    1
+	1    0    0    -1
 $EndComp
 Wire Wire Line

Commit message: Removed the use of exec, wrote basename function, made integration with eSim easier.
Parts:
- added C1: 12.5P, symbol C_PSPICE
- added nodeMarker (x5): nodeMarker, symbol nodeMarker_PSPICE
- added titleblk: titleblk, symbol titleblk_PSPICE
- PM1: renamed from U1; value LF411 -> PARAM; symbol LF411_PSPICE -> PARAM_PSPICE
- U1: renamed from V1; value VPWL -> LF411; symbol VPWL_PSPICE -> LF411_PSPICE
- V1: renamed from C1; value 12.5P -> VPWL; symbol C_PSPICE -> VPWL_PSPICE
Changed lines of the file:
@@
-EESchema Schematic File Version 2  date Wednesday 23 June 1999 09:51:37 AM IST
+EESchema Schematic File Version 2  date
 LIBS:power
 LIBS:device
@@
 LIBS:contrib
 LIBS:valves
-LIBS:ConvertedSchematicFiles/VCO-cache
 EELAYER 25  0
 EELAYER END
@@
 Sheet 1 1
 Title ""
-Date "23 Jun 1999"
+Date ""
 Rev ""
 Comp ""
@@
 $EndComp
 $Comp
+L PARAM_PSPICE PM1
+U 1 1 20383426
+P 3800 200
+F 0 "PM1" H 3800 200 30  0000 L CNN
+F 1 "PARAM" H 3800 280 30  0000 L CNN
+	1    3800 200
+	1    0    0    -1
+$EndComp
+$Comp
 L LF411_PSPICE U1
-U 1 1 20383426
+U 1 1 44089172
 P 1800 1400
 F 0 "U1" H 1800 1400 30  0000 L CNN
@@
 $Comp
 L VPWL_PSPICE V1
-U 1 1 44089172
+U 1 1 53455736
 P 300 600
 F 0 "V1" H 300 600 30  0000 L CNN
@@
 $Comp
 L C_PSPICE C1
-U 1 1 53455736
+U 1 1 45005211
 P 2000 400
 F 0 "C1" H 2000 400 30  0000 L CNN
@@
 	1    0    0    -1
 $EndComp
+$Comp
+L titleblk_PSPICE titleblk
+U 1 1 81595368
+P 11880 8400
+F 0 "titleblk" H 23760 16800 30  0001 L CNN
+F 1 "titleblk" H 23760 16880 30  0001 L CNN
+	1    11880 8400
+	1    0    0    -1
+$EndComp
+$Comp
+L nodeMarker_PSPICE nodeMarker
+U 1 1 34702567
+P 4700 1300
+F 0 "nodeMarker" H 9400 2600 30  0001 L CNN
+F 1 "nodeMarker" H 9400 2680 30  0001 L CNN
+	1    4700 1300
+	1    0    0    -1
+$EndComp
+$Comp
+L nodeMarker_PSPICE nodeMarker
+U 1 1 26956429
+P 3100 1200
+F 0 "nodeMarker" H 6200 2400 30  0001 L CNN
+F 1 "nodeMarker" H 6200 2480 30  0001 L CNN
+	1    3100 1200
+	1    0    0    -1
+$EndComp
+$Comp
+L nodeMarker_PSPICE nodeMarker
+U 1 1 76465782
+P 300 400
+F 0 "nodeMarker" H 600 800 30  0001 L CNN
+F 1 "nodeMarker" H 600 880 30  0001 L CNN
+	1    300 400
+	1    0    0    -1
+$EndComp
+$Comp
+L nodeMarker_PSPICE nodeMarker
+U 1 1 61021530
+P 1800 1400
+F 0 "nodeMarker" H 3600 2800 30  0001 L CNN
+F 1 "nodeMarker" H 3600 2880 30  0001 L CNN
+	1    1800 1400
+	1    0    0    -1
+$EndComp
+$Comp
+L nodeMarker_PSPICE nodeMarker
+U 1 1 18722862
+P 1800 1000
+F 0 "nodeMarker" H 3600 2000 30  0001 L CNN
+F 1 "nodeMarker" H 3600 2080 30  0001 L CNN
+	1    1800 1000
+	1    0    0    -1
+$EndComp
